File: hardware/pcb/magnetometer_node_mainboard/schematics/sensor_offset_drivers.kicad_sch (KiCad schematic)
At the start: 0 parts

Commit message: Schematic sensor stage done
Parts:
- added C4, C5, C6, C7, C8, C9: 100n, symbol Device:C
- added Q10, Q6, Q8: B772, Package_TO_SOT_SMD:SOT-89-3, symbol Device:Q_PNP
- added Q5, Q7, Q9: D882, Package_TO_SOT_SMD:SOT-89-3, symbol Device:Q_NPN
- added R10, R11, R12, R13, R14, R15, R19, R20, R21, R22, R8, R9: 10k, symbol Device:R
- added R16, R17, R23, R24, R5, R6: 100, symbol Device:R
- added R18: 20, Resistor_SMD:R_1206_3216Metric, symbol Device:R
- added R25, R7: 20, symbol Device:R
- added TP1: TestPoint, symbol Connector:TestPoint
- added U3: MCP4728, Package_SO:MSOP-10_3x3mm_P0.5mm, symbol Analog_DAC:MCP4728
- added U4: LM324, symbol Amplifier_Operational:LM324
Connections:
- new net: C6.1, R12.2, R14.1, U4.5 (+)
- new net: C6.2, Q7.E, Q8.E, R14.2, R18.1
- new net: C9.1, R20.2, R22.1, U4.9 (-)
- new net: C8.1, R19.2, R21.1, U4.10 (+)
- new net: C8.2, Q10.E, Q9.E, R21.2, R25.1
- new net: Q7.B, R16.2
- new net: C7.1, R13.2, R15.1, U4.6 (-)
- new net: R16.1, R17.1, U4.7
- new net: R23.1, R24.1, U4.8
- new net: Q10.B, R24.2
- new net: Q9.B, R23.2
- new net: U4.13 (-), U4.14
- new net: Q8.B, R17.2
- new net +3V3D: U3.1 (VDD)
- new net +4V5A: Q5.C, Q7.C, Q9.C, U4.4 (V+)
- new net -5VA: Q10.C, Q6.C, Q8.C, U4.11 (V-)
- new net DAC_LDAC_N: U3.4 (~{LDAC})
- new net DAC_OUT_REF: R13.1, R20.1, R9.1, U3.9 (VOUTD)
- new net DAC_OUT_X: R8.1, U3.6 (VOUTA)
- new net DAC_OUT_Y: R12.1, U3.7 (VOUTB)
- new net DAC_OUT_Z: R19.1, U3.8 (VOUTC)
- new net DAC_RDY_N: TP1.1, U3.5 (RDY/~{BSY})
- new net GND: U3.10 (VSS), U4.12 (+)
- new net I2C_DAC_SCL: U3.2 (SCL)
- new net I2C_DAC_SDA: U3.3 (SDA)
- new net OFFSET_X+: C5.2, R11.2, R7.2
- new net OFFSET_Y+: C7.2, R15.2, R18.2
- new net OFFSET_Z+: C9.2, R22.2, R25.2
- new net OFF_X_BN: Q5.B, R5.2
- new net OFF_X_BP: Q6.B, R6.2
- new net OFF_X_DRV: R5.1, R6.1, U4.1
- new net OFF_X_INN: C5.1, R11.1, R9.2, U4.2 (-)
- new net OFF_X_INP: C4.1, R10.1, R8.2, U4.3 (+)
- new net OFF_X_SENSE_P: C4.2, Q5.E, Q6.E, R10.2, R7.1
Other:
- note added: "DAC CH0 → OFFSET_X DAC CH1 → OFFSET_Y DAC CH2 → OFFSET_Z DAC_CH3 → idscale reference (Negative input of OPAMP)"
