File: hardware/pcb/magnetometer_node_mainboard/schematics/sensor_offset_drivers.kicad_sch (KiCad schematic)
At the start: 36 parts, among them Q10 B772, Q5 D882, Q6 B772, Q7 D882, Q8 B772, Q9 D882, U3 MCP4728, U4 LM324

Commit message: esp32_testing
Connections:
- net OFF_Y_INP: now reaches C6.1, R12.2, R14.1, U4.5 (+)
- net OFF_Y_SENSE_P: now reaches C6.2, Q7.E, Q8.E, R14.2, R18.1
- net OFF_Z_INN: now reaches C9.1, R20.2, R22.1, U4.9 (-)
- net OFF_Z_INP: now reaches C8.1, R19.2, R21.1, U4.10 (+)
- net OFF_Z_SENSE_P: now reaches C8.2, Q10.E, Q9.E, R21.2, R25.1
- net OFF_Y_BN: now reaches Q7.B, R16.2
- net OFF_Y_INN: now reaches C7.1, R13.2, R15.1, U4.6 (-)
- net OFF_Y_DRV: now reaches R16.1, R17.1, U4.7
- net OFF_Z_DRV: now reaches R23.1, R24.1, U4.8
- net OFF_Z_BP: now reaches Q10.B, R24.2
- net OFF_Z_BN: now reaches Q9.B, R23.2
- net UNUSED_LM324_CHD: now reaches U4.13 (-), U4.14
- net OFF_Y_BP: now reaches Q8.B, R17.2
Changed lines of the file:
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@@
+		)
+	)
+	(label "OFF_Y_BP"
+		(at 215.9 128.27 0)
+		(effects
+			(font
+				(size 0.635 0.635)
+			)
+			(justify left bottom)
+		)
+	)
+	(label "OFF_Y_INP"
+		(at 189.23 115.57 90)
+		(effects
+			(font
+				(size 0.635 0.635)
+			)
+			(justify left bottom)
+		)
+	)
+	(label "OFF_Z_INN"
+		(at 113.03 163.83 90)
+		(effects
+			(font
+				(size 0.635 0.635)
+			)
+			(justify left bottom)
 		)
 	)
@@
 			(font
 				(size 1.27 1.27)
+			)
+			(justify left bottom)
+		)
+	)
+	(label "OFF_Z_INP"
+		(at 113.03 146.05 90)
+		(effects
+			(font
+				(size 0.635 0.635)
 			)
 			(justify left bottom)
@@
 		)
 	)
+	(label "OFF_Y_INN"
+		(at 189.23 133.35 90)
+		(effects
+			(font
+				(size 0.635 0.635)
+			)
+			(justify left bottom)
+		)
+	)
+	(label "OFF_Y_SENSE_P"
+		(at 212.09 104.14 0)
+		(effects
+			(font
+				(size 0.635 0.635)
+			)
+			(justify left bottom)
+		)
+	)
+	(label "OFF_Z_DRV"
+		(at 130.81 151.13 90)
+		(effects
+			(font
+				(size 0.635 0.635)
+			)
+			(justify left bottom)
+		)
+	)
+	(label "OFF_Z_SENSE_P"
+		(at 134.62 134.62 0)
+		(effects
+			(font
+				(size 0.635 0.635)
+			)
+			(justify left bottom)
+		)
+	)
 	(label "DAC_OUT_REF"
 		(at 87.63 80.01 0)
@@
 			(font
 				(size 1.27 1.27)
+			)
+			(justify left bottom)
+		)
+	)
+	(label "OFF_Z_BP"
+		(at 139.7 158.75 0)
+		(effects
+			(font
+				(size 0.635 0.635)
 			)
 			(justify left bottom)
@@
 		)
 	)
+	(label "OFF_Z_BN"
+		(at 139.7 146.05 0)
+		(effects
+			(font
+				(size 0.635 0.635)
+			)
+			(justify left bottom)
+		)
+	)
+	(label "OFF_Y_DRV"
+		(at 207.01 120.65 90)
+		(effects
+			(font
+				(size 0.635 0.635)
+			)
+			(justify left bottom)
+		)
+	)
 	(label "OFF_X_DRV"
 		(at 207.01 50.8 90)
+		(effects
+			(font
+				(size 0.635 0.635)
+			)
+			(justify left bottom)
+		)
+	)
+	(label "UNUSED_LM324_CHD"
+		(at 43.18 185.42 0)
 		(effects
 			(font
@@
 		(effects
 			(font
+				(size 0.635 0.635)
+			)
+			(justify left bottom)
+		)
+	)
+	(label "OFF_Y_BN"
+		(at 215.9 115.57 0)
+		(effects
+			(font

Commit message: first code for the v1
Parts:
- removed Q10, Q6, Q8: B772, Package_TO_SOT_SMD:SOT-89-3, symbol Device:Q_PNP
- removed Q5, Q7, Q9: D882, Package_TO_SOT_SMD:SOT-89-3, symbol Device:Q_NPN
- removed R10, R11, R12, R13, R14, R15, R19, R20, R21, R22, R8, R9: 10k, symbol Device:R
- added C8: 100n, Capacitor_SMD:C_0603_1608Metric, symbol Device:C
- added Q10, Q6, Q8: B772, Package_TO_SOT_SMD:SOT-89-3, symbol magnode_symbols:B772
- added Q5, Q7, Q9: D882, Package_TO_SOT_SMD:SOT-89-3, symbol magnode_symbols:D882
- added RN1, RN2, RN3: 10k, Resistor_SMD:R_Array_Convex_4x0612, symbol Device:R_Network04_Split
- C10: renamed from C6; value 100n -> 10u; footprint (none) -> Capacitor_SMD:C_0805_2012Metric; LCSC (none) -> C15850
- C11: renamed from C8; value 100n -> 10u; footprint (none) -> Capacitor_SMD:C_0805_2012Metric; LCSC (none) -> C15850
- C12: renamed from C7; value 100n -> 10u; footprint (none) -> Capacitor_SMD:C_0805_2012Metric; LCSC (none) -> C15850
- C13: renamed from C9; value 100n -> 10u; footprint (none) -> Capacitor_SMD:C_0805_2012Metric; LCSC (none) -> C15850
- C7: renamed from C4; value 100n -> 10u; footprint (none) -> Capacitor_SMD:C_0805_2012Metric; LCSC (none) -> C15850
- C9: renamed from C5; value 100n -> 10u; footprint (none) -> Capacitor_SMD:C_0805_2012Metric; LCSC (none) -> C15850
- R10: renamed from R6; footprint (none) -> Resistor_SMD:R_0603_1608Metric; LCSC (none) -> C22775
- R11: renamed from R7; footprint (none) -> Resistor_SMD:R_1206_3216Metric; LCSC (none) -> C17955
- R12: renamed from R16; footprint (none) -> Resistor_SMD:R_0603_1608Metric; LCSC (none) -> C22775
- R13: renamed from R17; footprint (none) -> Resistor_SMD:R_0603_1608Metric; LCSC (none) -> C22775
- R14: renamed from R18; LCSC (none) -> C17955
- R15: renamed from R23; footprint (none) -> Resistor_SMD:R_0603_1608Metric; LCSC (none) -> C22775
- R16: renamed from R24; footprint (none) -> Resistor_SMD:R_0603_1608Metric; LCSC (none) -> C22775
- R17: renamed from R25; footprint (none) -> Resistor_SMD:R_1206_3216Metric; LCSC (none) -> C17955
- R9: renamed from R5; footprint (none) -> Resistor_SMD:R_0603_1608Metric; LCSC (none) -> C22775
- TP1: footprint (none) -> TestPoint:TestPoint_THTPad_1.0x1.0mm_Drill0.5mm
- U4: footprint (none) -> Package_SO:SOIC-14_3.9x8.7mm_P1.27mm
- renumbered U3 to U5
Connections:
- net +3V3D: now also C8.1
- net -5VA: now also Q10.2, Q6.2, Q8.2
- net DAC_OUT_REF: now also RN1.1 (R1), RN2.1 (R1), RN3.1 (R1)
- net DAC_OUT_X: now also RN1.1 (R1)
- net DAC_OUT_Y: now also RN2.1 (R1)
- net DAC_OUT_Z: now also RN3.1 (R1)
- net GND: now also C8.2
- net OFFSET_X+: now also RN1.5 (R4.2)
- net OFFSET_Y+: now also RN2.5 (R4.2)
- net OFFSET_Z+: now also RN3.5 (R4.2)
- net OFF_X_BN: now also Q5.1
- net OFF_X_BP: now also Q6.1
- net OFF_X_INN: now also RN1.1 (R1), RN1.3 (R2.2)
- net OFF_X_INP: now also RN1.1 (R1), RN1.2 (R1.2)
- net OFF_X_SENSE_P: now also Q5.3, Q6.3, RN1.4 (R3.2)
- net OFF_Y_BN: now also Q7.1
- net OFF_Y_BP: now also Q8.1
- net OFF_Y_INN: now also RN2.1 (R1), RN2.3 (R2.2)
- net OFF_Y_INP: now also RN2.1 (R1), RN2.2 (R1.2)
- net OFF_Y_SENSE_P: now also Q7.3, Q8.3, RN2.4 (R3.2)
- net OFF_Z_BN: now also Q9.1
- net OFF_Z_BP: now also Q10.1
- net OFF_Z_INN: now also RN3.1 (R1), RN3.3 (R2.2)
- net OFF_Z_INP: now also RN3.1 (R1), RN3.2 (R1.2)
- net OFF_Z_SENSE_P: now also Q10.3, Q9.3, RN3.4 (R3.2)
- net +4V5A renamed +5V
- net +5V: now also Q5.2, Q7.2, Q9.2
- net I2C_DAC_SCL renamed I2C.SCL
- net I2C_DAC_SDA renamed I2C.SDA
