File: hardware/pcb/magnetometer_node_mainboard/schematics/sensor_set_reset_driver.kicad_sch (KiCad schematic)
At the start: 0 parts

Commit message: Schematic sensor stage done
Parts:
- added C1: 1n, symbol Device:C
- added C2: 10u, symbol Device:C
- added C3: 220n, symbol Device:C
- added D2: 1N4148WS, Diode_SMD:D_SOD-323, symbol Diode:1N4148WS
- added Q1, Q4: D882, Package_TO_SOT_SMD:SOT-89-3, symbol Device:Q_NPN
- added Q2: B772, Package_TO_SOT_SMD:SOT-89-3, symbol Device:Q_PNP
- added Q3: DMC3028LSD, Package_SO:SO-8_3.9x4.9mm_P1.27mm, symbol magnode_symbols:DMC3028LSD
- added R1, R2, R3: 1k, symbol Device:R
- added R4: 220, symbol Device:R
Connections:
- new net: C3.1, Q3.5 (D2), Q3.6 (D2), Q3.7 (D1), Q3.8 (D1)
- new net: C1.2, D2.1 (K), Q1.B, R1.2
- new net: Q1.C, R2.2
- new net: C2.1, Q3.3 (S2), Q4.C, R3.1, R4.1
- new net: Q2.B, Q4.B, R2.1, R3.2
- new net: Q2.E, Q3.4 (G2), Q4.E
- new net +18V: R4.2
- new net GND: C2.2, D2.2 (A), Q1.E, Q2.C, Q3.1 (S1)
- new net RESET_CTRL: Q3.2 (G1)
- new net SETRESET_STRAP: C3.2
- new net SET_CTRL: C1.1, R1.1
Other:
- note added: "Quand je vais faire le pcb, vérifier l'ordre des pins des transitors"
