File: hardware/pcb/magnetometer_node_mainboard/schematics/sensor_set_reset_driver.kicad_sch (KiCad schematic)
At the start: 12 parts, among them Q1 D882, Q2 B772, Q3 DMC3028LSD, Q4 D882

Commit message: first code for the v1
Parts:
- removed Q1, Q4: D882, Package_TO_SOT_SMD:SOT-89-3, symbol Device:Q_NPN
- removed Q2: B772, Package_TO_SOT_SMD:SOT-89-3, symbol Device:Q_PNP
- added C2: 10u, Capacitor_SMD:C_0805_2012Metric, symbol Device:C
- added C3: 4u7, Capacitor_SMD:C_1206_3216Metric, symbol Device:C
- added C6: 10n, Capacitor_SMD:C_0603_1608Metric, symbol Device:C
- added D1: SS34, Diode_SMD:D_SMA, symbol Device:D_Schottky
- added L1: 10u, Capacitor_SMD:C_0805_2012Metric, symbol Device:L
- added Q1, Q4: D882, Package_TO_SOT_SMD:SOT-89-3, symbol magnode_symbols:D882
- added Q3: B772, Package_TO_SOT_SMD:SOT-89-3, symbol magnode_symbols:B772
- added R3: 49k9, Resistor_SMD:R_0603_1608Metric, symbol Device:R
- added R5: 100k, Resistor_SMD:R_0603_1608Metric, symbol Device:R
- added R6: 10k, Resistor_SMD:R_0603_1608Metric, symbol Device:R
- added R7: 3k6, Resistor_SMD:R_0603_1608Metric, symbol Device:R
- added U3: TPS61170, Package_SON:WSON-6-1EP_2x2mm_P0.65mm_EP1x1.6mm, symbol magnode_symbols:TPS61170
- C1: renamed from C2; footprint (none) -> Capacitor_SMD:C_0805_2012Metric; LCSC (none) -> C15850
- C4: renamed from C3; footprint (none) -> Capacitor_SMD:C_0603_1608Metric; LCSC (none) -> C21120
- C5: renamed from C1; footprint (none) -> Capacitor_SMD:C_0603_1608Metric; LCSC (none) -> C1588
- D2: LCSC (none) -> C2128
- R1: renamed from R4; footprint (none) -> Resistor_SMD:R_0805_2012Metric; LCSC (none) -> C17557
- R2: renamed from R3; footprint (none) -> Resistor_SMD:R_0603_1608Metric; LCSC (none) -> C21190
- R4: renamed from R2; footprint (none) -> Resistor_SMD:R_0603_1608Metric; LCSC (none) -> C21190
- R8: renamed from R1; footprint (none) -> Resistor_SMD:R_0603_1608Metric; LCSC (none) -> C21190
- renumbered Q3 to Q2
Connections:
- net +18V: now also C3.1, D1.1 (K), R3.1
- net GND: now also C2.2, C3.2, C6.2, Q3.2, Q4.3 (E), R5.2, R7.2, U3.3 (GND), U3.7 (TP)
- net at C5.2, D2.1 (K), R8.2: now also Q4.1 (B)
- net at R4.2: now also Q4.2 (C)
- net at C1.1, Q2.3 (S2), R1.1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: now also Q1.2 (C)
- net at R2.2, R4.1: now also Q1.1 (B), Q3.1
- net at Q2.4 (G2): now also Q1.3 (E), Q3.3
- net RESET_CTRL renamed SENSOR_RESET_CTRL
- net SET_CTRL renamed SENSOR_SET_CTRL
- new net: D1.2 (A), L1.2, U3.4 (SW)
- new net: R3.2, R7.1, U3.1 (FB)
- new net: R6.1, U3.2 (COMP)
- new net: C6.1, R6.2
- new net +5V: C2.1, L1.1, U3.6 (VIN)
- new net EN_BST_18V: R5.1, U3.5 (CTRL)
Other:
- note added: "Check ESR (résistance) vitesse de décharge"
- moved on the sheet: C1, C4, C5, D2, Q2A, Q2B, R1, R2, R4, R8
