File: hardware/pcb/magnetometer_node_mainboard/schematics/gnss_imu.kicad_sch (KiCad schematic)
At the start: 0 parts

Commit message: esp32_testing
Parts:
- added U11: DAN-F10N, magnode_footprints:u-blox_DAN-F10N_LCC-56_20x20mm, symbol magnode_symbols:DANF10N
Changed lines of the file:
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@@
 	(generator_version "9.0")
 	(paper "A4")
+	(symbol
+		(lib_id "magnode_symbols:DANF10N")
+		(at 142.24 96.52 0)
+		(unit 1)
+		(exclude_from_sim no)
+		(in_bom yes)
+		(on_board yes)
+		(dnp no)
+		(fields_autoplaced yes)
+		(property "Reference" "U11"
+			(at 146.9233 57.15 0)
+			(effects
+				(font
+					(size 1.27 1.27)
+				)
+				(justify left)
+			)
+		)
+		(property "Value" "DAN-F10N"
+			(at 146.9233 59.69 0)
+			(effects
+				(font
+					(size 1.27 1.27)
+				)
+				(justify left)
+			)
+		)
+		(property "Footprint" "magnode_footprints:u-blox_DAN-F10N_LCC-56_20x20mm"
+			(at 142.24 96.52 0)
+			(effects
+				(font
+					(size 1.27 1.27)
+				)
+				(hide yes)
+			)
+		)
+		(property "Datasheet" "https://content.u-blox.com/sites/default/files/documents/DAN-F10N_DataSheet_UBXDOC-963802114-13074.pdf"
+			(at 142.24 150.622 0)
+			(effects
+				(font
+					(size 1.27 1.27)
+				)
+				(hide yes)
+			)
+		)
+		(property "Description" "GNSS module"
+			(at 142.494 147.574 0)
+			(effects
+				(font
+					(size 1.27 1.27)
+				)
+				(hide yes)
+			)
+		)
+		(pin "4"
+		)
+		(pin "52"
+		)
+		(pin "5"
+		)
+		(pin "13"
+		)
+		(pin "14"
+		)
+		(pin "15"
+		)
+		(pin "10"
+		)
+		(pin "21"
+		)
+		(pin "22"
+		)
+		(pin "23"
+		)
+		(pin "35"
+		)
+		(pin "26"
+		)
+		(pin "27"
+		)
+		(pin "53"
+		)
+		(pin "6"
+		)
+		(pin "55"
+		)
+		(pin "7"
+		)
+		(pin "8"
+		)
+		(pin "37"
+		)
+		(pin "16"
+		)
+		(pin "28"
+		)
+		(pin "29"
+		)
+		(pin "19"
+		)
+		(pin "30"
+		)
+		(pin "33"
+		)
+		(pin "9"
+		)
+		(pin "38"
+		)
+		(pin "40"
+		)
+		(pin "41"
+		)
+		(pin "42"
+		)
+		(pin "43"
+		)
+		(pin "44"
+		)
+		(pin "47"
+		)
+		(pin "48"
+		)
+		(pin "49"
+		)
+		(pin "50"
+		)
+		(pin "51"
+		)
+		(pin "54"
+		)
+		(pin "56"
+		)
+		(pin "18"
+		)
+		(pin "17"
+		)
+		(pin "45"
+		)
+		(pin "46"
+		)
+		(pin "EP"
+		)
+		(pin "1"
+		)
+		(pin "2"
+		)
+		(pin "3"
+		)
+		(pin "32"
+		)
+		(pin "34"
+		)
+		(pin "39"
+		)
+		(pin "20"
+		)
+		(pin "24"
+		)
+		(pin "25"
+		)
+		(pin "36"
+		)
+		(pin "31"
+		)
+		(pin "11"
+		)
+		(pin "12"
+		)
+		(instances
+			(project ""
+				(path "/b5f9ef85-43f0-43d8-a1fd-ed489b1654c1/d652fa9a-929c-40ea-b9c9-ec80a94942ad"
+					(reference "U11")
+					(unit 1)
+				)
+			)
+		)
+	)
 )
