File: hardware/pcb/magnetometer_node_mainboard/schematics/analog_frontend_ina851.kicad_sch (KiCad schematic)
At the start: 0 parts

Commit message: first code for the v1
Parts:
- added C24, C27, C29, C32, C34, C37: 4u7, Capacitor_SMD:C_1206_3216Metric, symbol Device:C
- added C25, C28, C30, C33, C35, C38: 100n, Capacitor_SMD:C_0603_1608Metric, symbol Device:C
- added C26, C31, C36: 220n, Capacitor_SMD:C_0603_1608Metric, symbol Device:C
- added R30, R32, R33, R35, R36, R38: 1k, Resistor_SMD:R_0603_1608Metric, symbol Device:R
- added R31, R34, R37: 48,7, Resistor_SMD:R_1206_3216Metric, symbol Device:R
- added U10, U11, U12: INA851RGTR, Package_DFN_QFN:VQFN-16-1EP_3x3mm_P0.5mm_EP1.68x1.68mm, symbol magnode_symbols:INA851
Connections:
- new net +1V65: U10.13 (VOCM), U11.13 (VOCM), U12.13 (VOCM)
- new net +3V3A: U10.16 (VCLAMP+), U11.16 (VCLAMP+), U12.16 (VCLAMP+)
- new net +5VA: C24.1, C25.1, C27.1, C28.1, C32.1, C33.1, U10.14 (VS+), U11.14 (VS+), U12.14 (VS+)
- new net -5VA: C29.1, C30.1, C34.1, C35.1, C37.1, C38.1, U10.7 (VS-), U11.7 (VS-), U12.7 (VS-)
- new net BR_X+: U10.1 (IN-)
- new net BR_X-: U10.4 (IN+)
- new net BR_Y+: U12.4 (IN+)
- new net BR_Y-: U12.1 (IN-)
- new net BR_Z+: U11.4 (IN+)
- new net BR_Z-: U11.1 (IN-)
- new net GND: C24.2, C25.2, C27.2, C28.2, C29.2, C30.2, C32.2, C33.2, C34.2, C35.2, C37.2, C38.2, U10.17 (TP), U10.5 (VCLAMP-), U11.17 (TP), U11.5 (VCLAMP-), U12.17 (TP), U12.5 (VCLAMP-)
- new net X_INA_OUT+: C26.1, R30.2
- new net X_INA_OUT-: C26.2, R32.2
- new net X_INA_PRE_AAF+: R30.1, U10.11 (OUT+)
- new net X_INA_PRE_AAF-: R32.1, U10.10 (OUT-)
- new net X_RG+: R31.1, U10.2 (RG+)
- new net X_RG-: R31.2, U10.3 (RG-)
- new net Y_INA_OUT+: C36.1, R36.2
- new net Y_INA_OUT-: C36.2, R38.2
- new net Y_INA_PRE_AAF+: R36.1, U12.11 (OUT+)
- new net Y_INA_PRE_AAF-: R38.1, U12.10 (OUT-)
- new net Y_RG+: R37.1, U12.2 (RG+)
- new net Y_RG-: R37.2, U12.3 (RG-)
- new net Z_INA_OUT+: C31.1, R33.2
- new net Z_INA_OUT-: C31.2, R35.2
- new net Z_INA_PRE_AAF+: R33.1, U11.11 (OUT+)
- new net Z_INA_PRE_AAF-: R35.1, U11.10 (OUT-)
- new net Z_RG+: R34.1, U11.2 (RG+)
- new net Z_RG-: R34.2, U11.3 (RG-)
- no-connect marks 0 -> 15
