File: hardware/pcb/magnetometer_node_mainboard/schematics/connectors_io.kicad_sch (KiCad schematic)
At the start: 0 parts

Commit message: first code for the v1
Parts:
- added C42, C47: 1u, Capacitor_SMD:C_0805_2012Metric, symbol Device:C
- added C43, C48: 100n, Capacitor_SMD:C_0603_1608Metric, symbol Device:C
- added C44, C49: 10u, Capacitor_SMD:C_0805_2012Metric, symbol Device:C
- added C45, C50: 10n, Capacitor_SMD:C_0603_1608Metric, symbol Device:C
- added C46, C51: 1n, Capacitor_SMD:C_0603_1608Metric, symbol Device:C
- added D10, D11, D12, D13, D14, D15, D16, D18, D19, D5, D6, D7, D8, D9: H5VUD5BB, Diode_SMD:D_SOD-523, symbol magnode_symbols:H5VUD5BB
- added D17, D4: P6SMB6.8CA, Diode_SMD:D_SMB, symbol Diode:SMAJ6.5CA
- added H1, H2, H3, H4: MountingHole_Pad, MountingHole:MountingHole_3.2mm_M3_DIN965_Pad_TopBottom, symbol Mechanical:MountingHole_Pad
- added J1, J2: USB_C_RECEPTACLE_MOLEX, CONN_201267-0005_MOL, symbol magnode_symbols:USB_C_RECEPTACLE_MOLEX
- added Q11: AO3400A, Package_TO_SOT_SMD:SOT-23, symbol Transistor_FET:AO3400A
- added R39, R46: 470k, Resistor_SMD:R_0603_1608Metric, symbol Device:R
- added R40, R47, R53: 100k, Resistor_SMD:R_0603_1608Metric, symbol Device:R
- added R41, R48: 200k, Resistor_SMD:R_0603_1608Metric, symbol Device:R
- added R42, R49: 39k, Resistor_SMD:R_0603_1608Metric, symbol Device:R
- added R43: ~, Resistor_SMD:R_1206_3216Metric_Pad1.30x1.75mm_HandSolder, symbol Device:R
- added R44: ~, Resistor_THT:R_Axial_DIN0309_L9.0mm_D3.2mm_P15.24mm_Horizontal, symbol Device:R
- added R45, R50: 2k, Resistor_SMD:R_0603_1608Metric, symbol Device:R
- added R51, R52: 100, Resistor_SMD:R_0603_1608Metric, symbol Device:R
- added R54, R55: 5k1, Resistor_SMD:R_0603_1608Metric, symbol Device:R
- added TP2, TP3: TestPoint, TestPoint:TestPoint_THTPad_1.0x1.0mm_Drill0.5mm, symbol Connector:TestPoint
- added U14, U15: TPS25210LRPWR, magnode_footprints:VQFN-HR-10, symbol magnode_symbols:TPS2521xx
Connections:
- new net: J2.B5 (CC2), R54.1
- new net: C51.1, U15.7 (dV/dt)
- new net: R40.2, R42.1, U14.4 (PGTH)
- new net: R39.2, R41.1, TP2.1, U14.1 (EN/ULVO)
- new net: C45.1, U14.10 (ITIMER)
- new net: C46.1, U14.7 (dV/dt)
- new net: R45.1, U14.9 (ILM)
- new net: R46.2, R48.1, TP3.1, U15.1 (EN/ULVO)
- new net: C50.1, U15.10 (ITIMER)
- new net: R50.1, U15.9 (ILM)
- new net: J2.A5 (CC1), R55.1
- new net: R47.2, R49.1, U15.4 (PGTH)
- new net: J2.A1 (GND), J2.A12 (GND), J2.B1 (GND), J2.B12 (GND)
- new net +3V3: U14.3 (PG), U15.3 (PG)
- new net +5V: C44.1, C49.1, R40.1, R47.1, R51.1, U14.6 (OUT), U15.6 (OUT)
- new net +5VBUS_DATA: C42.1, C43.1, D4.2 (A2), J1.A4 (VBUS), J1.A9 (VBUS), J1.B4 (VBUS), J1.B9 (VBUS), R39.1, R43.2, R44.1, U14.5 (IN)
- new net +5VBUS_DEBUG: C47.1, C48.1, D17.2 (A2), J2.A4 (VBUS), J2.A9 (VBUS), J2.B4 (VBUS), J2.B9 (VBUS), R46.1, U15.5 (IN)
- new net CC1: D6.2, J1.A5 (CC1)
- new net CC2: D5.2, J1.B5 (CC2)
- new net D+: D16.2, D19.2, J1.A6 (D+), J1.B6 (D+), J2.A6 (D+), J2.B6 (D+)
- new net D-: D15.2, D18.2, J1.A7 (D-), J1.B7 (D-), J2.A7 (D-), J2.B7 (D-)
- new net EN_KEEPALIVE: R52.1
- new net EN_KEEPALIVE_DRAIN: Q11.3 (D), R51.2
- new net EN_KEEPALIVE_GATE: Q11.1 (G), R52.2, R53.1
- new net GND: C42.2, C43.2, C44.2, C45.2, C46.2, C47.2, C48.2, C49.2, C50.2, C51.2, D10.1, D11.1, D12.1, D13.1, D14.1, D15.1, D16.1, D17.1 (A1), D18.1, D19.1, D4.1 (A1), D5.1, D6.1, D7.1, D8.1, D9.1, H1.1, H2.1, H3.1, H4.1, J1.A1 (GND), J1.A12 (GND), J1.B1 (GND), J1.B12 (GND), Q11.2 (S), R41.2, R42.2, R43.1, R44.2, R45.2, R48.2, R49.2, R50.2, R53.2, R54.2, R55.2, U14.8 (GND), U15.8 (GND)
- new net RX1+: D9.2, J1.B11 (RX1+)
- new net RX1-: D10.2, J1.B10 (RX1-)
- new net RX2+: D7.2, J1.A11 (RX2+)
- new net RX2-: D8.2, J1.A10 (RX2-)
- new net TX1+: D14.2, J1.A2 (TX1+)
- new net TX1-: D13.2, J1.A3 (TX1-)
- new net TX2+: D12.2, J1.B2 (TX2+)
- new net TX2-: D11.2, J1.B3 (TX2-)
- no-connect marks 0 -> 14
Other:
- note added: "Sending a pulse of current through a 100 ohm resistor to keep the battery awake"
