File: hardware/pcb/magnetometer_node_mainboard/schematics/pwr_3v3a.kicad_sch (KiCad schematic)
At the start: 1 part, among them U9 XC6206PxxxMR

Commit message: first code for the v1
Parts:
- removed U9: XC6206PxxxMR, Package_TO_SOT_SMD:SOT-23-3, symbol Regulator_Linear:XC6206PxxxMR
- added C81, C84: 4u7, Capacitor_SMD:C_1206_3216Metric, symbol Device:C
- added C82, C83: 100n, Capacitor_SMD:C_0603_1608Metric, symbol Device:C
- added FB1: FerriteBead, symbol Device:FerriteBead
- added U19: TPS7A2033PDBVR, Package_TO_SOT_SMD:SOT-23-5, symbol Regulator_Linear:TPS7A20xxxDQN
Connections:
- new net +3V3A: C83.1, C84.1, U19.1 (OUT)
- new net +5V: FB1.1
- new net EN_LDO_3V3: U19.3 (EN)
- new net GND: C81.2, C82.2, C83.2, C84.2, U19.2 (GND), U19.5 (Pad)
- new net LDO_3V3_IN: C81.1, C82.1, FB1.2, U19.4 (IN)
