File: hardware/pcb/magnetometer_node_mainboard/schematics/pwr_3v3d.kicad_sch (KiCad schematic)
At the start: 0 parts

Commit message: first code for the v1
Parts:
- added C69: 1u, Capacitor_SMD:C_0805_2012Metric, symbol Device:C
- added C70: 100n, Capacitor_SMD:C_0603_1608Metric, symbol Device:C
- added C71: 10u, Capacitor_SMD:C_0805_2012Metric, symbol Device:C
- added C72, C73: 22u, Capacitor_SMD:C_1206_3216Metric, symbol Device:C
- added C74: 47u, Capacitor_SMD:C_1206_3216Metric, symbol Device:C
- added C75: 10p, Capacitor_SMD:C_0603_1608Metric, symbol Device:C
- added C76: 4n7, Capacitor_SMD:C_0603_1608Metric, symbol Device:C
- added C77, C78: 10n, Capacitor_SMD:C_0603_1608Metric, symbol Device:C
- added C79: 1n, Capacitor_SMD:C_0603_1608Metric, symbol Device:C
- added C80: 470mF, magnode_footprints:C_Radial_D8.0mm_P11.50mm, symbol Device:C
- added D20, D21, D22: SS34, Diode_SMD:D_SMA, symbol Device:D_Schottky
- added L3: 10u, Capacitor_SMD:C_0805_2012Metric, symbol Device:L
- added R68: 470k, Resistor_SMD:R_0603_1608Metric, symbol Device:R
- added R69: 100k, Resistor_SMD:R_0603_1608Metric, symbol Device:R
- added R70: 200k, Resistor_SMD:R_0603_1608Metric, symbol Device:R
- added R71: 39k, Resistor_SMD:R_0603_1608Metric, symbol Device:R
- added R72: 75k, Resistor_SMD:R_0603_1608Metric, symbol Device:R
- added R73: 10k, Resistor_SMD:R_0603_1608Metric, symbol Device:R
- added R74: 2k, Resistor_SMD:R_0603_1608Metric, symbol Device:R
- added R75: 24k, Resistor_SMD:R_0603_1608Metric, symbol Device:R
- added R76: 47, Resistor_THT:R_Axial_DIN0309_L9.0mm_D3.2mm_P12.70mm_Horizontal, symbol Device:R
- added TP4: TestPoint, TestPoint:TestPoint_THTPad_1.0x1.0mm_Drill0.5mm, symbol Connector:TestPoint
- added U17: TPS25210LRPWR, magnode_footprints:VQFN-HR-10, symbol magnode_symbols:TPS2521xx
- added U18: TPS54331DR, Package_SO:SOIC-8_3.9x4.9mm_P1.27mm, symbol magnode_symbols:TPS54331
Connections:
- new net +3V3: C74.1, L3.2, R72.1, U17.3 (PG)
- new net +5V: C69.1, C70.1, D21.2 (A), R68.1, U17.5 (IN)
- new net 3V3D_EFUSE_DVDT: C79.1, U17.7 (dV/dt)
- new net 3V3D_EFUSE_EN_ULVO: R68.2, R70.1, TP4.1, U17.1 (EN/ULVO)
- new net 3V3D_EFUSE_ILM: R74.1, U17.9 (ILM)
- new net 3V3D_EFUSE_ITIMER: C78.1, U17.10 (ITIMER)
- new net 3V3D_EFUSE_PGTH: R69.2, R71.1, U17.4 (PGTH)
- new net 5V_CAP_CHG: D21.1 (K), R76.1
- new net 5V_HOLDUP: C71.1, C73.1, D22.1 (K), R69.1, U17.6 (OUT), U18.2 (VIN), U18.3 (EN)
- new net 5V_SUPERCAP: C80.1, D22.2 (A), R76.2
- new net GND: C69.2, C70.2, C71.2, C73.2, C74.2, C75.2, C76.2, C77.2, C78.2, C79.2, C80.2, D20.2 (A), R70.2, R71.2, R74.2, R75.2, U17.8 (GND), U18.7 (GND)
- new net STPD_3V3_BOOT: C72.1, U18.1 (BOOT)
- new net STPD_3V3_COMP: C75.1, R73.1, U18.6 (COMP)
- new net STPD_3V3_COMP_F: C76.1, R73.2
- new net STPD_3V3_PH: C72.2, D20.1 (K), L3.1, U18.8 (PH)
- new net STPD_3V3_SS: C77.1, U18.4 (SS)
- new net STPD_3V3_VSENS: R72.2, R75.1, U18.5 (VSENSE)
- no-connect marks 0 -> 1
