File: hardware/pcb/magnetometer_node_mainboard/schematics/pwr_opamp_4v5_neg5.kicad_sch (KiCad schematic)
At the start: 1 part, among them U10 TPS7A2045PDBVR

Commit message: first code for the v1
Parts:
- removed U10: TPS7A2045PDBVR, Package_SON:Texas_X2SON-4_1x1mm_P0.65mm, symbol Regulator_Linear:TPS7A20xxxDQN
- added C100, C97, C98, C99: 4u7, Capacitor_SMD:C_1206_3216Metric, symbol Device:C
- added C101: 4n7, Capacitor_SMD:C_0603_1608Metric, symbol Device:C
- added C102, C89, C94: 100n, Capacitor_SMD:C_0603_1608Metric, symbol Device:C
- added C85, C87, C92, C93: 10u, Capacitor_SMD:C_0805_2012Metric, symbol Device:C
- added C86, C88, C95: 10n, Capacitor_SMD:C_0603_1608Metric, symbol Device:C
- added C90: 220n, Capacitor_SMD:C_0603_1608Metric, symbol Device:C
- added C91: 10p, Capacitor_SMD:C_0603_1608Metric, symbol Device:C
- added C96: 47u, Capacitor_SMD:C_1206_3216Metric, symbol Device:C
- added D23: SS34, Diode_SMD:D_SMA, symbol Device:D_Schottky
- added L4: 10u, Capacitor_SMD:C_0805_2012Metric, symbol Device:L
- added R77: 39k, Resistor_SMD:R_0603_1608Metric, symbol Device:R
- added R78: 12k, Resistor_SMD:R_0603_1608Metric, symbol Device:R
- added R79, R82, R84: 100k, Resistor_SMD:R_0603_1608Metric, symbol Device:R
- added R80: 10, Resistor_SMD:R_0603_1608Metric, symbol Device:R
- added R81: 510k, Resistor_SMD:R_0603_1608Metric, symbol Device:R
- added R83: 330k, Resistor_SMD:R_0603_1608Metric, symbol Device:R
- added U20: TPS7A4901DGNR, Package_SO:HVSSOP-8-1EP_3x3mm_P0.65mm_EP1.57x1.89mm, symbol magnode_symbols:TPS7A4901
- added U21: TPS63700DRCR, Package_SON:VSON-10-1EP_3x3mm_P0.5mm_EP1.2x2mm, symbol magnode_symbols:TPS63700
- added U22: TPS7A3301RGWR, Package_DFN_QFN:Texas_RGW0020A_VQFN-20-1EP_5x5mm_P0.65mm_EP3.15x3.15mm_ThermalVias, symbol Regulator_Linear:TPS7A3301RGW
Connections:
- new net +10V: C85.1, U20.5 (EN), U20.8 (IN)
- new net +5V: C92.1, R80.2, U21.5 (IN)
- new net +5VA: C86.1, C87.1, R77.1, U20.1 (OUT)
- new net -5VA: C95.1, C96.1, R83.1, U22.1 (OUT), U22.20 (OUT)
- new net EN_INV_-5V: U21.4 (EN)
- new net GND: C100.2, C101.2, C102.2, C85.2, C87.2, C88.2, C89.2, C90.2, C92.2, C93.2, C94.2, C96.2, C97.2, C98.2, C99.2, L4.2, R78.2, R84.2, U20.3 (NC), U20.4 (GND), U20.9 (PwPd), U21.11 (PowerPAD), U21.2 (GND), U21.7 (PSGND), U22.21 (EP), U22.7 (GND)
- new net INV_N5V5_COMP: C101.1, U21.1 (COMP)
- new net INV_N5V5_FB: C91.1, R79.2, R81.1, U21.9 (FB)
- new net INV_N5V5_FF: C91.2, R82.1
- new net INV_N5V5_SW: D23.1 (K), L4.1, U21.6 (SW)
- new net INV_N5V5_VIN: C89.1, R80.1, U21.3 (VIN)
- new net INV_N5V5_VREF: C90.1, R79.1, U21.10 (VREF)
- new net LDO_N5V_FB: C95.2, R83.2, R84.1, U22.3 (FB)
- new net LDO_N5V_NR: C102.1, U22.14 (NR/SS)
- new net LDO_P5V_FB: C86.2, R77.2, R78.1, U20.2 (FB)
- new net LDO_P5V_NR: C88.1, U20.6 (NR/SS)
- new net N5V5_PRE_N5VA: C100.1, C93.1, C94.1, C97.1, C98.1, C99.1, D23.2 (A), R81.2, R82.2, U21.8 (OUT), U22.13 (EN), U22.15 (IN), U22.16 (IN)
- no-connect marks 0 -> 1
Other:
- note removed: "Pins sont pas aux bon entroits"
