File: hardware/pcb/magnetometer_node_mainboard/schematics/sensor_hmc100x_3axis.kicad_sch (KiCad schematic)
At the start: 0 parts

Commit message: Schematic sensor stage done
Parts:
- added U1: HMC1001-RC, SIP8_HMC1001_HNW, symbol magnode_symbols:HMC1001-RC
- added U2: HMC1002-TR, SOIC20_HNW, symbol magnode_symbols:HMC1002-TR
Connections:
- new net +9VA: U1.7 (VBRIDGE), U2.11 (VBRIDGE(B)), U2.4 (VBRIDGE(A))
- new net BR_X+: U2.2 (OUT+(A))
- new net BR_X-: U2.5 (OUT-(A))
- new net BR_Y+: U2.9 (OUT+(B))
- new net BR_Y-: U2.12 (OUT-(B))
- new net BR_Z+: U1.8 (OUT-)
- new net BR_Z-: U1.5 (OUT+)
- new net GND: U1.4 (GND), U1.6 (OFFSET-), U2.1 (GND1(A)), U2.10 (OFFSET-(B)), U2.13 (GND2(B)), U2.18 (GND_PLN), U2.3 (OFFSET-(A)), U2.6 (GND2(A)), U2.7 (S/R-(B)), U2.8 (GND1(B))
- new net OFFSET_X+: U2.17 (OFFSET(+A))
- new net OFFSET_Y+: U2.15 (OFFSET+(B))
- new net OFFSET_Z+: U1.2 (OFFSET+)
- new net SETRESET_AFTER_1001: U1.3 (S/R-), U2.16 (S/R+(A))
- new net SETRESET_AFTER_1002A: U2.14 (S/R+(B)), U2.20 (S/R-(A))
- new net SETRESET_STRAP: U1.1 (S/R+)
Other:
- note added: "HMC1001 = Z HMC1002A = X HMC1002B = Y"

Commit message: first code for the v1
Parts:
- U1: footprint SIP8_HMC1001_HNW -> magnode_footprints:SIP8_HMC1001_HNW
- U2: footprint SOIC20_HNW -> magnode_footprints:SOIC20_HNW
Other:
- note added: "bypass cap"
