File: hardware/pcb/magnetometer_node_mainboard/magnetometer_node_mainboard.kicad_pcb (KiCad board)
At the start: 2 copper layers, 19 parts, among them Q1 D882, Q10 B772, Q2 B772, Q3 DMC3028LSD, Q4 D882, Q5 D882, Q6 B772, Q7 D882, Q8 B772, Q9 D882, U10 TPS7A20xxxDQN, U3 MCP4728, U5 LT3042xMSE, U6 TPS61040DBV, U7 ESP32-S3-WROOM-1, U8 AD7779, U9 XC6206PxxxMR

Commit message: esp32_testing
Parts:
- added U11: DAN-F10N, magnode_footprints:u-blox_DAN-F10N_LCC-56_20x20mm, F.Cu at (76.0, 70.8)
- U10: value TPS7A20xxxDQN -> TPS7A2045PDBVR
- moved U7 14.1 mm to (212.5, 44.8), turned to -90 degrees

Commit message: first code for the v1
Parts:
- added C1: 10u, Capacitor_SMD:C_0805_2012Metric, F.Cu at (165.1, 130.0)
- added C10: 10u, Capacitor_SMD:C_0805_2012Metric, F.Cu at (170.9, 132.0)
- added C100: 4u7, Capacitor_SMD:C_1206_3216Metric, F.Cu at (166.3, 65.3)
- added C101: 4n7, Capacitor_SMD:C_0603_1608Metric, F.Cu at (175.2, 54.0)
- added C102: 100n, Capacitor_SMD:C_0603_1608Metric, F.Cu at (175.2, 56.5)
- added C103: 1u, Capacitor_SMD:C_0805_2012Metric, F.Cu at (206.3, 61.5)
- added C104: 100n, Capacitor_SMD:C_0603_1608Metric, F.Cu at (241.2, 63.5)
- added C105: 100n, Capacitor_SMD:C_0603_1608Metric, F.Cu at (203.2, 78.5)
- added C106: 10u, Capacitor_SMD:C_0805_2012Metric, F.Cu at (206.3, 64.5)
- added C107: 100n, Capacitor_SMD:C_0603_1608Metric, F.Cu at (203.2, 81.0)
- added C108: 1u, Capacitor_SMD:C_0805_2012Metric, F.Cu at (206.3, 67.5)
- added C109: 100n, Capacitor_SMD:C_0603_1608Metric, F.Cu at (203.2, 83.5)
- added C11: 10u, Capacitor_SMD:C_0805_2012Metric, F.Cu at (170.9, 135.0)
- added C110: 100n, Capacitor_SMD:C_0603_1608Metric, F.Cu at (203.2, 86.0)
- added C111: 1u, Capacitor_SMD:C_0805_2012Metric, F.Cu at (206.3, 70.6)
- added C112: 18p, Capacitor_SMD:C_0603_1608Metric, F.Cu at (245.0, 69.0)
- added C113: 18p, Capacitor_SMD:C_0603_1608Metric, F.Cu at (245.2, 56.0)
- added C12: 10u, Capacitor_SMD:C_0805_2012Metric, F.Cu at (170.9, 138.0)
- added C13: 10u, Capacitor_SMD:C_0805_2012Metric, F.Cu at (170.9, 141.1)
- added C14: 4u7, Capacitor_SMD:C_1206_3216Metric, F.Cu at (63.0, 113.7)
- added C15: 22p, Capacitor_SMD:C_0603_1608Metric, F.Cu at (181.3, 116.0)
- added C16: 1u, Capacitor_SMD:C_0805_2012Metric, F.Cu at (191.2, 116.2)
- added C17: 10u, Capacitor_SMD:C_0805_2012Metric, F.Cu at (68.0, 116.5)
- added C18: 100n, Capacitor_SMD:C_0603_1608Metric, F.Cu at (58.2, 115.7)
- added C19: 4u7, Capacitor_SMD:C_1206_3216Metric, F.Cu at (63.0, 117.0)
- added C2: 10u, Capacitor_SMD:C_0805_2012Metric, F.Cu at (165.1, 133.0)
- added C20: 4u7, Capacitor_SMD:C_1206_3216Metric, F.Cu at (186.1, 123.1)
- added C21: 100n, Capacitor_SMD:C_0603_1608Metric, F.Cu at (210.2, 101.5)
- added C22: 10u, Capacitor_SMD:C_0805_2012Metric, F.Cu at (214.4, 109.9)
- added C23: 100n, Capacitor_SMD:C_0603_1608Metric, F.Cu at (210.2, 104.0)
- added C24: 4u7, Capacitor_SMD:C_1206_3216Metric, F.Cu at (128.3, 113.9)
- added C25: 100n, Capacitor_SMD:C_0603_1608Metric, F.Cu at (147.0, 130.5)
- added C26: 220n, Capacitor_SMD:C_0603_1608Metric, F.Cu at (147.0, 133.0)
- added C27: 4u7, Capacitor_SMD:C_1206_3216Metric, F.Cu at (128.3, 117.3)
- added C28: 100n, Capacitor_SMD:C_0603_1608Metric, F.Cu at (157.2, 125.0)
- added C29: 4u7, Capacitor_SMD:C_1206_3216Metric, F.Cu at (128.3, 120.6)
- added C3: 4u7, Capacitor_SMD:C_1206_3216Metric, F.Cu at (113.6, 140.2)
- added C30: 100n, Capacitor_SMD:C_0603_1608Metric, F.Cu at (141.1, 117.2)
- added C31: 220n, Capacitor_SMD:C_0603_1608Metric, F.Cu at (141.1, 119.8)
- added C32: 4u7, Capacitor_SMD:C_1206_3216Metric, F.Cu at (128.3, 124.0)
- added C33: 100n, Capacitor_SMD:C_0603_1608Metric, F.Cu at (141.1, 122.3)
- added C34: 4u7, Capacitor_SMD:C_1206_3216Metric, F.Cu at (128.3, 127.3)
- added C35: 100n, Capacitor_SMD:C_0603_1608Metric, F.Cu at (151.0, 130.5)
- added C36: 220n, Capacitor_SMD:C_0603_1608Metric, F.Cu at (151.0, 133.0)
- added C37: 4u7, Capacitor_SMD:C_1206_3216Metric, F.Cu at (128.3, 130.7)
- added C38: 100n, Capacitor_SMD:C_0603_1608Metric, F.Cu at (161.2, 125.0)
- added C39: 100n, Capacitor_SMD:C_0603_1608Metric, F.Cu at (198.7, 113.1)
- added C4: 220n, Capacitor_SMD:C_0603_1608Metric, F.Cu at (132.8, 132.5)
- added C40: 100n, Capacitor_SMD:C_0603_1608Metric, F.Cu at (198.7, 115.6)
- added C41: 10u, Capacitor_SMD:C_0805_2012Metric, F.Cu at (202.9, 117.4)
- added C42: 1u, Capacitor_SMD:C_0805_2012Metric, F.Cu at (211.0, 94.0)
- added C43: 100n, Capacitor_SMD:C_0603_1608Metric, F.Cu at (126.2, 46.5)
- added C44: 10u, Capacitor_SMD:C_0805_2012Metric, F.Cu at (172.0, 78.0)
- added C45: 10n, Capacitor_SMD:C_0603_1608Metric, F.Cu at (126.2, 49.0)
- added C46: 1n, Capacitor_SMD:C_0603_1608Metric, F.Cu at (126.2, 51.5)
- added C47: 1u, Capacitor_SMD:C_0805_2012Metric, F.Cu at (172.0, 81.0)
- added C48: 100n, Capacitor_SMD:C_0603_1608Metric, F.Cu at (126.2, 54.0)
- added C49: 10u, Capacitor_SMD:C_0805_2012Metric, F.Cu at (172.0, 84.0)
- added C5: 1n, Capacitor_SMD:C_0603_1608Metric, F.Cu at (132.8, 135.0)
- added C50: 10n, Capacitor_SMD:C_0603_1608Metric, F.Cu at (178.2, 45.0)
- added C51: 1n, Capacitor_SMD:C_0603_1608Metric, F.Cu at (148.0, 43.1)
- added C52: 10u, Capacitor_SMD:C_0805_2012Metric, F.Cu at (177.4, 88.7)
- added C53: 100n, Capacitor_SMD:C_0603_1608Metric, F.Cu at (161.2, 88.5)
- added C54: 100n, Capacitor_SMD:C_0603_1608Metric, F.Cu at (161.2, 91.0)
- added C55: 100n, Capacitor_SMD:C_0603_1608Metric, F.Cu at (161.2, 93.5)
- added C56: 100n, Capacitor_SMD:C_0603_1608Metric, F.Cu at (161.2, 96.0)
- added C57: 100n, Capacitor_SMD:C_0603_1608Metric, F.Cu at (161.2, 98.5)
- added C58: 100n, Capacitor_SMD:C_0603_1608Metric, F.Cu at (161.2, 101.0)
- added C59: 100n, Capacitor_SMD:C_0603_1608Metric, F.Cu at (165.2, 88.5)
- added C6: 10n, Capacitor_SMD:C_0603_1608Metric, F.Cu at (132.8, 137.5)
- added C60: 100n, Capacitor_SMD:C_0603_1608Metric, F.Cu at (165.2, 91.0)
- added C61: 10u, Capacitor_SMD:C_0805_2012Metric, F.Cu at (177.4, 91.8)
- added C62: 220n, Capacitor_SMD:C_0603_1608Metric, F.Cu at (165.2, 93.5)
- added C63: 100n, Capacitor_SMD:C_0603_1608Metric, F.Cu at (165.2, 96.0)
- added C64: 47u, Capacitor_SMD:C_1206_3216Metric, F.Cu at (162.0, 104.0)
- added C65: 100n, Capacitor_SMD:C_0603_1608Metric, F.Cu at (165.2, 98.5)
- added C66: 1u, Capacitor_SMD:C_0805_2012Metric, F.Cu at (177.4, 94.8)
- added C67: 1u, Capacitor_SMD:C_0805_2012Metric, F.Cu at (177.4, 97.8)
- added C68: 1u, Capacitor_SMD:C_0805_2012Metric, F.Cu at (177.4, 100.8)
- added C69: 1u, Capacitor_SMD:C_0805_2012Metric, F.Cu at (223.0, 87.0)
- added C7: 10u, Capacitor_SMD:C_0805_2012Metric, F.Cu at (170.9, 126.0)
- added C70: 100n, Capacitor_SMD:C_0603_1608Metric, F.Cu at (256.9, 58.7)
- added C71: 10u, Capacitor_SMD:C_0805_2012Metric, F.Cu at (269.2, 77.8)
- added C72: 22u, Capacitor_SMD:C_1206_3216Metric, F.Cu at (187.4, 79.1)
- added C73: 22u, Capacitor_SMD:C_1206_3216Metric, F.Cu at (187.4, 82.5)
- added C74: 47u, Capacitor_SMD:C_1206_3216Metric, F.Cu at (187.4, 85.8)
- added C75: 10p, Capacitor_SMD:C_0603_1608Metric, F.Cu at (182.6, 78.7)
- added C76: 4n7, Capacitor_SMD:C_0603_1608Metric, F.Cu at (182.6, 81.2)
- added C77: 10n, Capacitor_SMD:C_0603_1608Metric, F.Cu at (182.6, 83.7)
- added C78: 10n, Capacitor_SMD:C_0603_1608Metric, F.Cu at (256.9, 61.2)
- added C79: 1n, Capacitor_SMD:C_0603_1608Metric, F.Cu at (256.9, 63.8)
- added C8: 100n, Capacitor_SMD:C_0603_1608Metric, F.Cu at (96.0, 117.0)
- added C80: 470mF, magnode_footprints:C_Radial_D8.0mm_P11.50mm, F.Cu at (229.0, 107.0)
- added C81: 4u7, Capacitor_SMD:C_1206_3216Metric, F.Cu at (187.6, 100.3)
- added C82: 100n, Capacitor_SMD:C_0603_1608Metric, F.Cu at (192.4, 104.5)
- added C83: 100n, Capacitor_SMD:C_0603_1608Metric, F.Cu at (192.4, 107.0)
- added C84: 4u7, Capacitor_SMD:C_1206_3216Metric, F.Cu at (187.6, 103.6)
- added C85: 10u, Capacitor_SMD:C_0805_2012Metric, F.Cu at (183.4, 51.7)
- added C86: 10n, Capacitor_SMD:C_0603_1608Metric, F.Cu at (171.2, 51.5)
- added C87: 10u, Capacitor_SMD:C_0805_2012Metric, F.Cu at (183.4, 54.8)
- added C88: 10n, Capacitor_SMD:C_0603_1608Metric, F.Cu at (171.2, 54.0)
- added C89: 100n, Capacitor_SMD:C_0603_1608Metric, F.Cu at (171.2, 56.5)
- added C9: 10u, Capacitor_SMD:C_0805_2012Metric, F.Cu at (170.9, 129.0)
- added C90: 220n, Capacitor_SMD:C_0603_1608Metric, F.Cu at (171.2, 59.0)
- added C91: 10p, Capacitor_SMD:C_0603_1608Metric, F.Cu at (171.2, 61.5)
- added C92: 10u, Capacitor_SMD:C_0805_2012Metric, F.Cu at (183.4, 57.8)
- added C93: 10u, Capacitor_SMD:C_0805_2012Metric, F.Cu at (183.4, 60.8)
- added C94: 100n, Capacitor_SMD:C_0603_1608Metric, F.Cu at (171.2, 64.0)
- added C95: 10n, Capacitor_SMD:C_0603_1608Metric, F.Cu at (175.2, 51.5)
- added C96: 100n, Capacitor_SMD:C_0603_1608Metric, F.Cu at (241.0, 69.0)
- added C96: 47u, Capacitor_SMD:C_1206_3216Metric, F.Cu at (166.3, 51.9)
- added C97: 100n, Capacitor_SMD:C_0603_1608Metric, F.Cu at (241.2, 56.0)
- added C97: 4u7, Capacitor_SMD:C_1206_3216Metric, F.Cu at (166.3, 55.3)
- added C98: 4u7, Capacitor_SMD:C_1206_3216Metric, F.Cu at (166.3, 58.6)
- added C98: 100n, Capacitor_SMD:C_0603_1608Metric, F.Cu at (241.2, 58.5)
- added C99: 100n, Capacitor_SMD:C_0603_1608Metric, F.Cu at (241.2, 61.0)
- added C99: 4u7, Capacitor_SMD:C_1206_3216Metric, F.Cu at (166.3, 62.0)
- added D1: SS34, Diode_SMD:D_SMA, F.Cu at (154.0, 139.0)
- added D10: H5VUD5BB, Diode_SMD:D_SOD-523, F.Cu at (203.4, 93.7)
- added D11: H5VUD5BB, Diode_SMD:D_SOD-523, F.Cu at (164.4, 77.2)
- added D12: H5VUD5BB, Diode_SMD:D_SOD-523, F.Cu at (164.4, 79.6)
- added D13: H5VUD5BB, Diode_SMD:D_SOD-523, F.Cu at (164.4, 82.0)
- added D14: H5VUD5BB, Diode_SMD:D_SOD-523, F.Cu at (164.4, 84.5)
- added D15: H5VUD5BB, Diode_SMD:D_SOD-523, F.Cu at (207.0, 93.7)
- added D16: H5VUD5BB, Diode_SMD:D_SOD-523, F.Cu at (168.0, 77.2)
- added D17: P6SMB6.8CA, Diode_SMD:D_SMB, F.Cu at (170.0, 44.0)
- added D18: H5VUD5BB, Diode_SMD:D_SOD-523, F.Cu at (168.0, 79.6)
- added D19: H5VUD5BB, Diode_SMD:D_SOD-523, F.Cu at (168.0, 82.0)
- added D20: SS34, Diode_SMD:D_SMA, F.Cu at (194.3, 86.3)
- added D21: SS34, Diode_SMD:D_SMA, F.Cu at (243.0, 103.0)
- added D22: SS34, Diode_SMD:D_SMA, F.Cu at (227.0, 113.0)
- added D23: SS34, Diode_SMD:D_SMA, F.Cu at (191.0, 56.0)
- added D3: SS34, Diode_SMD:D_SMA, F.Cu at (198.0, 122.0)
- added D4: P6SMB6.8CA, Diode_SMD:D_SMB, F.Cu at (118.0, 49.0)
- added D5: H5VUD5BB, Diode_SMD:D_SOD-523, F.Cu at (199.8, 93.7)
- added D6: H5VUD5BB, Diode_SMD:D_SOD-523, F.Cu at (160.8, 77.2)
- added D7: H5VUD5BB, Diode_SMD:D_SOD-523, F.Cu at (160.8, 79.6)
- added D8: H5VUD5BB, Diode_SMD:D_SOD-523, F.Cu at (160.8, 82.0)
- added D9: H5VUD5BB, Diode_SMD:D_SOD-523, F.Cu at (160.8, 84.5)
- added H1, H5: MountingHole_Pad, MountingHole:MountingHole_3.2mm_M3_DIN965_Pad_TopBottom, F.Cu at (99.0, 47.0)
- added H2, H6: MountingHole_Pad, MountingHole:MountingHole_3.2mm_M3_DIN965_Pad_TopBottom, F.Cu at (199.0, 47.0)
- added H3, H7: MountingHole_Pad, MountingHole:MountingHole_3.2mm_M3_DIN965_Pad_TopBottom, F.Cu at (199.0, 138.0)
- added H4, H8: MountingHole_Pad, MountingHole:MountingHole_3.2mm_M3_DIN965_Pad_TopBottom, F.Cu at (99.0, 138.0)
- added H5: MountingHole_Pad, MountingHole:MountingHole_3.2mm_M3_DIN965_Pad_TopBottom, F.Cu at (70.0, 60.5)
- added H6: MountingHole_Pad, MountingHole:MountingHole_3.2mm_M3_DIN965_Pad_TopBottom, F.Cu at (70.0, 124.5)
- added H7: MountingHole_Pad, MountingHole:MountingHole_3.2mm_M3_DIN965_Pad_TopBottom, F.Cu at (150.0, 60.5)
- added H8: MountingHole_Pad, MountingHole:MountingHole_3.2mm_M3_DIN965_Pad_TopBottom, F.Cu at (150.0, 124.5)
- added J1: USB_C_RECEPTACLE_MOLEX, magnode_footprints:CONN_201267-0005_MOL, F.Cu at (231.7, 54.1)
- added J2: USB_C_RECEPTACLE_MOLEX, magnode_footprints:CONN_201267-0005_MOL, F.Cu at (244.0, 95.0)
- added J3: Micro_SD_CARD, magnode_footprints:CONN_503398-1892_MOL, F.Cu at (240.0, 80.0)
- added L1: 10u, Capacitor_SMD:C_0805_2012Metric, F.Cu at (165.1, 136.0)
- added L2: 10u, Capacitor_SMD:C_0805_2012Metric, F.Cu at (191.2, 122.2)
- added L3: 10u, Capacitor_SMD:C_0805_2012Metric, F.Cu at (192.5, 90.1)
- added L4: 10u, Capacitor_SMD:C_0805_2012Metric, F.Cu at (183.4, 63.8)
- added Q11: AO3400A, Package_TO_SOT_SMD:SOT-23, F.Cu at (234.0, 69.0)
- added Q12: AO3401A, Package_TO_SOT_SMD:SOT-23, F.Cu at (210.9, 62.4)
- added Q13: AO3400A, Package_TO_SOT_SMD:SOT-23, F.Cu at (210.9, 67.0)
- added R1: 220, Resistor_SMD:R_0805_2012Metric, F.Cu at (165.0, 139.0)
- added R10: 100, Resistor_SMD:R_0603_1608Metric, F.Cu at (96.0, 122.0)
- added R100: 100k, Resistor_SMD:R_0603_1608Metric, F.Cu at (211.2, 86.0)
- added R101: 100k, Resistor_SMD:R_0603_1608Metric, F.Cu at (220.2, 55.0)
- added R102: 680, Resistor_SMD:R_0603_1608Metric, F.Cu at (220.2, 57.5)
- added R103: 100k, Resistor_SMD:R_0603_1608Metric, F.Cu at (220.2, 60.0)
- added R104: 100k, Resistor_SMD:R_0603_1608Metric, F.Cu at (222.0, 50.0)
- added R105: 900k, Resistor_SMD:R_0603_1608Metric, F.Cu at (191.0, 72.0)
- added R11: 20, Resistor_SMD:R_1206_3216Metric, F.Cu at (101.0, 125.0)
- added R12: 100, Resistor_SMD:R_0603_1608Metric, F.Cu at (96.0, 124.5)
- added R13: 100, Resistor_SMD:R_0603_1608Metric, F.Cu at (174.9, 124.0)
- added R14: 20, Resistor_SMD:R_1206_3216Metric, F.Cu at (101.0, 121.0)
- added R15: 100, Resistor_SMD:R_0603_1608Metric, F.Cu at (174.9, 126.5)
- added R16: 100, Resistor_SMD:R_0603_1608Metric, F.Cu at (174.9, 129.0)
- added R17: 20, Resistor_SMD:R_1206_3216Metric, F.Cu at (121.0, 130.0)
- added R19: 2k, Resistor_SMD:R_0603_1608Metric, F.Cu at (58.2, 120.8)
- added R2: 1k, Resistor_SMD:R_0603_1608Metric, F.Cu at (132.8, 140.0)
- added R20: 200k, Resistor_SMD:R_0603_1608Metric, F.Cu at (181.3, 126.0)
- added R21: 90k9, Resistor_SMD:R_1206_3216Metric, F.Cu at (63.0, 123.7)
- added R22: 100k, Resistor_SMD:R_0603_1608Metric, F.Cu at (181.3, 128.5)
- added R23: 10k, Resistor_SMD:R_0603_1608Metric, F.Cu at (210.2, 106.5)
- added R24: 10k, Resistor_SMD:R_0603_1608Metric, F.Cu at (210.2, 109.0)
- added R25: 22, Resistor_SMD:R_0603_1608Metric, F.Cu at (210.2, 111.5)
- added R26: 22, Resistor_SMD:R_0603_1608Metric, F.Cu at (210.2, 114.0)
- added R27: 22, Resistor_SMD:R_0603_1608Metric, F.Cu at (210.2, 116.5)
- added R28: 10k, Resistor_SMD:R_0603_1608Metric, F.Cu at (210.2, 119.0)
- added R29: 10k, Resistor_SMD:R_0603_1608Metric, F.Cu at (210.2, 121.5)
- added R3: 49k9, Resistor_SMD:R_0603_1608Metric, F.Cu at (132.8, 142.5)
- added R30: 1k, Resistor_SMD:R_0603_1608Metric, F.Cu at (145.1, 117.2)
- added R31: 48,7, Resistor_SMD:R_1206_3216Metric, F.Cu at (141.9, 125.2)
- added R32: 1k, Resistor_SMD:R_0603_1608Metric, F.Cu at (145.1, 119.8)
- added R33: 1k, Resistor_SMD:R_0603_1608Metric, F.Cu at (145.1, 122.3)
- added R34: 48,7, Resistor_SMD:R_1206_3216Metric, F.Cu at (141.9, 128.5)
- added R35: 1k, Resistor_SMD:R_0603_1608Metric, F.Cu at (155.0, 130.5)
- added R36: 1k, Resistor_SMD:R_0603_1608Metric, F.Cu at (155.0, 133.0)
- added R37: 48,7, Resistor_SMD:R_1206_3216Metric, F.Cu at (141.9, 131.8)
- added R38: 1k, Resistor_SMD:R_0603_1608Metric, F.Cu at (165.2, 125.0)
- added R39: 470k, Resistor_SMD:R_0603_1608Metric, F.Cu at (148.0, 45.6)
- added R4: 1k, Resistor_SMD:R_0603_1608Metric, F.Cu at (136.8, 132.5)
- added R40: 100k, Resistor_SMD:R_0603_1608Metric, F.Cu at (130.2, 46.5)
- added R41: 200k, Resistor_SMD:R_0603_1608Metric, F.Cu at (130.2, 49.0)
- added R42: 39k, Resistor_SMD:R_0603_1608Metric, F.Cu at (130.2, 51.5)
- added R43: ~, Resistor_SMD:R_1206_3216Metric_Pad1.30x1.75mm_HandSolder, F.Cu at (177.2, 83.4)
- added R44: ~, Resistor_THT:R_Axial_DIN0309_L9.0mm_D3.2mm_P15.24mm_Horizontal, F.Cu at (212.0, 58.0)
- added R45: 2k, Resistor_SMD:R_0603_1608Metric, F.Cu at (130.2, 54.0)
- added R46: 470k, Resistor_SMD:R_0603_1608Metric, F.Cu at (182.2, 45.0)
- added R47: 100k, Resistor_SMD:R_0603_1608Metric, F.Cu at (152.0, 43.1)
- added R48: 200k, Resistor_SMD:R_0603_1608Metric, F.Cu at (152.0, 45.6)
- added R49: 39k, Resistor_SMD:R_0603_1608Metric, F.Cu at (134.2, 46.5)
- added R5: 100k, Resistor_SMD:R_0603_1608Metric, F.Cu at (136.8, 135.0)
- added R50: 2k, Resistor_SMD:R_0603_1608Metric, F.Cu at (134.2, 49.0)
- added R51: 100, Resistor_SMD:R_0603_1608Metric, F.Cu at (134.2, 51.5)
- added R52: 100, Resistor_SMD:R_0603_1608Metric, F.Cu at (134.2, 54.0)
- added R53: 100k, Resistor_SMD:R_0603_1608Metric, F.Cu at (134.2, 56.5)
- added R54: 5k1, Resistor_SMD:R_0603_1608Metric, F.Cu at (156.0, 43.1)
- added R55: 5k1, Resistor_SMD:R_0603_1608Metric, F.Cu at (156.0, 45.6)
- added R56: 22, Resistor_SMD:R_0603_1608Metric, F.Cu at (165.2, 101.0)
- added R57: 100k, Resistor_SMD:R_0603_1608Metric, F.Cu at (169.2, 88.5)
- added R58: 300k, Resistor_SMD:R_0603_1608Metric, F.Cu at (169.2, 91.0)
- added R59: 1k, Resistor_SMD:R_0603_1608Metric, F.Cu at (169.2, 93.5)
- added R6: 10k, Resistor_SMD:R_0603_1608Metric, F.Cu at (136.8, 137.5)
- added R60: 100k, Resistor_SMD:R_0603_1608Metric, F.Cu at (169.2, 96.0)
- added R61: 100k, Resistor_SMD:R_0603_1608Metric, F.Cu at (169.2, 98.5)
- added R62: 1k, Resistor_SMD:R_0603_1608Metric, F.Cu at (169.2, 101.0)
- added R63: 100k, Resistor_SMD:R_0603_1608Metric, F.Cu at (173.2, 88.5)
- added R64: 1k, Resistor_SMD:R_0603_1608Metric, F.Cu at (173.2, 91.0)
- added R65: 2k4, Resistor_SMD:R_0805_2012Metric, F.Cu at (172.3, 103.8)
- added R66: 100k, Resistor_SMD:R_0603_1608Metric, F.Cu at (173.2, 93.5)
- added R67: 1k, Resistor_SMD:R_0603_1608Metric, F.Cu at (173.2, 96.0)
- added R68: 470k, Resistor_SMD:R_0603_1608Metric, F.Cu at (256.9, 66.3)
- added R69: 100k, Resistor_SMD:R_0603_1608Metric, F.Cu at (256.9, 68.8)
- added R7: 3k6, Resistor_SMD:R_0603_1608Metric, F.Cu at (136.8, 140.0)
- added R70: 200k, Resistor_SMD:R_0603_1608Metric, F.Cu at (256.9, 71.3)
- added R71: 39k, Resistor_SMD:R_0603_1608Metric, F.Cu at (256.9, 73.8)
- added R72: 75k, Resistor_SMD:R_0603_1608Metric, F.Cu at (182.6, 86.2)
- added R73: 10k, Resistor_SMD:R_0603_1608Metric, F.Cu at (182.6, 88.8)
- added R74: 2k, Resistor_SMD:R_0603_1608Metric, F.Cu at (256.9, 76.3)
- added R75: 24k, Resistor_SMD:R_0603_1608Metric, F.Cu at (182.6, 91.3)
- added R76: 47, Resistor_THT:R_Axial_DIN0309_L9.0mm_D3.2mm_P12.70mm_Horizontal, F.Cu at (237.0, 100.7)
- added R77: 39k, Resistor_SMD:R_0603_1608Metric, F.Cu at (175.2, 59.0)
- added R78: 12k, Resistor_SMD:R_0603_1608Metric, F.Cu at (175.2, 61.5)
- added R79: 100k, Resistor_SMD:R_0603_1608Metric, F.Cu at (175.2, 64.0)
- added R8: 1k, Resistor_SMD:R_0603_1608Metric, F.Cu at (136.8, 142.5)
- added R80: 10, Resistor_SMD:R_0603_1608Metric, F.Cu at (179.2, 51.5)
- added R81: 510k, Resistor_SMD:R_0603_1608Metric, F.Cu at (179.2, 54.0)
- added R82: 100k, Resistor_SMD:R_0603_1608Metric, F.Cu at (179.2, 56.5)
- added R83: 330k, Resistor_SMD:R_0603_1608Metric, F.Cu at (179.2, 59.0)
- added R84: 100k, Resistor_SMD:R_0603_1608Metric, F.Cu at (179.2, 61.5)
- added R85: 39k, Resistor_SMD:R_0603_1608Metric, F.Cu at (245.2, 58.5)
- added R86: 100, Resistor_SMD:R_0603_1608Metric, F.Cu at (245.2, 61.0)
- added R87: 330k, Resistor_SMD:R_0603_1608Metric, F.Cu at (245.2, 63.5)
- added R88: 100, Resistor_SMD:R_0603_1608Metric, F.Cu at (207.2, 78.5)
- added R89: 100k, Resistor_SMD:R_0603_1608Metric, F.Cu at (207.2, 81.0)
- added R9: 100, Resistor_SMD:R_0603_1608Metric, F.Cu at (96.0, 119.5)
- added R90: 10k, Resistor_SMD:R_0603_1608Metric, F.Cu at (207.2, 83.5)
- added R91: 10k, Resistor_SMD:R_0603_1608Metric, F.Cu at (207.2, 86.0)
- added R92: 10k, Resistor_SMD:R_0603_1608Metric, F.Cu at (216.2, 55.0)
- added R93: 10k, Resistor_SMD:R_0603_1608Metric, F.Cu at (216.2, 57.5)
- added R94: 10k, Resistor_SMD:R_0603_1608Metric, F.Cu at (216.2, 60.0)
- added R95: 2k, Resistor_SMD:R_0603_1608Metric, F.Cu at (218.0, 50.0)
- added R96: 2k, Resistor_SMD:R_0603_1608Metric, F.Cu at (218.0, 52.5)
- added R97: 100k, Resistor_SMD:R_0603_1608Metric, F.Cu at (211.2, 78.5)
- added R98: 100k, Resistor_SMD:R_0603_1608Metric, F.Cu at (211.2, 81.0)
- added R99: 100k, Resistor_SMD:R_0603_1608Metric, F.Cu at (211.2, 83.5)
- added RN1: 10k, Resistor_SMD:R_Array_Convex_4x0612, F.Cu at (117.7, 126.3)
- added RN2: 10k, Resistor_SMD:R_Array_Convex_4x0612, F.Cu at (117.7, 122.7)
- added RN3: 10k, Resistor_SMD:R_Array_Convex_4x0612, F.Cu at (117.7, 119.0)
- added SW1: TS-1088-AR02016, magnode_footprints:TS-1088-AR02016, F.Cu at (215.4, 102.3)
- added SW2: TS-1088-AR02016, magnode_footprints:TS-1088-AR02016, F.Cu at (215.4, 106.4)
- added TP1: TestPoint, TestPoint:TestPoint_THTPad_1.0x1.0mm_Drill0.5mm, F.Cu at (120.0, 138.0)
- added TP2: TestPoint, TestPoint:TestPoint_THTPad_1.0x1.0mm_Drill0.5mm, F.Cu at (164.0, 44.0)
- added TP3: TestPoint, TestPoint:TestPoint_THTPad_1.0x1.0mm_Drill0.5mm, F.Cu at (159.5, 45.0)
- added TP4: TestPoint, TestPoint:TestPoint_THTPad_1.0x1.0mm_Drill0.5mm, F.Cu at (273.0, 79.0)
- added TP5: GL3224_SPI_CS, TestPoint:TestPoint_THTPad_1.0x1.0mm_Drill0.5mm, F.Cu at (202.5, 61.5)
- added TP6: GL3224_SPI_CK, TestPoint:TestPoint_THTPad_1.0x1.0mm_Drill0.5mm, F.Cu at (202.5, 64.6)
- added TP7: GL3224_SPI_MISO, TestPoint:TestPoint_THTPad_1.0x1.0mm_Drill0.5mm, F.Cu at (202.5, 67.7)
- added TP8: GL3224_SPI_MOSI, TestPoint:TestPoint_THTPad_1.0x1.0mm_Drill0.5mm, F.Cu at (202.5, 70.7)
- added U1: HMC1001-RC, magnode_footprints:SIP8_HMC1001_HNW, F.Cu at (79.6, 143.8)
- added U12: INA851RGTR, Package_DFN_QFN:VQFN-16-1EP_3x3mm_P0.5mm_EP1.68x1.68mm, F.Cu at (133.8, 125.5)
- added U13: ISM330DHCXTR, Package_LGA:LGA-14_3x2.5mm_P0.5mm_LayoutBorder3x4y, F.Cu at (203.0, 113.9)
- added U14: TPS25210LRPWR, magnode_footprints:VQFN-HR-10, F.Cu at (218.3, 65.8)
- added U15: TPS25210LRPWR, magnode_footprints:VQFN-HR-10, F.Cu at (176.3, 79.7)
- added U16: AD7779, Package_DFN_QFN:QFN-64-1EP_9x9mm_P0.5mm_EP7.65x7.65mm, F.Cu at (159.8, 115.8)
- added U17: TPS25210LRPWR, magnode_footprints:VQFN-HR-10, F.Cu at (273.6, 75.4)
- added U18: TPS54331DR, Package_SO:SOIC-8_3.9x4.9mm_P1.27mm, F.Cu at (194.5, 79.4)
- added U19: TPS7A2033PDBVR, Package_TO_SOT_SMD:SOT-23-5, F.Cu at (193.0, 101.0)
- added U2: HMC1002-TR, magnode_footprints:SOIC20_HNW, F.Cu at (71.6, 139.3)
- added U20: TPS7A4901DGNR, Package_SO:HVSSOP-8-1EP_3x3mm_P0.65mm_EP1.57x1.89mm, F.Cu at (180.9, 67.7)
- added U21: TPS63700DRCR, Package_SON:VSON-10-1EP_3x3mm_P0.5mm_EP1.2x2mm, F.Cu at (172.2, 72.2)
- added U22: TPS7A3301RGWR, Package_DFN_QFN:Texas_RGW0020A_VQFN-20-1EP_5x5mm_P0.65mm_EP3.15x3.15mm_ThermalVias, F.Cu at (192.0, 64.0)
- added U23: TS3A27518ERTW, Package_DFN_QFN:WQFN-24-1EP_4x4mm_P0.5mm_EP2.6x2.6mm, F.Cu at (226.7, 79.3)
- added U24: GL3224-OIY04, Package_DFN_QFN:QFN-32-1EP_5x5mm_P0.5mm_EP3.1x3.1mm, F.Cu at (226.6, 70.8)
- added U25: HD3SS3220RNHR, Package_DFN_QFN:Texas_RNH0030A_WQFN-30-1EP_2.5x4.5mm_P0.4mm_EP1.2x3.2mm, F.Cu at (232.0, 63.2)
- added U26: 2x08_pheonix_connector_male, magnode_footprints:GPS_TILE_3D, F.Cu at (151.0, 100.1)
- added U4: LM324, Package_SO:SOIC-14_3.9x8.7mm_P1.27mm, F.Cu at (109.5, 120.7)
- added Y1: OT2JI-111-8.192M, Crystal:Crystal_SMD_3225-4Pin_3.2x2.5mm, F.Cu at (168.1, 119.0)
- added Y2: X322525MOB4SI, Crystal:Crystal_SMD_3225-4Pin_3.2x2.5mm, F.Cu at (219.9, 72.2)
- Q2: value B772 -> DMC3028LSD; footprint Package_TO_SOT_SMD:SOT-89-3 -> Package_SO:SO-8_3.9x4.9mm_P1.27mm
- Q3: value DMC3028LSD -> B772; footprint Package_SO:SO-8_3.9x4.9mm_P1.27mm -> Package_TO_SOT_SMD:SOT-89-3
- R18: value 20 -> 510k; footprint Resistor_SMD:R_1206_3216Metric -> Resistor_SMD:R_0603_1608Metric
- U10: value TPS7A2045PDBVR -> INA851RGTR; footprint Package_SON:Texas_X2SON-4_1x1mm_P0.65mm -> Package_DFN_QFN:VQFN-16-1EP_3x3mm_P0.5mm_EP1.68x1.68mm
- U11: value DAN-F10N -> INA851RGTR; footprint magnode_footprints:u-blox_DAN-F10N_LCC-56_20x20mm -> Package_DFN_QFN:VQFN-16-1EP_3x3mm_P0.5mm_EP1.68x1.68mm
- U3: value MCP4728 -> TPS61170; footprint Package_SO:MSOP-10_3x3mm_P0.5mm -> Package_SON:WSON-6-1EP_2x2mm_P0.65mm_EP1x1.6mm
- U5: value LT3042xMSE -> MCP4728; footprint Package_SO:MSOP-10-1EP_3x3mm_P0.5mm_EP1.68x1.88mm -> Package_SO:MSOP-10_3x3mm_P0.5mm
- U6: value TPS61040DBV -> LT3042xMSE; footprint Package_TO_SOT_SMD:SOT-23-5 -> Package_SO:MSOP-10-1EP_3x3mm_P0.5mm_EP1.68x1.88mm
- U7: value ESP32-S3-WROOM-1 -> TPS61040DBV; footprint RF_Module:ESP32-S3-WROOM-1 -> Package_TO_SOT_SMD:SOT-23-5
- U8: value AD7779 -> ESP32-S3-WROOM-1; footprint Package_DFN_QFN:QFN-64-1EP_9x9mm_P0.5mm_EP7.65x7.65mm -> RF_Module:ESP32-S3-WROOM-1
- U9: value XC6206PxxxMR -> 74HC595D,118; footprint Package_TO_SOT_SMD:SOT-23-3 -> Package_SO:SOIC-16_3.9x9.9mm_P1.27mm
- moved U6 138.2 mm to (61.6, 129.5)
- moved U7 95.6 mm to (178.0, 134.0), turned to 0 degrees
- moved U5 85.2 mm to (124.9, 135.0)
- moved U3 78.7 mm to (160.1, 139.7)
- moved Q3 78.4 mm to (109.0, 129.0)
- moved Q1 76.4 mm to (115.0, 134.0)
- moved U11 75.9 mm to (133.8, 120.2)
- moved Q5 74.9 mm to (86.0, 124.0)
- moved D2 73.8 mm to (165.1, 142.5)
- moved Q6 73.0 mm to (78.8, 121.1)
- moved Q7 73.0 mm to (78.8, 127.2)
- moved U10 72.6 mm to (133.8, 114.9)
- moved Q2 70.1 mm to (145.0, 141.0)
- moved Q10 67.1 mm to (86.0, 144.4)
- moved Q8 67.1 mm to (86.0, 132.1)
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Connections:
- Q1 pad 1: (no net) -> Net-(Q1-B)
- Q1 pad 2: (no net) -> Net-(Q1-C)
- Q1 pad 3: (no net) -> Net-(Q1-E)
- Q10 pad 1: (no net) -> /SENSOR_OFFSET_DRIVERS/OFF_Z_BP
- Q10 pad 2: (no net) -> -5VA
- Q10 pad 3: (no net) -> /SENSOR_OFFSET_DRIVERS/OFF_Z_SENSE_P
- Q2 pad 1: (no net) -> GND
- Q2 pad 2: (no net) -> /MCU_ESP32S3/SENSOR_RESET_CTRL
- Q2 pad 3: (no net) -> Net-(Q1-C)
- Q3 pad 1: GND -> Net-(Q1-B)
- Q3 pad 2: /SENSOR_SET_RESET_DRIVER/RESET_CTRL -> GND
- Q3 pad 3: Net-(Q3B-S2) -> Net-(Q1-E)
- Q4 pad 1: (no net) -> Net-(D2-K)
- Q4 pad 2: (no net) -> Net-(Q4-C)
- Q4 pad 3: (no net) -> GND
- Q5 pad 1: (no net) -> /SENSOR_OFFSET_DRIVERS/OFF_X_BN
- Q5 pad 2: (no net) -> +5V
- Q5 pad 3: (no net) -> /SENSOR_OFFSET_DRIVERS/OFF_X_SENSE_P
- Q6 pad 1: (no net) -> /SENSOR_OFFSET_DRIVERS/OFF_X_BP
- Q6 pad 2: (no net) -> -5VA
- Q6 pad 3: (no net) -> /SENSOR_OFFSET_DRIVERS/OFF_X_SENSE_P
- Q7 pad 1: (no net) -> /SENSOR_OFFSET_DRIVERS/OFF_Y_BN
- Q7 pad 2: (no net) -> +5V
- Q7 pad 3: (no net) -> /SENSOR_OFFSET_DRIVERS/OFF_Y_SENSE_P
- Q8 pad 1: (no net) -> /SENSOR_OFFSET_DRIVERS/OFF_Y_BP
- Q8 pad 2: (no net) -> -5VA
- Q8 pad 3: (no net) -> /SENSOR_OFFSET_DRIVERS/OFF_Y_SENSE_P
- Q9 pad 1: (no net) -> /SENSOR_OFFSET_DRIVERS/OFF_Z_BN
- Q9 pad 2: (no net) -> +5V
- Q9 pad 3: (no net) -> /SENSOR_OFFSET_DRIVERS/OFF_Z_SENSE_P
- R18 pad 1: Net-(C6-Pad2) -> /PWR_5VA_NEG5/+10V
- R18 pad 2: /SENSOR_3AXIS_HMC100X/OFFSET_Y+ -> Net-(R18-Pad2)
- U10 pad 1: unconnected-(U10-OUT-Pad1) -> /ANALOG_FRONTEND_INA851/BR_X+
- U10 pad 2: unconnected-(U10-GND-Pad2) -> /ANALOG_FRONTEND_INA851/X_RG+
- U10 pad 3: unconnected-(U10-EN-Pad3) -> /ANALOG_FRONTEND_INA851/X_RG-
- U10 pad 4: unconnected-(U10-IN-Pad4) -> /ANALOG_FRONTEND_INA851/BR_X-
- U10 pad 5: unconnected-(U10-Pad-Pad5) -> GND
- U11 pad 1: unconnected-(U11-GND-Pad1) -> /ANALOG_FRONTEND_INA851/BR_Z-
- U11 pad 10: unconnected-(U11-TXD-Pad10) -> /ANALOG_FRONTEND_INA851/Z_INA_PRE_AAF-
- U11 pad 11: unconnected-(U11-NC-Pad11) -> /ANALOG_FRONTEND_INA851/Z_INA_PRE_AAF+
- U11 pad 13: unconnected-(U11-GND-Pad13) -> +1V65
- U11 pad 14: unconnected-(U11-GND-Pad14) -> +5VA
- U11 pad 16: unconnected-(U11-RESET_N-Pad16) -> +3V3A
- U11 pad 17: unconnected-(U11-EXTINT-Pad17) -> GND
- U11 pad 2: unconnected-(U11-GND-Pad2) -> /ANALOG_FRONTEND_INA851/Z_RG+
- U11 pad 3: unconnected-(U11-GND-Pad3) -> /ANALOG_FRONTEND_INA851/Z_RG-
- U11 pad 4: unconnected-(U11-GND-Pad4) -> /ANALOG_FRONTEND_INA851/BR_Z+
- U11 pad 5: unconnected-(U11-GND-Pad5) -> GND
- U11 pad 7: unconnected-(U11-GND-Pad7) -> -5VA
- U3 pad 1: +3V3D -> Net-(U3-FB)
- U3 pad 2: /SENSOR_OFFSET_DRIVERS/I2C_DAC_SCL -> Net-(U3-COMP)
- U3 pad 3: /SENSOR_OFFSET_DRIVERS/I2C_DAC_SDA -> GND
- U3 pad 4: /SENSOR_OFFSET_DRIVERS/DAC_LDAC_N -> Net-(D1-A)
- U3 pad 5: /SENSOR_OFFSET_DRIVERS/DAC_RDY_N -> /MCU_ESP32S3/EN_BST_18V
- U3 pad 6: /SENSOR_OFFSET_DRIVERS/DAC_OUT_X -> +5V
- U3 pad 7: /SENSOR_OFFSET_DRIVERS/DAC_OUT_Y -> GND
- U5 pad 1: Net-(U5-IN-Pad1) -> +3V3D
- U5 pad 10: unconnected-(U5-OUT-Pad10) -> GND
- U5 pad 2: Net-(U5-IN-Pad1) -> /IMU/I2C.SCL
- U5 pad 3: unconnected-(U5-EN/UV-Pad3) -> /IMU/I2C.SDA
- U5 pad 4: unconnected-(U5-PG-Pad4) -> /MCU_ESP32S3/DAC_LDAC_N
- U5 pad 5: unconnected-(U5-ILIM-Pad5) -> /SENSOR_OFFSET_DRIVERS/DAC_RDY_N
- U5 pad 6: unconnected-(U5-PGFB-Pad6) -> /SENSOR_OFFSET_DRIVERS/DAC_OUT_X
- U5 pad 7: unconnected-(U5-SET-Pad7) -> /SENSOR_OFFSET_DRIVERS/DAC_OUT_Y
- U5 pad 8: Net-(U5-GND-Pad11) -> /SENSOR_OFFSET_DRIVERS/DAC_OUT_Z
- U5 pad 9: unconnected-(U5-OUTS-Pad9) -> /SENSOR_OFFSET_DRIVERS/DAC_OUT_REF
- U6 pad 1: unconnected-(U6-SW-Pad1) -> /PWR_5VA_NEG5/+10V
- U6 pad 2: unconnected-(U6-GND-Pad2) -> /PWR_5VA_NEG5/+10V
- U6 pad 3: unconnected-(U6-FB-Pad3) -> /PWR_5VA_NEG5/+10V
- U6 pad 5: unconnected-(U6-VIN-Pad5) -> /PWR_9V_BRIDGE/LDO_9V_ILIM
- U7 pad 1: Net-(U7-GND-Pad1) -> /PWR_9V_BRIDGE/BST_10V_SW
- U7 pad 2: unconnected-(U7-3V3-Pad2) -> GND
- U7 pad 3: unconnected-(U7-EN-Pad3) -> /PWR_9V_BRIDGE/BST_10V_FB
- U7 pad 4: unconnected-(U7-IO4-Pad4) -> /MCU_ESP32S3/EN_BST_10V
- U7 pad 5: unconnected-(U7-IO5-Pad5) -> +5V
- U8 pad 1: unconnected-(U8-AIN0--Pad1) -> GND
- U8 pad 10: unconnected-(U8-AIN2+-Pad10) -> /ADC_AD777X/ADC_RESET
- U8 pad 11: unconnected-(U8-AIN3--Pad11) -> /ADC_AD777X/ADC_CONVST_SAR
- U8 pad 12: unconnected-(U8-AIN3+-Pad12) -> /MCU_ESP32S3/ADC_SPI_SDI
- U8 pad 13: unconnected-(U8-MODE0/GPIO0-Pad13) -> /DATA_SAVING/D-
- U8 pad 14: unconnected-(U8-MODE1/GPIO1-Pad14) -> /DATA_SAVING/D+
- U8 pad 15: unconnected-(U8-MODE2/GPIO2-Pad15) -> /IMU/I2C.SDO
- U8 pad 16: unconnected-(U8-MODE3/ALERT-Pad16) -> /GPS_TILE/GPS_UART.RX
- U8 pad 17: unconnected-(U8-CONVST_SAR-Pad17) -> /MCU_ESP32S3/SENSOR_RESET_CTRL
- U8 pad 18: unconnected-(U8-ALERT/~{CS}-Pad18) -> /MCU_ESP32S3/SENSOR_SET_CTRL
- U8 pad 19: unconnected-(U8-DCLK2/SCLK-Pad19) -> Net-(U8-IO11)
- U8 pad 2: unconnected-(U8-AIN0+-Pad2) -> +3V3
- U8 pad 21: unconnected-(U8-DCLK0/SDO-Pad21) -> Net-(U8-IO13)
- U8 pad 22: unconnected-(U8-DGND-Pad22) -> Net-(U8-IO14)
- U8 pad 24: unconnected-(U8-IOVDD-Pad24) -> /GPS_TILE/GPS_UART.TX
- U8 pad 25: unconnected-(U8-DOUT3-Pad25) -> /IO_CONNECTOR/EN_KEEPALIVE
- U8 pad 26: unconnected-(U8-DOUT2-Pad26) -> /DATA_SAVING/D3
- U8 pad 27: unconnected-(U8-DOUT1-Pad27) -> /MCU_ESP32S3/ESP32_BOOTH
- U8 pad 3: unconnected-(U8-AIN1--Pad3) -> /MCU_ESP32S3/ESP32_EN
- U8 pad 31: unconnected-(U8-XTAL1-Pad31) -> /DATA_SAVING/CMD
- U8 pad 32: unconnected-(U8-XTAL2/MCLK-Pad32) -> /DATA_SAVING/CLK
- U8 pad 33: unconnected-(U8-~{START}-Pad33) -> /DATA_SAVING/D0
- U8 pad 34: unconnected-(U8-~{SYNC_OUT}-Pad34) -> /DATA_SAVING/D1
- U8 pad 35: unconnected-(U8-~{SYNC_IN}-Pad35) -> /DATA_SAVING/D2
- U8 pad 36: unconnected-(U8-~{RESET}-Pad36) -> /ADC_AD777X/ADC_MCLK_EN
- U8 pad 37: unconnected-(U8-AIN7+-Pad37) -> /ADC_AD777X/ADC_START
- U8 pad 38: unconnected-(U8-AIN7--Pad38) -> /IMU/I2C.SCL
- U8 pad 39: unconnected-(U8-AIN6+-Pad39) -> /ADC_AD777X/ADC_DRDY
- U8 pad 4: unconnected-(U8-AIN1+-Pad4) -> /IMU/I2C.SDA
- U8 pad 40: unconnected-(U8-AIN6--Pad40) -> GND
- U8 pad 41: unconnected-(U8-REF2+-Pad41) -> GND
- U8 pad 5: unconnected-(U8-AVSS1A-Pad5) -> /MCU_ESP32S3/ADC_SPI_CS
- U8 pad 6: unconnected-(U8-AVDD1A-Pad6) -> /MCU_ESP32S3/ADC_SPI_SCLK
- U8 pad 7: unconnected-(U8-REF1--Pad7) -> /ADC_AD777X/SPI.SDO
- U8 pad 8: unconnected-(U8-REF1+-Pad8) -> /GPS_TILE/GPS_TIMEPULSE
- U8 pad 9: unconnected-(U8-AIN2--Pad9) -> Net-(U8-IO16)
- U9 pad 1: unconnected-(U9-GND-Pad1) -> /MCU_ESP32S3/EN_LDO_3V3
- U9 pad 2: unconnected-(U9-VO-Pad2) -> /MCU_ESP32S3/EN_INV_-5V
- U9 pad 3: unconnected-(U9-VI-Pad3) -> /MCU_ESP32S3/EN_BST_18V
Routing:
- net /PWR_3V3D/5V_SUPERCAP: track 0.00 -> 14.1 mm
- net /PWR_3V3D/5V_CAP_CHG: track 0.00 -> 4.97 mm
Other:
- board outline added: 193 x 110 mm
