File: hardware/pcb/Expension_card_design/geophys_mainboard/schematics/sd_card_saving_usb_to_pc.kicad_sch (KiCad schematic)
At the start: 37 parts, among them J4 Micro_SD_CARD, U16 TS3A27518EPWR, U17 USB2641-HZH-02, X1 X322524MOB4SI

Commit message: SD mux and 3V3D power sequencing bring-up
Parts:
- removed U16: TS3A27518EPWR, Package_SO:TSSOP-24_4.4x7.8mm_P0.65mm, symbol magnode_symbols:TS3A27518ERTW
- added U16: TS3A27518EPWR, Package_SO:TSSOP-24_4.4x7.8mm_P0.65mm, symbol magnode_symbols:TS3A27518EPWR
Connections:
- net +3V3: now also U16.8 (VCC)
- net EN_SD_MUX: now also U16.20 (~{EN})
- net E_CLK: now also U16.23 (NC3)
- net E_CMD: now also U16.21 (NC4)
- net E_D0: now also U16.1 (NC2)
- net E_D1: now also U16.2 (NC1)
- net E_D2: now also U16.22 (NC6)
- net E_D3: now also U16.19 (NC5)
- net GND: now also U16.5 (GND)
- net MCLK: now also U16.7 (COM3)
- net MCMD: now also U16.9 (COM4)
- net MD0: now also U16.6 (COM2)
- net MD1: now also U16.4 (COM1)
- net MD2: now also U16.12 (COM6)
- net MD3: now also U16.10 (COM5)
- net SD_MUX_SEL: now also U16.14 (IN2), U16.24 (IN1)
- net USB_CLK: now also U16.15 (NO3)
- net USB_CMD: now also U16.17 (NO4)
- net USB_D0: now also U16.13 (NO2)
- net USB_D1: now also U16.11 (NO1)
- net USB_D2: now also U16.16 (NO6)
- net USB_D3: now also U16.18 (NO5)
