File: hardware/pcb/Expension_card_design/geophys_mainboard/schematics/sensor_set_reset_driver.kicad_sch (KiCad schematic)
At the start: 12 parts, among them U1 TPS61170

Commit message: Backup avant deletion offset/dac
Parts:
- L1: footprint Inductor_SMD:L_Sunlord_MWSA0503S -> magnode_footprints:ZEMS0850-100M_8.5x8.0mm; LCSC C177248 -> C41413139
Changed lines of the file:
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@@
+			)
+		)
+		(property "Sim.Enable" ""
+			(at 114.3 109.22 0)
+			(effects
+				(font
+					(size 1.27 1.27)
+				)
+				(hide yes)
 			)
 		)
@@
 			)
 		)
+		(property "Sim.Enable" ""
+			(at 154.94 97.79 0)
+			(effects
+				(font
+					(size 1.27 1.27)
+				)
+				(hide yes)
+			)
+		)
 		(pin "2"
 		)
@@
 			)
 		)
-		(property "Footprint" "Inductor_SMD:L_Sunlord_MWSA0503S"
+		(property "Footprint" "magnode_footprints:ZEMS0850-100M_8.5x8.0mm"
 			(at 132.08 86.36 0)
 			(effects
@@
 			)
 		)
-		(property "LCSC" "C177248"
+		(property "LCSC" "C41413139"
 			(at 132.08 86.36 90)
 			(effects
@@
 		)
 		(property "Sim.Pins" ""
+			(at 132.08 86.36 90)
+			(effects
+				(font
+					(size 1.27 1.27)
+				)
+				(hide yes)
+			)
+		)
+		(property "Sim.Enable" ""
 			(at 132.08 86.36 90)
 			(effects
@@
 			)
 		)
+		(property "Sim.Enable" ""
+			(at 184.15 102.87 0)
+			(effects
+				(font
+					(size 1.27 1.27)
+				)
+				(hide yes)
+			)
+		)
 		(pin "2"
 		)
@@
 		)
 		(property "Sim.Pins" ""
+			(at 77.47 97.79 90)
+			(effects
+				(font
+					(size 1.27 1.27)
+				)
+				(hide yes)
+			)
+		)
+		(property "Sim.Enable" ""
 			(at 77.47 97.79 90)
 			(effects
@@
 			)
 		)
+		(property "Sim.Enable" ""
+			(at 132.08 105.41 0)
+			(effects
+				(font
+					(size 1.27 1.27)
+				)
+				(hide yes)
+			)
+		)
 		(pin "5"
 		)
@@
 			)
 		)
+		(property "Sim.Enable" ""
+			(at 162.56 113.03 90)
+			(effects
+				(font
+					(size 1.27 1.27)
+				)
+				(hide yes)
+			)
+		)
 		(pin "2"
 		)
@@
 			)
 		)
+		(property "Sim.Enable" ""
+			(at 196.85 101.6 0)
+			(effects
+				(font
+					(size 1.27 1.27)
+				)
+				(hide yes)
+			)
+		)
 		(pin "1"
 		)
@@
 			)
 		)
+		(property "Sim.Enable" ""
+			(at 209.55 97.79 90)
+			(effects
+				(font
+					(size 1.27 1.27)
+				)
+				(hide yes)
+			)
+		)
 		(pin "2"
 		)
@@
 			)
 		)
+		(property "Sim.Enable" ""
+			(at 173.99 116.84 0)
+			(effects
+				(font
+					(size 1.27 1.27)
+				)
+				(hide yes)
+			)
+		)
 		(pin "1"
 		)
@@
 		)
 		(property "Sim.Pins" ""
+			(at 184.15 113.03 0)
+			(effects
+				(font
+					(size 1.27 1.27)
+				)
+				(hide yes)
+			)
+		)
+		(property "Sim.Enable" ""
 			(at 184.15 113.03 0)
 			(effects
@@
 			(at 90.17 101.6 0)
 			(effects
+				(font
+					(size 1.27 1.27)
+				)
+				(hide yes)
+			)
+		)
+		(property "Sim.Enable" ""
+			(at 90.17 101.6 0)
+			(effects
