File: hardware/pcb/Expension_card_design/geophys_mainboard/schematics/pwr_3v3a.kicad_sch (KiCad schematic)
At the start: 9 parts, among them U11 TPS7A2033PDBVR

Commit message: Work in progress rev2
Parts:
- removed C37, C40: 4u7, Capacitor_SMD:C_1206_3216Metric, symbol Device:C
- removed C38, C39: 100n, Capacitor_SMD:C_0603_1608Metric, symbol Device:C
- removed FB2: 120Ω@100MHz 2A 50mΩ, Inductor_SMD:L_0603_1608Metric, symbol PCM_Device_AKL:Ferrite_Bead
- removed R50, R51: 0, Resistor_SMD:R_1206_3216Metric, symbol Device:R
- removed TP9: TestPoint, TestPoint:TestPoint_THTPad_1.0x1.0mm_Drill0.5mm, symbol Connector:TestPoint
- removed U11: TPS7A2033PDBVR, Package_TO_SOT_SMD:SOT-23-5, symbol magnode_symbols:TPS7A2033PDBVR
Other:
- note removed: "+3.3V LDO"
- note removed: "Voltage for analog domain of the ADC"
