File: hardware/pcb/Expension_card_design/geophys_mainboard/schematics/pwr_9v_bridge.kicad_sch (KiCad schematic)
At the start: 22 parts, among them U2 LT3042xMSE, U3 TPS61040DBV

Commit message: Backup avant deletion offset/dac
Parts:
- L2: footprint Inductor_SMD:L_Sunlord_MWSA0503S -> magnode_footprints:ZEMS0850-100M_8.5x8.0mm; LCSC C177248 -> C41413139
Changed lines of the file:
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@@
+			)
+		)
+		(property "Sim.Enable" ""
+			(at 227.33 95.25 0)
+			(effects
+				(font
+					(size 1.27 1.27)
+				)
+				(hide yes)
 			)
 		)
@@
 			)
 		)
+		(property "Sim.Enable" ""
+			(at 88.9 90.17 0)
+			(effects
+				(font
+					(size 1.27 1.27)
+				)
+				(hide yes)
+			)
+		)
 		(pin "1"
 		)
@@
 			)
 		)
+		(property "Sim.Enable" ""
+			(at 96.52 93.98 0)
+			(effects
+				(font
+					(size 1.27 1.27)
+				)
+				(hide yes)
+			)
+		)
 		(pin "2"
 		)
@@
 			)
 		)
+		(property "Sim.Enable" ""
+			(at 120.65 97.79 0)
+			(effects
+				(font
+					(size 1.27 1.27)
+				)
+				(hide yes)
+			)
+		)
 		(pin "1"
 		)
@@
 			)
 		)
+		(property "Sim.Enable" ""
+			(at 189.23 100.33 0)
+			(effects
+				(font
+					(size 1.27 1.27)
+				)
+				(hide yes)
+			)
+		)
 		(pin "1"
 		)
@@
 			)
 		)
+		(property "Sim.Enable" ""
+			(at 205.74 106.68 0)
+			(effects
+				(font
+					(size 1.27 1.27)
+				)
+				(hide yes)
+			)
+		)
 		(pin "1"
 		)
@@
 			)
 		)
+		(property "Sim.Enable" ""
+			(at 107.95 97.79 0)
+			(effects
+				(font
+					(size 1.27 1.27)
+				)
+				(hide yes)
+			)
+		)
 		(pin "1"
 		)
@@
 			)
 		)
+		(property "Sim.Enable" ""
+			(at 251.46 92.71 0)
+			(effects
+				(font
+					(size 1.27 1.27)
+				)
+				(hide yes)
+			)
+		)
 		(pin "1"
 		)
@@
 			)
 		)
+		(property "Sim.Enable" ""
+			(at 121.92 90.17 0)
+			(effects
+				(font
+					(size 1.27 1.27)
+				)
+				(hide yes)
+			)
+		)
 		(pin "1"
 		)
@@
 			)
 		)
+		(property "Sim.Enable" ""
+			(at 128.27 90.17 90)
+			(effects
+				(font
+					(size 1.27 1.27)
+				)
+				(hide yes)
+			)
+		)
 		(pin "2"
 		)
@@
 			)
 		)
+		(property "Sim.Enable" ""
+			(at 96.52 102.87 0)
+			(effects
+				(font
+					(size 1.27 1.27)
+				)
+				(hide yes)
+			)
+		)
 		(pin "2"
 		)
@@
 			)
 		)
+		(property "Sim.Enable" ""
+			(at 180.34 100.33 0)
+			(effects
+				(font
+					(size 1.27 1.27)
+				)
+				(hide yes)
+			)
+		)
 		(pin "1"
 		)
@@
 			)
 		)
+		(property "Sim.Enable" ""
+			(at 175.26 92.71 90)
+			(effects
+				(font
+					(size 1.27 1.27)
+				)
+				(hide yes)
+			)
+		)
 		(pin "2"
 		)
@@
 		)
 		(property "Sim.Pins" ""
+			(at 215.9 106.68 0)
+			(effects
+				(font
+					(size 1.27 1.27)
+				)
+				(hide yes)
+			)
+		)
+		(property "Sim.Enable" ""
 			(at 215.9 106.68 0)
 			(effects
@@
 			)
 		)
+		(property "Sim.Enable" ""
+			(at 71.12 106.68 0)
+			(effects
+				(font
+					(size 1.27 1.27)
+				)
+				(hide yes)
+			)
+		)
 		(pin "4"
 		)
@@
 			)
 		)
+		(property "Sim.Enable" ""
+			(at 256.54 92.71 90)
+			(effects
+				(font
+					(size 1.27 1.27)
+				)
+				(hide yes)
+			)
+		)
 		(pin "2"
 		)
@@
 			)
 		)
+		(property "Sim.Enable" ""
+			(at 46.99 113.03 0)
+			(effects
+				(font
+					(size 1.27 1.27)
+				)
+				(hide yes)
+			)
+		)
 		(pin "1"
 		)
@@
 			)
 		)
+		(property "Sim.Enable" ""
+			(at 38.1 104.14 90)
+			(effects
+				(font
+					(size 1.27 1.27)
+				)
+				(hide yes)
+			)
+		)
 		(pin "2"
 		)
@@
 		)
 		(property "Sim.Pins" ""
+			(at 92.71 111.76 0)
+			(effects
+				(font
+					(size 1.27 1.27)
+				)
+				(hide yes)
+			)
+		)
+		(property "Sim.Enable" ""
 			(at 92.71 111.76 0)
 			(effects
@@
 			)
 		)
-		(property "Footprint" "Inductor_SMD:L_Sunlord_MWSA0503S"
+		(property "Footprint" "magnode_footprints:ZEMS0850-100M_8.5x8.0mm"
 			(at 71.12 90.17 0)
 			(effects
@@
 			)
 		)
-		(property "LCSC" "C177248"
+		(property "LCSC" "C41413139"
 			(at 71.12 90.17 90)
 			(effects
@@
 		)
 		(property "Sim.Pins" ""
+			(at 71.12 90.17 90)
+			(effects
+				(font
+					(size 1.27 1.27)
+				)
+				(hide yes)
+			)
+		)
+		(property "Sim.Enable" ""
 			(at 71.12 90.17 90)
 			(effects
@@
 			)
 		)
+		(property "Sim.Enable" ""
+			(at 248.92 99.06 0)
+			(effects
+				(font
+					(size 1.27 1.27)
+				)
+				(hide yes)
+			)
+		)
 		(pin "1"
 		)
@@
 			(at 207.01 97.79 90)
 			(effects
+				(font
+					(size 1.27 1.27)
+				)
+				(hide yes)
+			)
+		)
+		(property "Sim.Enable" ""
+			(at 207.01 97.79 90)
+			(effects

Commit message: Work in progress rev2
Parts:
- removed C10, C6, C9: 4u7, Capacitor_SMD:C_1206_3216Metric, symbol Device:C
- removed C4: 22p, Capacitor_SMD:C_0603_1608Metric, symbol Device:C
- removed C5: 1u, Capacitor_SMD:C_0805_2012Metric, symbol Device:C
- removed C7: 10u, Capacitor_SMD:C_0805_2012Metric, symbol Device:C
- removed C8: 100n, Capacitor_SMD:C_0603_1608Metric, symbol Device:C
- removed D2: SS34, Diode_SMD:D_SMA, symbol Device:D_Schottky
- removed L2: 10u, magnode_footprints:ZEMS0850-100M_8.5x8.0mm, symbol Device:L
- removed R10, R11, R15, R9: 0, Resistor_SMD:R_1206_3216Metric, symbol Device:R
- removed R12: 510k, Resistor_SMD:R_0603_1608Metric, symbol Device:R
- removed R13: 1k, Resistor_SMD:R_0603_1608Metric, symbol Device:R
- removed R14: 200k, Resistor_SMD:R_0603_1608Metric, symbol Device:R
- removed R16: 90k9, Resistor_SMD:R_1206_3216Metric, symbol Device:R
- removed R17: 100k, Resistor_SMD:R_0603_1608Metric, symbol Device:R
- removed TP1, TP2: TestPoint, TestPoint:TestPoint_THTPad_1.0x1.0mm_Drill0.5mm, symbol Connector:TestPoint
- removed U2: LT3042xMSE, Package_SO:MSOP-10-1EP_3x3mm_P0.5mm_EP1.68x1.88mm, symbol Regulator_Linear:LT3042xMSE
- removed U3: TPS61040DBV, Package_TO_SOT_SMD:SOT-23-5, symbol Regulator_Switching:TPS61040DBV
Connections:
- no-connect marks 1 -> 0
Other:
- note removed: "+10V Boost"
- note removed: "+9V LDO"
- note removed: "Voltage for bridge of the magnetic sensors"
- note removed: "Voltage for the +9V and +5V LDO"
