File: hardware/pcb/Expension_card_design/geophys_mainboard/schematics/pwr_opamp_4v5_neg5.kicad_sch (KiCad schematic)
At the start: 41 parts, among them U13 TPS7A4901DGNR, U14 TPS7A3301RGWR, U15 TPS63700DRCR

Commit message: Backup avant deletion offset/dac
Parts:
- L4: footprint Inductor_SMD:L_Sunlord_MWSA0503S -> magnode_footprints:ZEMS0850-100M_8.5x8.0mm; LCSC C177248 -> C41413139

Commit message: Work in progress rev2
Parts:
- removed C65, C67, C71, C77: 10u, Capacitor_SMD:C_0805_2012Metric, symbol Device:C
- removed C66, C68, C73, C78: 10n, Capacitor_SMD:C_0603_1608Metric, symbol Device:C
- removed C69, C72, C76: 100n, Capacitor_SMD:C_0603_1608Metric, symbol Device:C
- removed C70: 220n, Capacitor_SMD:C_0603_1608Metric, symbol Device:C
- removed C74: 47u, Capacitor_SMD:C_1206_3216Metric, symbol Device:C
- removed C75: 10p, Capacitor_SMD:C_0603_1608Metric, symbol Device:C
- removed C79, C80, C81, C82: 4u7, Capacitor_SMD:C_1206_3216Metric, symbol Device:C
- removed C83: 4n7, Capacitor_SMD:C_0603_1608Metric, symbol Device:C
- removed D10: SS34, Diode_SMD:D_SMA, symbol Device:D_Schottky
- removed L4: 10u, magnode_footprints:ZEMS0850-100M_8.5x8.0mm, symbol Device:L
- removed R81, R82, R85, R86, R91, R94: 0, Resistor_SMD:R_1206_3216Metric, symbol Device:R
- removed R83: 39k, Resistor_SMD:R_0603_1608Metric, symbol Device:R
- removed R84: 12k, Resistor_SMD:R_0603_1608Metric, symbol Device:R
- removed R87, R90, R93: 100k, Resistor_SMD:R_0603_1608Metric, symbol Device:R
- removed R88: 330k, Resistor_SMD:R_0603_1608Metric, symbol Device:R
- removed R89: 10, Resistor_SMD:R_0603_1608Metric, symbol Device:R
- removed R92: 510k, Resistor_SMD:R_0603_1608Metric, symbol Device:R
- removed TP10, TP11, TP12: TestPoint, TestPoint:TestPoint_THTPad_1.0x1.0mm_Drill0.5mm, symbol Connector:TestPoint
- removed U13: TPS7A4901DGNR, magnode_footprints:HVSSOP-8-1EP_3x3mm_P0.65mm_EP1.57x1.89mm, symbol magnode_symbols:TPS7A4901
- removed U14: TPS7A3301RGWR, Package_DFN_QFN:Texas_RGW0020A_VQFN-20-1EP_5x5mm_P0.65mm_EP3.15x3.15mm, symbol Regulator_Linear:TPS7A3301RGW
- removed U15: TPS63700DRCR, Package_SON:VSON-10-1EP_3x3mm_P0.5mm_EP1.2x2mm, symbol magnode_symbols:TPS63700
Connections:
- no-connect marks 1 -> 0
Other:
- note removed: "+5V LDO"
- note removed: "-5V LDO"
- note removed: "-6.2V Inverter"
- note removed: "Voltage for the instrumentation Op-Amps"
- note removed: "Voltage needed for the -5V LDO"
- note removed: "taken du board #2"
