File: hardware/pcb/Expension_card_design/geophys_mainboard/geophys_mainboard.kicad_pcb (KiCad board)
At the start: 4 copper layers, 190 x 110 mm, 322 parts, among them J1 550910274, J2 USB_C_Receptacle_USB2.0_16P, J3 550910274, J4 Micro_SD_CARD, Q1 AO3400A, Q2 AO3401A, Q3 AO3400A, U1 TPS61170, U10 TPS54331DR, U11 TPS7A2033PDBVR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

Commit message: Work in progress rev2
Parts:
- added C10: 4u7, Capacitor_SMD:C_1206_3216Metric, F.Cu at (217.9, -42.8)
- added C37: 4u7, Capacitor_SMD:C_1206_3216Metric, F.Cu at (217.9, -39.5)
- added C38: 100n, Capacitor_SMD:C_0603_1608Metric, F.Cu at (222.7, -44.9)
- added C39: 100n, Capacitor_SMD:C_0603_1608Metric, F.Cu at (222.7, -42.4)
- added C4: 22p, Capacitor_SMD:C_0603_1608Metric, F.Cu at (222.7, -49.9)
- added C40: 4u7, Capacitor_SMD:C_1206_3216Metric, F.Cu at (217.9, -36.1)
- added C5: 1u, Capacitor_SMD:C_0805_2012Metric, F.Cu at (250.1, -49.7)
- added C6: 4u7, Capacitor_SMD:C_1206_3216Metric, F.Cu at (217.9, -49.5)
- added C65: 10u, Capacitor_SMD:C_0805_2012Metric, F.Cu at (250.1, -43.7)
- added C66: 10n, Capacitor_SMD:C_0603_1608Metric, F.Cu at (222.7, -39.9)
- added C67: 10u, Capacitor_SMD:C_0805_2012Metric, F.Cu at (250.1, -40.7)
- added C68: 10n, Capacitor_SMD:C_0603_1608Metric, F.Cu at (222.7, -37.4)
- added C69: 100n, Capacitor_SMD:C_0603_1608Metric, F.Cu at (222.7, -34.9)
- added C7: 10u, Capacitor_SMD:C_0805_2012Metric, F.Cu at (250.1, -46.7)
- added C70: 220n, Capacitor_SMD:C_0603_1608Metric, F.Cu at (222.7, -32.4)
- added C71: 10u, Capacitor_SMD:C_0805_2012Metric, F.Cu at (250.1, -37.7)
- added C72: 100n, Capacitor_SMD:C_0603_1608Metric, F.Cu at (226.7, -49.9)
- added C73: 10n, Capacitor_SMD:C_0603_1608Metric, F.Cu at (226.7, -47.4)
- added C74: 47u, Capacitor_SMD:C_1206_3216Metric, F.Cu at (217.9, -32.8)
- added C75: 10p, Capacitor_SMD:C_0603_1608Metric, F.Cu at (226.7, -44.9)
- added C76: 100n, Capacitor_SMD:C_0603_1608Metric, F.Cu at (226.7, -42.4)
- added C77: 10u, Capacitor_SMD:C_0805_2012Metric, F.Cu at (250.1, -34.6)
- added C78: 10n, Capacitor_SMD:C_0603_1608Metric, F.Cu at (226.7, -39.9)
- added C79: 4u7, Capacitor_SMD:C_1206_3216Metric, F.Cu at (217.9, -29.4)
- added C8: 100n, Capacitor_SMD:C_0603_1608Metric, F.Cu at (222.7, -47.4)
- added C80: 4u7, Capacitor_SMD:C_1206_3216Metric, F.Cu at (217.9, -26.1)
- added C81: 4u7, Capacitor_SMD:C_1206_3216Metric, F.Cu at (217.9, -22.7)
- added C82: 4u7, Capacitor_SMD:C_1206_3216Metric, F.Cu at (217.9, -19.4)
- added C83: 4n7, Capacitor_SMD:C_0603_1608Metric, F.Cu at (226.7, -37.4)
- added C9: 4u7, Capacitor_SMD:C_1206_3216Metric, F.Cu at (217.9, -46.2)
- added D10: SS34, Diode_SMD:D_SMA, F.Cu at (246.0, -25.5)
- added D2: SS34, Diode_SMD:D_SMA, F.Cu at (246.0, -30.0)
- added J1: 550910374, magnode_footprints:CONN_MOLEX_02x15_55091-0374, F.Cu at (114.9, 70.8)
- added L2: 10u, magnode_footprints:ZEMS0850-100M_8.5x8.0mm, F.Cu at (242.3, -46.5)
- added L4: 10u, magnode_footprints:ZEMS0850-100M_8.5x8.0mm, F.Cu at (242.3, -37.0)
- added R12: 510k, Resistor_SMD:R_0603_1608Metric, F.Cu at (226.7, -34.9)
- added R13: 1k, Resistor_SMD:R_0603_1608Metric, F.Cu at (226.7, -32.4)
- added R14: 200k, Resistor_SMD:R_0603_1608Metric, F.Cu at (230.7, -49.9)
- added R16: 90k9, Resistor_SMD:R_1206_3216Metric, F.Cu at (230.8, -20.2)
- added R17: 100k, Resistor_SMD:R_0603_1608Metric, F.Cu at (230.7, -47.4)
- added R43: 75k, Resistor_SMD:R_0603_1608Metric, F.Cu at (230.7, -44.9)
- added R48: 200k, Resistor_SMD:R_0603_1608Metric, F.Cu at (230.7, -42.4)
- added R77: 10k, Resistor_SMD:R_0603_1608Metric, F.Cu at (256.3, -49.9)
- added R79: 10k, Resistor_SMD:R_0603_1608Metric, F.Cu at (256.3, -47.4)
- added R83: 39k, Resistor_SMD:R_0603_1608Metric, F.Cu at (230.7, -39.9)
- added R84: 12k, Resistor_SMD:R_0603_1608Metric, F.Cu at (230.7, -37.4)
- added R87: 100k, Resistor_SMD:R_0603_1608Metric, F.Cu at (230.7, -34.9)
- added R88: 330k, Resistor_SMD:R_0603_1608Metric, F.Cu at (230.7, -32.4)
- added R89: 10, Resistor_SMD:R_0603_1608Metric, F.Cu at (234.7, -49.9)
- added R90: 100k, Resistor_SMD:R_0603_1608Metric, F.Cu at (234.7, -47.4)
- added R92: 510k, Resistor_SMD:R_0603_1608Metric, F.Cu at (234.7, -44.9)
- added R93: 100k, Resistor_SMD:R_0603_1608Metric, F.Cu at (234.7, -42.4)
- added U11: TPS7A2033PDBVR, Package_TO_SOT_SMD:SOT-23-5, F.Cu at (239.3, -25.3)
- added U13: TPS7A4901DGNR, magnode_footprints:HVSSOP-8-1EP_3x3mm_P0.65mm_EP1.57x1.89mm, F.Cu at (224.4, -28.7)
- added U14: TPS7A3301RGWR, Package_DFN_QFN:Texas_RGW0020A_VQFN-20-1EP_5x5mm_P0.65mm_EP3.15x3.15mm, F.Cu at (224.4, -22.8)
- added U15: TPS63700DRCR, Package_SON:VSON-10-1EP_3x3mm_P0.5mm_EP1.2x2mm, F.Cu at (231.1, -24.1)
- added U2: LT3042xMSE, Package_SO:MSOP-10-1EP_3x3mm_P0.5mm_EP1.68x1.88mm, F.Cu at (245.5, -20.9)
- added U3: TPS61040DBV, Package_TO_SOT_SMD:SOT-23-5, F.Cu at (239.3, -29.9)
Connections:
- U10 pad 3: /POWER/5V_STEP_DOWN_IN -> Net-(U10-EN)
- U4 pad 10: unconnected-(U4-~{SRCLR}-Pad10) -> Net-(U4-~{SRCLR})
- U6 pad 10: unconnected-(U6-~{SRCLR}-Pad10) -> Net-(U6-~{SRCLR})

Commit message: ...
Parts:
- added C104: 100n, Capacitor_SMD:C_0402_1005Metric, F.Cu at (234.5, 141.1)
- added C105: 100n, Capacitor_SMD:C_0402_1005Metric, F.Cu at (234.5, 143.0)
- added C106: 100n, Capacitor_SMD:C_0402_1005Metric, F.Cu at (234.5, 145.0)
- added C24: 10u, Capacitor_SMD:C_0603_1608Metric, F.Cu at (229.7, 147.4)
- added J3: 550910374, magnode_footprints:CONN_MOLEX_02x15_55091-0374, F.Cu at (266.7, 114.4)
- added J5: Conn_Coaxial, Connector_Coaxial:U.FL_Hirose_U.FL-R-SMT-1_Vertical, F.Cu at (230.3, 143.1)
- added U20: MAX-M10S, RF_GPS:ublox_MAX, F.Cu at (208.1, 143.7)
Connections:
- J1 pad 22: +3V3D -> +3V3A
- J1 pad 23: +3V3A -> +3V3D
- U5 pad 37: /MCU_ESP32S3/GPS_UART_TX -> /GNSS/GPS_TX
- U5 pad 38: /MCU_ESP32S3/GPS_UART_RX -> /GNSS/GPS_RX

Commit message: clearing git
Parts:
- removed the J1 at (115.0, 70.0)
- removed the J1 at (114.9, 70.8)
- removed the J3 at (266.7, 114.4)
- removed the J3 at (115.0, 113.0)
- removed TP2: TestPoint, TestPoint:TestPoint_THTPad_1.0x1.0mm_Drill0.5mm
- added J1: 550910374, magnode_footprints:CONN_MOLEX_02x15_55091-0374, F.Cu at (120.0, 73.0)
- added J3: 550910374, magnode_footprints:CONN_MOLEX_02x15_55091-0374, F.Cu at (120.0, 118.0)
- moved R8 140.7 mm to (255.3, 116.3)
- moved R7 140.3 mm to (255.3, 113.8)
- moved R52 133.0 mm to (255.3, 99.7)
- moved R53 132.9 mm to (255.3, 102.2)
- moved H12 6.71 mm to (120.0, 134.0)
- moved H3 6.00 mm to (65.0, 102.0)
- moved H4 6.00 mm to (65.0, 134.0)
- moved H10 5.00 mm to (120.0, 89.0)
- moved H1 4.00 mm to (65.0, 57.0)
- moved H2 4.00 mm to (65.0, 89.0)
- moved H11 3.61 mm to (120.0, 102.0)
- moved H9 3.00 mm to (120.0, 57.0)
- moved C48 1.97 mm to (127.0, 87.4)
- moved C41 1.41 mm to (127.7, 99.0)
- moved C42 1.41 mm to (133.9, 101.6)
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Routing:
- net /DEVICE_DETECT_2: track 186.4 -> 0.00 mm, vias 1 -> 0
- net /MCU_ESP32S3/EN_SUPERCAP_CHARGE: track 84.9 -> 270.6 mm
- net /DEVICE_DETECT_1: track 116.3 -> 0.00 mm, vias 1 -> 0
- net unconnected-(U5-GPIO39-Pad31): track 0.00 -> 115.0 mm
- net +3V3A: track 161.0 -> 101.7 mm, vias 8 -> 6
- net +1V65: track 56.2 -> 1.00 mm, vias 3 -> 1
- net /RESET_2: track 97.2 -> 54.7 mm
- net /SET_2: track 90.4 -> 48.7 mm
- net /ADC_AD777x/AIN5+: track 34.4 -> 1.86 mm
- net /ADC_AD777x/AIN0+: track 33.7 -> 1.14 mm
- net /ADC_AD777x/AIN5-: track 34.1 -> 1.73 mm
- net +9VA: track 80.7 -> 112.8 mm, vias 4 -> 1
- net /ADC_AD777x/AIN4-: track 33.2 -> 1.48 mm
- net /ADC_AD777x/AIN4+: track 33.1 -> 1.36 mm
- net /ADC_AD777x/AIN0-: track 33.1 -> 1.59 mm
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Other:
- board text added: "Digital Board v2 Layer stack up: JLC0416H-7628 standard 1 oz, 0.5oz, 1.6mm For 90 Ohms USB lines"
- board text removed: "Digital Board v1 Layer stack up: JLC0416H-7628 standard 1 oz, 0.5oz, 1.6mm For 90 Ohms USB lines"
