File: hardware/pcb/Expension_card_design/magnetic_expension/schematics/sensor_set_reset_driver.kicad_sch (KiCad schematic)
At the start: 13 parts, among them Q1 D882, Q2 DMC3028LSD, Q3 B772, Q4 D882

Commit message: ...
Parts:
- renumbered R2 to R1, R3 to R2, R4 to R3, R5 to R4
Changed lines of the file:
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@@
 		(on_board yes)
 		(dnp no)
-		(property "Reference" "#PWR029"
+		(property "Reference" "#PWR019"
 			(at 110.49 130.81 0)
 			(effects
@@
 			(project ""
 				(path "/b5f9ef85-43f0-43d8-a1fd-ed489b1654c1/209adda1-10e4-4d62-92d8-b16a998ad2d8"
-					(reference "#PWR029")
+					(reference "#PWR019")
 					(unit 1)
 				)
@@
 		(on_board yes)
 		(dnp no)
-		(property "Reference" "R3"
+		(property "Reference" "R2"
 			(at 128.524 72.39 0)
 			(effects
@@
 			(project "magnetometer_node_mainboard"
 				(path "/b5f9ef85-43f0-43d8-a1fd-ed489b1654c1/209adda1-10e4-4d62-92d8-b16a998ad2d8"
-					(reference "R3")
+					(reference "R2")
 					(unit 1)
 				)
@@
 		(on_board yes)
 		(dnp no)
-		(property "Reference" "R5"
+		(property "Reference" "R4"
 			(at 104.14 110.49 90)
 			(effects
@@
 			(project ""
 				(path "/b5f9ef85-43f0-43d8-a1fd-ed489b1654c1/209adda1-10e4-4d62-92d8-b16a998ad2d8"
-					(reference "R5")
+					(reference "R4")
 					(unit 1)
 				)
@@
 		(on_board yes)
 		(dnp no)
-		(property "Reference" "R4"
+		(property "Reference" "R3"
 			(at 128.524 99.06 0)
 			(effects
@@
 			(project ""
 				(path "/b5f9ef85-43f0-43d8-a1fd-ed489b1654c1/209adda1-10e4-4d62-92d8-b16a998ad2d8"
-					(reference "R4")
+					(reference "R3")
 					(unit 1)
 				)
@@
 		(dnp no)
 		(fields_autoplaced yes)
-		(property "Reference" "#PWR023"
+		(property "Reference" "#PWR013"
 			(at 203.2 69.85 0)
 			(effects
@@
 			(project ""
 				(path "/b5f9ef85-43f0-43d8-a1fd-ed489b1654c1/209adda1-10e4-4d62-92d8-b16a998ad2d8"
-					(reference "#PWR023")
+					(reference "#PWR013")
 					(unit 1)
 				)
@@
 		(on_board yes)
 		(dnp no)
-		(property "Reference" "#PWR026"
+		(property "Reference" "#PWR016"
 			(at 138.43 104.14 0)
 			(effects
@@
 			(project "magnetometer_node_mainboard"
 				(path "/b5f9ef85-43f0-43d8-a1fd-ed489b1654c1/209adda1-10e4-4d62-92d8-b16a998ad2d8"
-					(reference "#PWR026")
+					(reference "#PWR016")
 					(unit 1)
 				)
@@
 		(on_board yes)
 		(dnp no)
-		(property "Reference" "R2"
+		(property "Reference" "R1"
 			(at 196.85 64.77 90)
 			(effects
@@
 			(project "magnetometer_node_mainboard"
 				(path "/b5f9ef85-43f0-43d8-a1fd-ed489b1654c1/209adda1-10e4-4d62-92d8-b16a998ad2d8"
-					(reference "R2")
+					(reference "R1")
 					(unit 1)
 				)
@@
 		(on_board yes)
 		(dnp no)
-		(property "Reference" "#PWR025"
+		(property "Reference" "#PWR015"
 			(at 185.42 82.55 0)
 			(effects
@@
 			(project "magnetic_expension"
 				(path "/b5f9ef85-43f0-43d8-a1fd-ed489b1654c1/209adda1-10e4-4d62-92d8-b16a998ad2d8"
-					(reference "#PWR025")
+					(reference "#PWR015")
 					(unit 1)
 				)
@@
 		(on_board yes)
 		(dnp no)
-		(property "Reference" "#PWR024"
+		(property "Reference" "#PWR014"
 			(at 175.26 82.55 0)
 			(effects
@@
 			(project "magnetometer_node_mainboard"
 				(path "/b5f9ef85-43f0-43d8-a1fd-ed489b1654c1/209adda1-10e4-4d62-92d8-b16a998ad2d8"
-					(reference "#PWR024")
+					(reference "#PWR014")
 					(unit 1)
 				)
@@
 		(on_board yes)
 		(dnp no)
-		(property "Reference" "#PWR028"
+		(property "Reference" "#PWR018"
 			(at 167.64 124.46 0)
 			(effects
@@
 			(project "magnetometer_node_mainboard"
 				(path "/b5f9ef85-43f0-43d8-a1fd-ed489b1654c1/209adda1-10e4-4d62-92d8-b16a998ad2d8"
-					(reference "#PWR028")
+					(reference "#PWR018")
 					(unit 1)
 				)
@@
 		(on_board yes)
 		(dnp no)
-		(property "Reference" "#PWR027"
+		(property "Reference" "#PWR017"
 			(at 127 124.46 0)
 			(effects
@@
 			(project "magnetometer_node_mainboard"
 				(path "/b5f9ef85-43f0-43d8-a1fd-ed489b1654c1/209adda1-10e4-4d62-92d8-b16a998ad2d8"
-					(reference "#PWR027")
-					(unit 1)
-				)
+					(reference "#PWR017")
+					(unit 1)
+				)
