File: hardware/pcb/Expension_card_design/magnetic_expension/schematics/Bridge_offset.kicad_sch (KiCad schematic)
At the start: 20 parts, among them U10 OPA4197xPW, U11 THS4551IRGTR, U12 DAC8571IDGK, U8 THS4551IRGTR, U9 OPA4197xPW

Commit message: clearing git
Parts:
- removed R43, R44: 1k, symbol Device:R
- removed U10, U9: OPA4197xPW, Package_SO:TSSOP-14_4.4x5mm_P0.65mm, symbol Amplifier_Operational:OPA4197xPW
- added C38, C41, C42, C45: 1u, symbol Device:C
- added C39, C43, C49: 1n, Capacitor_SMD:C_0603_1608Metric, symbol Device:C
- added C44, C50: 220n, Capacitor_SMD:C_0603_1608Metric, symbol Device:C
- added C46, C52: 100n, Capacitor_SMD:C_0603_1608Metric, symbol Device:C
- added C47, C48, C51, C53: 4u7, Capacitor_SMD:C_1206_3216Metric, symbol Device:C
- added R53, R55, R56, R57: 1k, Resistor_SMD:R_0603_1608Metric, symbol Device:R
- added R54: 20k, Resistor_SMD:R_0603_1608Metric, symbol Device:R
- added RN10, RN11, RN14, RN15, RN6, RN7: 5k, Resistor_SMD:R_Array_Convex_2x0603, symbol Device:R_Pack02_Split
- added RN12, RN4, RN8: 20k, Resistor_SMD:R_Array_Convex_2x0603, symbol Device:R_Pack02_Split
- added RN13, RN5, RN9: 10k, Resistor_SMD:R_Array_Convex_4x0603, symbol Device:R_Pack04_Split
- added U11, U12, U14: THS4551IRGTR, magnode_footprints:VQFN-16-1EP_3x3mm_P0.5mm_EP1.68x1.68mm, symbol magnode_symbols:THS4551IRGTR
- added U13: DAC7678SPWR, Package_SO:TSSOP-16_4.4x5mm_P0.65mm, symbol magnode_symbols:DAC7678SPWR
- renumbered C23 to C40, R47 to R41, R48 to R42, R53 to R43, R51 to R44, R50 to R45, R49 to R46, R45 to R47, R52 to R48, R54 to R49, R46 to R50, R27 to R51, R29 to R52, U12 to U10, U11 to U8, U8 to U9
Connections:
- net +1V65B: now also R41.2, U11.9 (V_{OCM}), U12.9 (V_{OCM}), U14.9 (V_{OCM})
- net +3V3A: now also C46.1, C47.1, C52.1, C53.1, U11.12 (~{PD}), U11.5 (V_{S+}), U11.6 (V_{S+}), U11.7 (V_{S+}), U11.8 (V_{S+}), U12.12 (~{PD}), U12.5 (V_{S+}), U12.6 (V_{S+}), U12.7 (V_{S+}), U12.8 (V_{S+}), U13.2 (ADDR0), U13.3 (AV_{DD}), U13.8 (V_{REFIN}/V_{REFOUT}), U14.12 (~{PD}), U14.5 (V_{S+}), U14.6 (V_{S+}), U14.7 (V_{S+}), U14.8 (V_{S+})
- net COMP_POS_FB: now also R41.1; no longer R41.2
- net GND: now also C38.2, C41.2, C42.2, C45.2, C46.2, C47.2, C48.2, C51.2, C52.2, C53.2, U11.13 (V_{S-}), U11.14 (V_{S-}), U11.15 (V_{S-}), U11.16 (V_{S-}), U11.17 (EP), U12.13 (V_{S-}), U12.14 (V_{S-}), U12.15 (V_{S-}), U12.16 (V_{S-}), U12.17 (EP), U13.14 (GND), U14.13 (V_{S-}), U14.14 (V_{S-}), U14.15 (V_{S-}), U14.16 (V_{S-}), U14.17 (EP); no longer R41.1
- net X_CONN+: now also C50.2, R57.2
- net X_CONN-: now also C50.1, R56.2
- net Y_CONN+: now also C44.2, R55.2
- net Y_CONN-: now also C44.1, R53.2
- net COMP+ renamed V_{COMP}+
- net COMP- renamed V_{COMP}-
- net COMP_NEG_FB: no longer names the net of R47.2, R50.1, U8.3 (-)
- net DAC_COMP_OUT renamed V_{DAC}
- net SUM_NEG_FB: no longer names the net of R46.2, R48.2, R49.1, U9.3 (-)
- net SUM_POS_FB: no longer names the net of R43.1, R44.2, R45.2, U9.2 (+)
- net X_INA_OUT_F+ renamed V_{IN}+
- net X_INA_OUT_F- renamed V_{IN}-
- net X_INA_PRE_AAF+ renamed V_{OUT}-
- net V_{OUT}-: no longer R51.1
- net X_INA_PRE_AAF- renamed V_{OUT}+
- net V_{OUT}+: no longer R52.1
- new net: R54.1, U13.9 (~{CLR})
- new net +5VA: R54.2
- new net DAC_B_OUTA: RN5.8 (R1.2), U13.4 (V_{OUT}A)
- new net DAC_B_OUTB: RN5.6 (R3.2), U13.13 (V_{OUT}B)
- new net DAC_B_OUTC: RN9.8 (R1.2), U13.5 (V_{OUT}C)
- new net DAC_B_OUTD: RN9.6 (R3.2), U13.12 (V_{OUT}D)
- new net DAC_B_OUTE: RN13.8 (R1.2), U13.6 (V_{OUT}E)
- new net DAC_B_OUTF: RN13.6 (R3.2), U13.11 (V_{OUT}F)
- new net I2C.SCL: U13.16 (SCL)
- new net I2C.SDA: U13.15 (SDA)
- new net X_COMP_FILT+: C38.1, RN5.1 (R1.1), RN5.7 (R2.2)
- new net X_COMP_FILT-: C41.1, RN5.3 (R3.1), RN5.5 (R4.2)
- new net X_INA_FILT+: C39.1, RN6.2 (R2.1), RN7.3 (R2.2)
- new net X_INA_FILT-: C39.2, RN6.1 (R1.1), RN7.4 (R1.2)
- new net X_INA_OUT+: RN6.3 (R2.2)
- new net X_INA_OUT-: RN6.4 (R1.2)
- new net X_SUM_FB+: RN4.3 (R2.2), RN5.4 (R4.1), RN7.2 (R2.1), U11.3 (-)
- new net X_SUM_FB-: RN4.4 (R1.2), RN5.2 (R2.1), RN7.1 (R1.1), U11.2 (+)
- new net X_SUM_OUT+: R52.1, RN4.2 (R2.1), U11.10 (+)
- new net X_SUM_OUT-: R51.1, RN4.1 (R1.1), U11.11 (-)
- new net Y_COMP_FILT+: C42.1, RN9.1 (R1.1), RN9.7 (R2.2)
- new net Y_COMP_FILT-: C45.1, RN9.3 (R3.1), RN9.5 (R4.2)
- new net Y_INA_FILT+: C43.1, RN10.2 (R2.1), RN11.3 (R2.2)
- new net Y_INA_FILT-: C43.2, RN10.1 (R1.1), RN11.4 (R1.2)
- new net Y_INA_OUT+: RN10.3 (R2.2)
- new net Y_INA_OUT-: RN10.4 (R1.2)
- new net Y_SUM_FB+: RN11.2 (R2.1), RN8.3 (R2.2), RN9.4 (R4.1), U12.3 (-)
- new net Y_SUM_FB-: RN11.1 (R1.1), RN8.4 (R1.2), RN9.2 (R2.1), U12.2 (+)
- new net Y_SUM_OUT+: R55.1, RN8.2 (R2.1), U12.10 (+)
- new net Y_SUM_OUT-: R53.1, RN8.1 (R1.1), U12.11 (-)
- new net Z_COMP_FILT+: C48.1, RN13.1 (R1.1), RN13.7 (R2.2)
- new net Z_COMP_FILT-: C51.1, RN13.3 (R3.1), RN13.5 (R4.2)
- new net Z_INA_FILT+: C49.1, RN14.2 (R2.1), RN15.3 (R2.2)
- new net Z_INA_FILT-: C49.2, RN14.1 (R1.1), RN15.4 (R1.2)
- new net Z_INA_OUT+: RN14.3 (R2.2)
- new net Z_INA_OUT-: RN14.4 (R1.2)
- new net Z_SUM_FB+: RN12.3 (R2.2), RN13.4 (R4.1), RN15.2 (R2.1), U14.3 (-)
- new net Z_SUM_FB-: RN12.4 (R1.2), RN13.2 (R2.1), RN15.1 (R1.1), U14.2 (+)
- new net Z_SUM_OUT+: R57.1, RN12.2 (R2.1), U14.10 (+)
- new net Z_SUM_OUT-: R56.1, RN12.1 (R1.1), U14.11 (-)
- no-connect marks 4 -> 13
Other:
- note added: "Bridge DC offset: -60mV to +30mV INA Gain = 61 Offset after INA: -60mV * 61 to +30mV * 61 = 3.66V to 1.83V From the sensors measured the heighest was -15mV If INA gain = 51 then offset: -60mV * 51 to +30mV * 51 = 3.06V to 1.53V Total gain needed: 125 G1 = 125/51 = 2.45 If we keep RF = 20k R_{in} = RF/G1 = 20k/2.45 = 8k2 If I use 2x 3.9k then I get G1 = 2.56 total gain: 51 * 2.56 = 130.56 With 8x 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"
- note added: "DAC B for Bridge offset compensation"
- note added: "Filter 2: prevent DAC noise and step fc = 1 / (2*pi*10k*1uF) ≈ 15.9 Hz"
- note added: "Filter 3: Shunt high-frequency differential noise before the THS4551 summing stage fc = 1 / (2*pi*(5k + 5k)*1nF) ≈ 64 kHz"
- note added: "Filter 4: Anti-Aliasing with ADC at 1kSPS fc = 1 / (2*pi*(1k + 1k)*220nF) ≈ 362 Hz"
- note added: "V_{OUT}+ - V_{OUT}- = G_{1} * (V_{IN}+ - V_{IN}- ) + G_{2} * (V_{DAC B} - V_{DAC A}) V_{DAC} goes from 0 to 3.3V G_{1} = RF / R_{in} G_{2} = RF / (R_{DAC}1 + R_{DAC}2) G_{1} = 20k / (5k + 5k) = 2 G_{2} = 20k / (10k + 10k) = 1"
- note added: "V_{OUT}+ - V_{OUT}- = V_{IN}+ - V_{IN}- + 0.1 * (1.65 V - V_{DAC})"
- moved on the sheet: C40, R41, R42, R43, R44, R45, R46, R47, R48, R49, R50, R51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
