File: hardware/pcb/Expension_card_design/magnetic_expension/schematics/CONN.kicad_sch (KiCad schematic)
At the start: 8 parts, among them J1 550910374

Commit message: Work in progress rev2
Parts:
- removed J1: 550910374, magnode_footprints:CONN_MOLEX_02x15_55091-0374, symbol magnode_symbols:55091-0374
- removed R19: 10k, Resistor_SMD:R_0603_1608Metric, symbol Device:R
- removed R7, R8: 100k, Resistor_SMD:R_0603_1608Metric, symbol Device:R
- added J2: 528850374, magnode_footprints:CONN_MOLEX_02x15_52885-0374, symbol magnode_symbols:52885-0374
- added R1: 20k, Resistor_SMD:R_0603_1608Metric, symbol Device:R
Connections:
- net +18V: now also J2.18
- net +1V65: now also J2.17
- net +3V3A: now also J2.22
- net +3V3D: now also J2.23
- net +5VA: now also J2.19
- net +9VA: now also J2.21
- net -5VA: now also J2.20
- net DEVICE_DETECT: now also J2.2, R1.1
- net GND: now also J2.1, J2.12, J2.15, J2.16, J2.24, J2.27, J2.3, J2.30, J2.6, J2.9, J2.P1, J2.P2, R1.2
- net I2C.SCL: now also J2.28
- net I2C.SDA: now also J2.29
- net SENSOR_RESET_CTRL: now also J2.26
- net SENSOR_SET_CTRL: now also J2.25
- new net X_INA_OUT+: J2.10
- new net X_INA_OUT-: J2.11
- new net Y_INA_OUT+: J2.7
- new net Y_INA_OUT-: J2.8
- new net Z_INA_OUT+: J2.4
- new net Z_INA_OUT-: J2.5
Other:
- note removed: "Mainboard: 550910274 / 55091-0274 -> 550910374 / 55091-0374 Add-on boards: 528850274 / 52885-0274 -> 528850374 / 52885-0374"

Commit message: ...
Parts:
- renumbered J2 to J1, R1 to R25
Changed lines of the file:
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@@
 		(on_board yes)
 		(dnp no)
-		(property "Reference" "#PWR04"
+		(property "Reference" "#PWR053"
 			(at 102.87 93.98 0)
 			(effects
@@
 			(project "magnetic_expension"
 				(path "/b5f9ef85-43f0-43d8-a1fd-ed489b1654c1/0a13a391-065e-4b36-b802-09a3f1325672"
-					(reference "#PWR04")
+					(reference "#PWR053")
 					(unit 1)
 				)
@@
 		(on_board yes)
 		(dnp no)
-		(property "Reference" "R1"
+		(property "Reference" "R25"
 			(at 184.658 73.66 0)
 			(effects
@@
 			(project "magnetic_expension"
 				(path "/b5f9ef85-43f0-43d8-a1fd-ed489b1654c1/0a13a391-065e-4b36-b802-09a3f1325672"
-					(reference "R1")
+					(reference "R25")
 					(unit 1)
 				)
@@
 		(on_board yes)
 		(dnp no)
-		(property "Reference" "#PWR05"
+		(property "Reference" "#PWR049"
 			(at 128.27 83.82 0)
 			(effects
@@
 			(project "magnetic_expension"
 				(path "/b5f9ef85-43f0-43d8-a1fd-ed489b1654c1/0a13a391-065e-4b36-b802-09a3f1325672"
-					(reference "#PWR05")
+					(reference "#PWR049")
 					(unit 1)
 				)
@@
 		(on_board yes)
 		(dnp no)
-		(property "Reference" "#PWR08"
+		(property "Reference" "#PWR052"
 			(at 109.22 90.805 0)
 			(effects
@@
 			(project "magnetic_expension"
 				(path "/b5f9ef85-43f0-43d8-a1fd-ed489b1654c1/0a13a391-065e-4b36-b802-09a3f1325672"
-					(reference "#PWR08")
+					(reference "#PWR052")
 					(unit 1)
 				)
@@
 		(on_board yes)
 		(dnp no)
-		(property "Reference" "J2"
+		(property "Reference" "J1"
 			(at 149.86 67.31 0)
 			(effects
@@
 			(project "magnetic_expension"
 				(path "/b5f9ef85-43f0-43d8-a1fd-ed489b1654c1/0a13a391-065e-4b36-b802-09a3f1325672"
-					(reference "J2")
+					(reference "J1")
 					(unit 1)
 				)
@@
 		(on_board yes)
 		(dnp no)
-		(property "Reference" "#PWR010"
+		(property "Reference" "#PWR056"
 			(at 148.59 124.46 0)
 			(effects
@@
 			(project "magnetic_expension"
 				(path "/b5f9ef85-43f0-43d8-a1fd-ed489b1654c1/0a13a391-065e-4b36-b802-09a3f1325672"
-					(reference "#PWR010")
+					(reference "#PWR056")
 					(unit 1)
 				)
@@
 		(on_board yes)
 		(dnp no)
-		(property "Reference" "#PWR087"
+		(property "Reference" "#PWR054"
 			(at 96.52 96.52 0)
 			(effects
@@
 			(project "magnetic_expension"
 				(path "/b5f9ef85-43f0-43d8-a1fd-ed489b1654c1/0a13a391-065e-4b36-b802-09a3f1325672"
-					(reference "#PWR087")
+					(reference "#PWR054")
 					(unit 1)
 				)
@@
 		(on_board yes)
 		(dnp no)
-		(property "Reference" "#PWR06"
+		(property "Reference" "#PWR050"
 			(at 121.92 86.36 0)
 			(effects
@@
 			(project "magnetic_expension"
 				(path "/b5f9ef85-43f0-43d8-a1fd-ed489b1654c1/0a13a391-065e-4b36-b802-09a3f1325672"
-					(reference "#PWR06")
+					(reference "#PWR050")
 					(unit 1)
 				)
@@
 		(on_board yes)
 		(dnp no)
-		(property "Reference" "#PWR09"
+		(property "Reference" "#PWR057"
 			(at 161.29 124.46 0)
 			(effects
@@
 			(project "magnetic_expension"
 				(path "/b5f9ef85-43f0-43d8-a1fd-ed489b1654c1/0a13a391-065e-4b36-b802-09a3f1325672"
-					(reference "#PWR09")
+					(reference "#PWR057")
 					(unit 1)
 				)
@@
 		(on_board yes)
 		(dnp no)
-		(property "Reference" "#PWR03"
+		(property "Reference" "#PWR048"
 			(at 134.62 81.28 0)
 			(effects
@@
 			(project "magnetic_expension"
 				(path "/b5f9ef85-43f0-43d8-a1fd-ed489b1654c1/0a13a391-065e-4b36-b802-09a3f1325672"
-					(reference "#PWR03")
+					(reference "#PWR048")
 					(unit 1)
 				)
@@
 		(on_board yes)
 		(dnp no)
-		(property "Reference" "#PWR07"
+		(property "Reference" "#PWR051"
 			(at 115.57 88.9 0)
 			(effects
@@
 			(project "magnetic_expension"
 				(path "/b5f9ef85-43f0-43d8-a1fd-ed489b1654c1/0a13a391-065e-4b36-b802-09a3f1325672"
-					(reference "#PWR07")
+					(reference "#PWR051")
 					(unit 1)
 				)
@@
 		(on_board yes)
 		(dnp no)
-		(property "Reference" "#PWR01"
+		(property "Reference" "#PWR047"
 			(at 196.85 76.2 0)
 			(effects
@@
 			(project "magnetic_expension"
 				(path "/b5f9ef85-43f0-43d8-a1fd-ed489b1654c1/0a13a391-065e-4b36-b802-09a3f1325672"
-					(reference "#PWR01")
+					(reference "#PWR047")
 					(unit 1)
 				)
@@
 		(on_board yes)
 		(dnp no)
-		(property "Reference" "#PWR088"
+		(property "Reference" "#PWR055"
 			(at 138.43 124.46 0)
 			(effects
@@
 			(project "magnetic_expension"
 				(path "/b5f9ef85-43f0-43d8-a1fd-ed489b1654c1/0a13a391-065e-4b36-b802-09a3f1325672"
-					(reference "#PWR088")
-					(unit 1)
-				)
+					(reference "#PWR055")
+					(unit 1)
+				)

Commit message: clearing git
Connections:
- net X_INA_OUT+ renamed X_CONN+
- net X_INA_OUT- renamed X_CONN-
- net Y_INA_OUT+ renamed Y_CONN+
- net Y_INA_OUT- renamed Y_CONN-
- net Z_INA_OUT+ renamed Z_CONN+
- net Z_INA_OUT- renamed Z_CONN-
Changed lines of the file:
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@@
+		)
+	)
+	(hierarchical_label "X_CONN-"
+		(shape output)
+		(at 167.64 100.33 0)
+		(effects
+			(font
+				(size 1.27 1.27)
+			)
+			(justify left)
+		)
+	)
+	(hierarchical_label "Y_CONN-"
+		(shape output)
+		(at 167.64 92.71 0)
+		(effects
+			(font
+				(size 1.27 1.27)
+			)
+			(justify left)
 		)
 	)
@@
 		)
 	)
-	(hierarchical_label "Z_INA_OUT-"
-		(shape input)
+	(hierarchical_label "X_CONN+"
+		(shape output)
+		(at 167.64 97.79 0)
+		(effects
+			(font
+				(size 1.27 1.27)
+			)
+			(justify left)
+		)
+	)
+	(hierarchical_label "Z_CONN-"
+		(shape output)
 		(at 167.64 85.09 0)
 		(effects
@@
 		)
 	)
-	(hierarchical_label "Y_INA_OUT+"
-		(shape input)
+	(hierarchical_label "Y_CONN+"
+		(shape output)
 		(at 167.64 90.17 0)
 		(effects
@@
 		)
 	)
-	(hierarchical_label "X_INA_OUT+"
-		(shape input)
-		(at 167.64 97.79 0)
-		(effects
-			(font
-				(size 1.27 1.27)
-			)
-			(justify left)
-		)
-	)
-	(hierarchical_label "Y_INA_OUT-"
-		(shape input)
-		(at 167.64 92.71 0)
-		(effects
-			(font
-				(size 1.27 1.27)
-			)
-			(justify left)
-		)
-	)
-	(hierarchical_label "Z_INA_OUT+"
-		(shape input)
+	(hierarchical_label "Z_CONN+"
+		(shape output)
 		(at 167.64 82.55 0)
-		(effects
-			(font
-				(size 1.27 1.27)
-			)
-			(justify left)
-		)
-	)
-	(hierarchical_label "X_INA_OUT-"
-		(shape input)
-		(at 167.64 100.33 0)
 		(effects
 			(font
@@
 			)
 		)
+		(property "Sim.Enable" ""
+			(at 209.55 90.17 0)
+			(effects
+				(font
+					(size 1.27 1.27)
+				)
+				(hide yes)
+			)
+		)
 		(instances
 			(project "magnetic_expension"
@@
 			)
 		)
+		(property "Sim.Enable" ""
+			(at 209.55 95.25 0)
+			(effects
+				(font
+					(size 1.27 1.27)
+				)
+				(hide yes)
+			)
+		)
 		(instances
 			(project "magnetic_expension"
@@
 		)
 		(property "LCSC" "C4184"
+			(at 187.96 73.66 0)
+			(effects
+				(font
+					(size 1.27 1.27)
+				)
+				(hide yes)
+			)
+		)
+		(property "Sim.Enable" ""
 			(at 187.96 73.66 0)
 			(effects
@@
 			)
 		)
+		(property "Sim.Enable" ""
+			(at 149.86 92.71 0)
+			(effects
+				(font
+					(size 1.27 1.27)
+				)
+				(hide yes)
+			)
+		)
 		(pin "15"
 		)
@@
 			)
 		)
+		(property "Sim.Enable" ""
+			(at 209.55 105.41 90)
+			(effects
+				(font
+					(size 1.27 1.27)
+				)
+				(hide yes)
+			)
+		)
 		(instances
 			(project "magnetic_expension"
@@
 			(at 209.55 100.33 0)
 			(effects
+				(font
+					(size 1.27 1.27)
+				)
+				(hide yes)
+			)
+		)
+		(property "Sim.Enable" ""
+			(at 209.55 100.33 0)
+			(effects
