File: hardware/pcb/Expension_card_design/magnetic_expension/schematics/analog_frontend_ina851.kicad_sch (KiCad schematic)
At the start: 27 parts, among them U5 INA851RGTR, U6 INA851RGTR, U7 INA851RGTR

Commit message: ADC_Fixed
Parts:
- added C35, C36, C37: 100n, Capacitor_SMD:C_0603_1608Metric, symbol Device:C
- added R35, R36, R37, R38, R39, R40: 48,7, Resistor_SMD:R_0603_1608Metric, symbol Device:R
Connections:
- net BR_X+: now also R36.1; no longer U5.1 (IN-)
- net BR_X-: now also R35.1; no longer U5.4 (IN+)
- net BR_Y+: now also R37.1; no longer U7.1 (IN-)
- net BR_Y-: now also R38.1; no longer U7.4 (IN+)
- net BR_Z+: now also R39.1; no longer U6.1 (IN-)
- net BR_Z-: now also R40.1; no longer U6.4 (IN+)
- new net BR_FTL_X+: C35.1, C36.1, C37.1, R36.2, R37.2, R39.2, U5.1 (IN-), U6.1 (IN-), U7.1 (IN-)
- new net BR_FTL_X-: C35.2, C36.2, C37.2, R35.2, R38.2, R40.2, U5.4 (IN+), U6.4 (IN+), U7.4 (IN+)

Commit message: Work in progress rev2
Changed lines of the file:
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@@
 		)
 		(property "Value" "-5VA"
-			(at 81.28 101.6 0)
+			(at 81.28 101.854 0)
 			(effects
 				(font

Commit message: ...
Parts:
- removed C18, C23, C28: 220n, Capacitor_SMD:C_0603_1608Metric, symbol Device:C
- removed R17, R19, R20, R22, R23, R25: 1k, Resistor_SMD:R_0603_1608Metric, symbol Device:R
- added C29, C35, C38: 1n, Capacitor_SMD:C_0603_1608Metric, symbol Device:C
- added R32, R34, R37, R39, R41, R42: 100, Resistor_SMD:R_0603_1608Metric, symbol Device:R
- renumbered C16 to C20, C17 to C21, C35 to C22, C19 to C24, C20 to C25, C21 to C26, C22 to C27, C37 to C28, C24 to C30, C25 to C31, C26 to C32, C27 to C33, C36 to C34, C29 to C36, C30 to C37, R36 to R26, R18 to R28, R35 to R30, R39 to R31, R21 to R33, R40 to R35, R37 to R36, R24 to R38, R38 to R40
Connections:
- net X_INA_PRE_AAF+ is gone; now on net X_INA_OUT+: U5.11 (OUT+)
- net X_INA_PRE_AAF- is gone; now on net X_INA_OUT-: U5.10 (OUT-)
- net Y_INA_PRE_AAF+ is gone; now on net Y_INA_OUT+: U7.11 (OUT+)
- net Y_INA_PRE_AAF- is gone; now on net Y_INA_OUT-: U7.10 (OUT-)
- net Z_INA_PRE_AAF+ is gone; now on net Z_INA_OUT+: U6.11 (OUT+)
- net Z_INA_PRE_AAF- is gone; now on net Z_INA_OUT-: U6.10 (OUT-)
- net X_INA_OUT+: now also R41.1
- net X_INA_OUT-: now also R42.1
- net Y_INA_OUT+: now also R37.1
- net Y_INA_OUT-: now also R39.1
- net Z_INA_OUT+: now also R32.1
- net Z_INA_OUT-: now also R34.1
- new net X_INA_OUT_F+: C38.2, R41.2
- new net X_INA_OUT_F-: C38.1, R42.2
- new net Y_INA_OUT_F+: C35.2, R37.2
- new net Y_INA_OUT_F-: C35.1, R39.2
- new net Z_INA_OUT_F+: C29.2, R32.2
- new net Z_INA_OUT_F-: C29.1, R34.2
Other:
- moved on the sheet: C22, R26, R30

Commit message: clearing git
Parts:
- removed C29, C35, C38: 1n, Capacitor_SMD:C_0603_1608Metric, symbol Device:C
- removed R32, R34, R37, R39, R41, R42: 100, Resistor_SMD:R_0603_1608Metric, symbol Device:R
- C22, C28, C34: value 100n -> 10n; LCSC C14663 -> (none)
- R26, R30, R31, R35, R36, R40: value 48,7 -> 49.9; LCSC C2692820 -> (none)
- R28, R33, R38: value 48,7 -> 100; LCSC C2692820 -> (none)
Connections:
- net X_RG+: now also R28.2; no longer R28.1
- net X_RG-: now also R28.1; no longer R28.2
- net Y_RG+: now also R38.2; no longer R38.1
- net Y_RG-: now also R38.1; no longer R38.2
- net Z_RG+: now also R33.2; no longer R33.1
- net Z_RG-: now also R33.1; no longer R33.2
- net +5VA renamed +9V_INA
Other:
- note added: "Filter 1: attenuate RF and high-frequency differential noise before the INA851 fc = 1 / (2*pi*(49.9 + 49.9)*1nF) ≈ 159 kHz"
