File: hardware/pcb/Expension_card_design/magnetic_expension/schematics/sensor_hmc100x_3axis.kicad_sch (KiCad schematic)
At the start: 6 parts, among them U1 HMC1001-RC, U2 HMC1002-TR

Commit message: Backup avant deletion offset/dac
Parts:
- U1, U2: now fitted
Changed lines of the file:
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@@
 		(in_bom yes)
 		(on_board yes)
-		(dnp yes)
+		(dnp no)
 		(fields_autoplaced yes)
 		(property "Reference" "U2"
@@
 		(in_bom yes)
 		(on_board yes)
-		(dnp yes)
+		(dnp no)
 		(fields_autoplaced yes)
 		(property "Reference" "U1"

Commit message: clearing git
Connections:
- net +9VA renamed +9V_BRIDGE
Other:
- note removed: "bypass cap"
