File: hardware/pcb/Expension_card_design/magnetic_expension/schematics/sensor_offset_drivers.kicad_sch (KiCad schematic)
At the start: 31 parts, among them Q10 B772, Q5 D882, Q6 B772, Q7 D882, Q8 B772, Q9 D882, U3 LM324DT, U4 MCP4728

Commit message: ADC_Fixed
Parts:
- removed U3: LM324DT, Package_SO:SOIC-14_3.9x8.7mm_P1.27mm, symbol Amplifier_Operational:LM324
- removed U4: MCP4728, Package_SO:MSOP-10_3x3mm_P0.5mm, symbol Analog_DAC:MCP4728
- added C32, C33: 4u7, Capacitor_SMD:C_1206_3216Metric, symbol Device:C
- added C34: 100n, Capacitor_SMD:C_0603_1608Metric, symbol Device:C
- added R27: 20k, Resistor_SMD:R_0603_1608Metric, symbol Device:R
- added R28: 10, Resistor_SMD:R_0603_1608Metric, symbol Device:R
- added R29: 22k, Resistor_SMD:R_0603_1608Metric, symbol Device:R
- added R30, R31, R33: 200, Resistor_SMD:R_1206_3216Metric, symbol Device:R
- added R32, R34: 470, Resistor_SMD:R_0603_1608Metric, symbol Device:R
- added U3: DAC7678SPWR, Package_SO:TSSOP-16_4.4x5mm_P0.65mm, symbol magnode_symbols:DAC7678SPWR
- added U8: OPA4197xPW, Package_SO:TSSOP-14_4.4x5mm_P0.65mm, symbol Amplifier_Operational:OPA4197xPW
- C11, C12, C13, C14, C15, C9: value 10u -> 4u7; footprint Capacitor_SMD:C_0805_2012Metric -> Capacitor_SMD:C_1206_3216Metric; LCSC C15850 -> C29823
- R10, R9: value 4k7 -> 3k3; footprint Resistor_SMD:R_0603_1608Metric -> (none); LCSC C23162 -> (none)
- R11, R14, R15: value 100 -> 22k; LCSC C22775 -> (none)
- R12, R6, R7: value 100 -> 470; LCSC C22775 -> (none)
- R13, R16: value 20 -> 22k; footprint Resistor_SMD:R_1206_3216Metric -> Resistor_SMD:R_0603_1608Metric; LCSC C17955 -> (none)
- R8: value 20 -> 470; footprint Resistor_SMD:R_1206_3216Metric -> Resistor_SMD:R_0603_1608Metric; LCSC C17955 -> (none)
Connections:
- net DAC_OUT_Z is gone; now on net OFF_Z_INN: RN3.4
- net +1V65: now also U8.12 (+)
- net +5VA: now also R27.2, R28.1, U8.4 (V+)
- net -5VA: now also U8.11 (V-)
- net 1V65_FB: now also U8.13 (-), U8.14
- net GND: now also C11.2, C12.2, C13.2, C14.2, C15.2, C9.2, C32.2, C33.2, C34.2, U3.14 (GND), U3.2 (ADDR0)
- net I2C.SCL: now also U3.16 (SCL)
- net I2C.SDA: now also U3.15 (SDA)
- net OFFSET_X+: now also R30.2; no longer C11.2, R8.2
- net OFFSET_Y+: now also R31.2; no longer C14.2, R13.2
- net OFFSET_Z+: now also RN3.5, R33.2; no longer C15.2, R16.2, RN3.7
- net OFF_X_BN: now also R15.2
- net OFF_X_BP: now also R29.2
- net OFF_X_DRV: now also U8.1
- net OFF_X_INN: now also U8.2 (-)
- net OFF_X_INP: now also U8.3 (+)
- net OFF_X_SENSE_P: now also R15.1, R29.1, R30.1; no longer C9.2, R8.1
- net OFF_Y_BN: now also R8.2
- net OFF_Y_BP: now also R13.2, R32.2; no longer R12.2
- net OFF_Y_DRV: now also R8.1, R32.1, U8.7; no longer R11.1, R12.1
- net OFF_Y_INN: now also C12.1, U8.6 (-); no longer C14.1
- net OFF_Y_INP: now also C13.1, U8.5 (+); no longer C12.1
- net OFF_Y_SENSE_P: now also R11.1, R31.1; no longer C12.2
- net OFF_Z_BN: now also R12.2
- net OFF_Z_BP: now also R16.2, R34.2; no longer R15.2
- net OFF_Z_DRV: now also R12.1, R34.1, U8.8; no longer R14.1, R15.1
- net OFF_Z_INN: now also C14.1, RN3.7, U8.9 (-); no longer C15.1, RN3.2, RN3.8
- net OFF_Z_INP: now also C15.1, RN3.8, U8.10 (+); no longer C13.1, RN3.5
- net OFF_Z_SENSE_P: now also R14.1, R33.1; no longer C13.2
- net +3V3A renamed +3V3D
- net +3V3D: no longer C10.1
- removed net DAC_OUT_REF: RN1.2, RN2.2, RN3.1
- net DAC_OUT_X renamed VOUTA
- net VOUTA: now also U3.4 (V_{OUT}A)
- net DAC_OUT_Y renamed VOUTC
- net VOUTC: now also U3.5 (V_{OUT}C)
- new net: C10.1, C32.1, U3.8 (V_{REFIN}/V_{REFOUT})
- new net: R27.1, U3.9 (~{CLR})
- new net: C33.1, C34.1, R28.2, U3.3 (AV_{DD})
- new net VOUTB: RN1.2, U3.13 (V_{OUT}B)
- new net VOUTD: RN2.2, U3.12 (V_{OUT}D)
- new net VOUTE: RN3.1, U3.6 (V_{OUT}E)
- new net VOUTF: RN3.2, U3.11 (V_{OUT}F)
- no-connect marks 1 -> 2
Other:
- moved on the sheet: C31, Q5, Q6, R26, RN1A, RN1B, RN1C, RN1D

Commit message: Work in progress rev2
Connections:
- net +5V is gone; now on net +5VA: Q5.2, Q7.2, Q9.2
- no-connect marks 2 -> 3
Other:
- note removed: "DAC CH0 → OFFSET_X DAC CH1 → OFFSET_Y DAC CH2 → OFFSET_Z DAC_CH3 → idscale reference (Negative input of OPAMP)"
- moved on the sheet: C12, C13, C14, C15, C31, Q10, Q7, Q8, Q9, R11, R12, R13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

Commit message: ...
Parts:
- added Q7: MMBT5551, PCM_Package_TO_SOT_SMD_AKL:SOT-23, symbol PCM_Transistor_BJT_AKL:MMBT5551
- added Q8: MMBT5401, PCM_Package_TO_SOT_SMD_AKL:SOT-23, symbol PCM_Transistor_BJT_AKL:MMBT5401
- renumbered C33 to C10, C9 to C12, C10 to C13, C32 to C14, C12 to C15, C13 to C16, C31 to C17, C14 to C18, C15 to C19, C34 to C9, Q8 to Q10, Q9 to Q11, Q10 to Q12, Q7 to Q9, R7 to R10, R27 to R11, R9 to R12, R10 to R13, R8 to R14, R11 to R15, R13 to R16, R31 to R17, R32 to R18, R12 to R19, R14 to R20, R26 to R21, R16 to R22, R33 to R23, R34 to R24, R6 to R5, R15 to R6, R28 to R7, R29 to R8, R30 to R9, U8 to U3, U3 to U4
Connections:
- new net: Q7.2 (E), Q8.2 (E)

Commit message: clearing git
Parts:
- RN1, RN2, RN3: footprint Resistor_SMD:R_Array_Convex_4x0612 -> Resistor_SMD:R_Array_Convex_4x0603; LCSC C29718 -> C454436
Connections:
- net VOUTA: no longer U4.4 (V_{OUT}A)
- net VOUTB: no longer U4.13 (V_{OUT}B)
- net VOUTC: no longer U4.5 (V_{OUT}C)
- net VOUTD: no longer U4.12 (V_{OUT}D)
- net VOUTE: no longer U4.6 (V_{OUT}E)
- net VOUTF: no longer U4.11 (V_{OUT}F)
- new net DAC_M_OUTA: U4.4 (V_{OUT}A)
- new net DAC_M_OUTB: U4.13 (V_{OUT}B)
- new net DAC_M_OUTC: U4.5 (V_{OUT}C)
- new net DAC_M_OUTD: U4.12 (V_{OUT}D)
- new net DAC_M_OUTE: U4.6 (V_{OUT}E)
- new net DAC_M_OUTF: U4.11 (V_{OUT}F)
Other:
- note added: "DAC M for Magnetic offset calibration (ambient)"
