File: hardware/pcb/Expension_card_design/magnetic_expension/magnetic_expension.kicad_pcb (KiCad board)
At the start: 4 copper layers, 40 x 60 mm, 83 parts, among them J1 528850274, Q1 D882, Q10 B772, Q2 DMC3028LSD, Q3 B772, Q4 D882, Q5 D882, Q6 B772, Q7 D882, Q8 B772, Q9 D882, U1 HMC1001-RC, U2 HMC1002-TR, U3 LM324DT, U4 MCP4728, U5 INA851RGTR, U6 INA851RGTR, U7 INA851RGTR

Commit message: Python app works as I want
Parts:
- removed U4: MCP4728, Package_SO:MSOP-10_3x3mm_P0.5mm
- added C10: 100n, Capacitor_SMD:C_0603_1608Metric, F.Cu at (141.6, 36.7)
- added C11: 4u7, Capacitor_SMD:C_1206_3216Metric, F.Cu at (130.7, 40.4)
- added C12: 4u7, Capacitor_SMD:C_1206_3216Metric, F.Cu at (130.7, 43.8)
- added C13: 4u7, Capacitor_SMD:C_1206_3216Metric, F.Cu at (130.7, 47.1)
- added C14: 4u7, Capacitor_SMD:C_1206_3216Metric, F.Cu at (130.7, 50.5)
- added C15: 4u7, Capacitor_SMD:C_1206_3216Metric, F.Cu at (130.7, 53.8)
- added C32: 4u7, Capacitor_SMD:C_1206_3216Metric, F.Cu at (130.7, 57.2)
- added C33: 4u7, Capacitor_SMD:C_1206_3216Metric, F.Cu at (130.7, 60.5)
- added C34: 100n, Capacitor_SMD:C_0603_1608Metric, F.Cu at (141.6, 39.2)
- added C35: 100n, Capacitor_SMD:C_0603_1608Metric, F.Cu at (124.2, 52.1)
- added C36: 100n, Capacitor_SMD:C_0603_1608Metric, F.Cu at (124.2, 54.6)
- added C37: 100n, Capacitor_SMD:C_0603_1608Metric, F.Cu at (124.2, 57.1)
- added C9: 4u7, Capacitor_SMD:C_1206_3216Metric, F.Cu at (130.7, 37.1)
- added Q10: B772, Package_TO_SOT_SMD:SOT-89-3, F.Cu at (136.8, 56.9)
- added Q7: D882, Package_TO_SOT_SMD:SOT-89-3, F.Cu at (136.8, 38.5)
- added Q8: B772, Package_TO_SOT_SMD:SOT-89-3, F.Cu at (136.8, 44.6)
- added Q9: D882, Package_TO_SOT_SMD:SOT-89-3, F.Cu at (136.8, 50.8)
- added R11: 22k, Resistor_SMD:R_0603_1608Metric, F.Cu at (141.6, 49.2)
- added R12: 470, Resistor_SMD:R_0603_1608Metric, F.Cu at (145.6, 36.7)
- added R13: 22k, Resistor_SMD:R_0603_1608Metric, F.Cu at (145.6, 39.2)
- added R14: 22k, Resistor_SMD:R_0603_1608Metric, F.Cu at (145.6, 41.7)
- added R15: 22k, Resistor_SMD:R_0603_1608Metric, F.Cu at (145.6, 44.2)
- added R16: 22k, Resistor_SMD:R_0603_1608Metric, F.Cu at (145.6, 46.7)
- added R27: 20k, Resistor_SMD:R_0603_1608Metric, F.Cu at (145.6, 49.2)
- added R28: 10, Resistor_SMD:R_0603_1608Metric, F.Cu at (149.7, 36.7)
- added R29: 22k, Resistor_SMD:R_0603_1608Metric, F.Cu at (149.7, 39.2)
- added R30: 200, Resistor_SMD:R_1206_3216Metric, F.Cu at (142.4, 52.1)
- added R31: 200, Resistor_SMD:R_1206_3216Metric, F.Cu at (142.4, 55.4)
- added R32: 470, Resistor_SMD:R_0603_1608Metric, F.Cu at (149.7, 41.7)
- added R33: 200, Resistor_SMD:R_1206_3216Metric, F.Cu at (142.4, 58.7)
- added R34: 470, Resistor_SMD:R_0603_1608Metric, F.Cu at (149.7, 44.2)
- added R35: 48,7, Resistor_SMD:R_0603_1608Metric, F.Cu at (124.2, 59.6)
- added R36: 48,7, Resistor_SMD:R_0603_1608Metric, F.Cu at (124.2, 62.1)
- added R37: 48,7, Resistor_SMD:R_0603_1608Metric, F.Cu at (124.2, 64.6)
- added R38: 48,7, Resistor_SMD:R_0603_1608Metric, F.Cu at (124.2, 67.1)
- added R39: 48,7, Resistor_SMD:R_0603_1608Metric, F.Cu at (124.2, 69.6)
- added R40: 48,7, Resistor_SMD:R_0603_1608Metric, F.Cu at (124.2, 72.1)
- added R6: 470, Resistor_SMD:R_0603_1608Metric, F.Cu at (141.6, 41.7)
- added R7: 470, Resistor_SMD:R_0603_1608Metric, F.Cu at (141.6, 44.2)
- added R8: 470, Resistor_SMD:R_0603_1608Metric, F.Cu at (141.6, 46.7)
- added RN2: 10k, Resistor_SMD:R_Array_Convex_4x0612, F.Cu at (147.1, 59.4)
- added RN3: 10k, Resistor_SMD:R_Array_Convex_4x0612, F.Cu at (150.7, 59.4)
- added U8: OPA4197xPW, Package_SO:TSSOP-14_4.4x5mm_P0.65mm, F.Cu at (91.7, 73.3)
- U3: value LM324DT -> DAC7678SPWR; footprint Package_SO:SOIC-14_3.9x8.7mm_P1.27mm -> Package_SO:TSSOP-16_4.4x5mm_P0.65mm
- moved U3 8.98 mm to (92.9, 82.2)
Connections:
- J1 pad 11: GND -> +1V65
- J1 pad 12: +1V65 -> +18V
- J1 pad 13: +18V -> +5VA
- J1 pad 14: +5VA -> -5VA
- J1 pad 15: -5VA -> +9VA
- J1 pad 16: +9VA -> /SENSOR_SET_CTRL
- J1 pad 17: /SENSOR_SET_CTRL -> /SENSOR_RESET_CTRL
- J1 pad 18: /SENSOR_RESET_CTRL -> +3V3D
- RN1 pad 1: /SENSOR_OFFSET_DRIVERS/DAC_OUT_X -> /SENSOR_OFFSET_DRIVERS/VOUTA
- RN1 pad 2: /SENSOR_OFFSET_DRIVERS/DAC_OUT_REF -> /SENSOR_OFFSET_DRIVERS/VOUTB
- U3 pad 1: /SENSOR_OFFSET_DRIVERS/OFF_X_DRV -> unconnected-(U3-~{LDAC}-Pad1)
- U3 pad 10: /SENSOR_OFFSET_DRIVERS/OFF_Z_INP -> unconnected-(U3-V_{OUT}H-Pad10)
- U3 pad 11: -5VA -> /SENSOR_OFFSET_DRIVERS/VOUTF
- U3 pad 12: +1V65 -> /SENSOR_OFFSET_DRIVERS/VOUTD
- U3 pad 13: /SENSOR_OFFSET_DRIVERS/1V65_FB -> /SENSOR_OFFSET_DRIVERS/VOUTB
- U3 pad 14: /SENSOR_OFFSET_DRIVERS/1V65_FB -> GND
- U3 pad 2: /SENSOR_OFFSET_DRIVERS/OFF_X_INN -> GND
- U3 pad 3: /SENSOR_OFFSET_DRIVERS/OFF_X_INP -> Net-(U3-AV_{DD})
- U3 pad 4: +5VA -> /SENSOR_OFFSET_DRIVERS/VOUTA
- U3 pad 5: /SENSOR_OFFSET_DRIVERS/OFF_Y_INP -> /SENSOR_OFFSET_DRIVERS/VOUTC
- U3 pad 6: /SENSOR_OFFSET_DRIVERS/OFF_Y_INN -> /SENSOR_OFFSET_DRIVERS/VOUTE
- U3 pad 7: /SENSOR_OFFSET_DRIVERS/OFF_Y_DRV -> unconnected-(U3-V_{OUT}G-Pad7)
- U3 pad 8: /SENSOR_OFFSET_DRIVERS/OFF_Z_DRV -> Net-(U3-V_{REFIN}/V_{REFOUT})
- U3 pad 9: /SENSOR_OFFSET_DRIVERS/OFF_Z_INN -> Net-(U3-~{CLR})
- U5 pad 1: /ANALOG_FRONTEND_INA851/BR_X+ -> /ANALOG_FRONTEND_INA851/BR_FTL_X+
- U5 pad 4: /ANALOG_FRONTEND_INA851/BR_X- -> /ANALOG_FRONTEND_INA851/BR_FTL_X-
- U6 pad 1: /ANALOG_FRONTEND_INA851/BR_Z+ -> /ANALOG_FRONTEND_INA851/BR_FTL_X+
- U6 pad 4: /ANALOG_FRONTEND_INA851/BR_Z- -> /ANALOG_FRONTEND_INA851/BR_FTL_X-
- U7 pad 1: /ANALOG_FRONTEND_INA851/BR_Y+ -> /ANALOG_FRONTEND_INA851/BR_FTL_X+
- U7 pad 4: /ANALOG_FRONTEND_INA851/BR_Y- -> /ANALOG_FRONTEND_INA851/BR_FTL_X-
Routing:
- net +18V: track 38.3 -> 51.2 mm, vias 1 -> 3
- net +1V65: track 12.9 -> 1.89 mm, vias 2 -> 1
- net /SENSOR_OFFSET_DRIVERS/VOUTA: track 0.00 -> 8.96 mm
- net /SENSOR_OFFSET_DRIVERS/DAC_OUT_X: track 8.96 -> 0.00 mm
- net GND: track 65.1 -> 60.2 mm, vias 135 -> 132
- net /SENSOR_OFFSET_DRIVERS/VOUTE: track 0.00 -> 1.60 mm, vias 0 -> 1
- net /SENSOR_OFFSET_DRIVERS/VOUTB: track 0.00 -> 1.33 mm, vias 0 -> 1

Commit message: Work in progress rev2
Parts:
- removed the C10 at (94.1, 84.8)
- removed the C10 at (141.6, 36.7)
- removed the C11 at (84.2, 69.3)
- removed the C11 at (130.7, 40.4)
- removed the C12 at (90.2, 66.7)
- removed the C12 at (130.7, 43.8)
- removed the C13 at (100.2, 76.6)
- removed the C13 at (130.7, 47.1)
- removed the C14 at (88.5, 63.9)
- removed the C14 at (130.7, 50.5)
- removed the C15 at (130.7, 53.8)
- removed the C15 at (100.2, 73.1)
- removed the C9 at (130.7, 37.1)
- removed the C9 at (82.7, 73.2)
- removed J1: 528850274, magnode_footprints:CON_528850274_MOL
- removed the Q10 at (101.3, 28.6)
- removed the Q10 at (136.8, 56.9)
- removed the Q7 at (82.6, 60.0)
- removed the Q7 at (136.8, 38.5)
- removed the Q8 at (88.5, 60.2)
- removed the Q8 at (136.8, 44.6)
- removed the Q9 at (106.9, 33.9)
- removed the Q9 at (136.8, 50.8)
- removed R10, R9: 4k7, Resistor_SMD:R_0603_1608Metric
- removed the R11 at (83.7, 63.3)
- removed the R11 at (141.6, 49.2)
- removed the R12 at (90.2, 55.8)
- removed the R12 at (145.6, 36.7)
- removed the R13 at (145.6, 39.2)
- removed the R13 at (91.6, 46.2)
- removed the R14 at (108.3, 29.5)
- removed the R14 at (145.6, 41.7)
- removed the R15 at (97.1, 30.6)
- removed the R15 at (145.6, 44.2)
- removed the R16 at (145.6, 46.7)
- removed the R16 at (102.9, 33.9)
- removed the R6 at (83.0, 51.0)
- removed the R6 at (141.6, 41.7)
- removed the R7 at (141.6, 44.2)
- removed the R7 at (87.4, 55.5)
- removed the R8 at (91.6, 49.4)
- removed the R8 at (141.6, 46.7)
- removed the RN2 at (87.3, 66.6)
- removed the RN2 at (147.1, 59.4)
- removed the RN3 at (150.7, 59.4)
- removed the RN3 at (97.8, 75.0)
- added C10: 100n, Capacitor_SMD:C_0603_1608Metric, F.Cu at (143.0, 24.6)
- added C11: 4u7, Capacitor_SMD:C_1206_3216Metric, F.Cu at (138.2, 28.4)
- added C12: 4u7, Capacitor_SMD:C_1206_3216Metric, F.Cu at (138.2, 31.8)
- added C13: 4u7, Capacitor_SMD:C_1206_3216Metric, F.Cu at (138.2, 35.1)
- added C14: 4u7, Capacitor_SMD:C_1206_3216Metric, F.Cu at (138.2, 38.5)
- added C15: 4u7, Capacitor_SMD:C_1206_3216Metric, F.Cu at (138.2, 41.8)
- added C9: 4u7, Capacitor_SMD:C_1206_3216Metric, F.Cu at (138.2, 25.1)
- added J2: 528850374, magnode_footprints:CONN_MOLEX_02x15_52885-0374, F.Cu at (139.1, 65.6)
- added Q10: B772, Package_TO_SOT_SMD:SOT-89-3, F.Cu at (132.6, 57.1)
- added Q7: D882, Package_TO_SOT_SMD:SOT-89-3, F.Cu at (132.6, 38.7)
- added Q8: B772, Package_TO_SOT_SMD:SOT-89-3, F.Cu at (132.6, 44.9)
- added Q9: D882, Package_TO_SOT_SMD:SOT-89-3, F.Cu at (132.6, 51.0)
- added R11: 22k, Resistor_SMD:R_0603_1608Metric, F.Cu at (147.0, 24.6)
- added R12: 470, Resistor_SMD:R_0603_1608Metric, F.Cu at (147.0, 27.1)
- added R13: 22k, Resistor_SMD:R_0603_1608Metric, F.Cu at (147.0, 29.7)
- added R14: 22k, Resistor_SMD:R_0603_1608Metric, F.Cu at (147.0, 32.2)
- added R15: 22k, Resistor_SMD:R_0603_1608Metric, F.Cu at (147.0, 34.7)
- added R16: 22k, Resistor_SMD:R_0603_1608Metric, F.Cu at (147.0, 37.2)
- added R6: 470, Resistor_SMD:R_0603_1608Metric, F.Cu at (143.0, 32.2)
- added R7: 470, Resistor_SMD:R_0603_1608Metric, F.Cu at (143.0, 34.7)
- added R8: 470, Resistor_SMD:R_0603_1608Metric, F.Cu at (143.0, 37.2)
- added RN2: 10k, Resistor_SMD:R_Array_Convex_4x0612, F.Cu at (152.1, 40.8)
- added RN3: 10k, Resistor_SMD:R_Array_Convex_4x0612, F.Cu at (155.7, 40.8)
- moved U7 91.7 mm to (183.9, 36.7), turned to 0 degrees
- moved U6 90.1 mm to (183.9, 31.4), turned to 0 degrees
- moved R22 89.7 mm to (175.2, 32.2), turned to 0 degrees
- moved R20 88.6 mm to (175.2, 27.1), turned to 0 degrees
- moved C28 87.2 mm to (171.2, 24.6), turned to 0 degrees
- moved U5 86.4 mm to (183.9, 26.0), turned to 0 degrees
- moved C30 85.4 mm to (171.2, 27.1), turned to 0 degrees
- moved R23 84.8 mm to (175.2, 34.7), turned to 0 degrees
- moved R25 84.7 mm to (175.2, 39.7), turned to 0 degrees
- moved R24 82.4 mm to (175.2, 37.2), turned to 0 degrees
- moved R19 82.1 mm to (175.2, 24.6), turned to 0 degrees
- moved C23 80.9 mm to (167.2, 34.7), turned to 0 degrees
- moved R21 78.5 mm to (175.2, 29.7), turned to 0 degrees
- moved C20 75.6 mm to (167.2, 29.7), turned to 0 degrees
- moved C18 74.4 mm to (167.2, 27.1), turned to 0 degrees
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Connections:
- net /SENSOR_SET_CTRL renamed /CONNECTOR/SENSOR_SET_CTRL
- Q2 pad 2: /SENSOR_RESET_CTRL -> /CONNECTOR/SENSOR_RESET_CTRL
- Q5 pad 2: +5V -> +5VA
- R1 pad 1: /DEVICE_DETECT -> /CONNECTOR/DEVICE_DETECT
- U3 pad 15: /SENSOR_OFFSET_DRIVERS/I2C.SDA -> /CONNECTOR/I2C.SDA
- U3 pad 16: /SENSOR_OFFSET_DRIVERS/I2C.SCL -> /CONNECTOR/I2C.SCL
Routing:
- net +5VA: track 131.8 -> 0.00 mm, vias 6 -> 0
- net -5VA: track 117.3 -> 0.00 mm, vias 6 -> 0
- net +3V3A: track 106.2 -> 0.00 mm, vias 5 -> 0
- net +9VA: track 74.6 -> 0.00 mm, vias 4 -> 0
- net /SENSOR_OFFSET_DRIVERS/OFF_Z_DRV: track 74.1 -> 0.00 mm, vias 3 -> 0
- net +5V: track 66.4 -> 0.00 mm, vias 2 -> 0
- net GND: track 60.2 -> 0.00 mm, vias 132 -> 0
- net /SENSOR_OFFSET_DRIVERS/OFF_Z_SENSE_P: track 55.0 -> 0.00 mm, vias 2 -> 0
- net +1V65B: track 51.9 -> 0.00 mm, vias 5 -> 0
- net +18V: track 51.2 -> 0.00 mm, vias 3 -> 0
- net /SENSOR_3AXIS_HMC100X/OFFSET_Z+: track 47.3 -> 0.00 mm, vias 1 -> 0
- net /SENSOR_RESET_CTRL: track 46.5 -> 0.00 mm, vias 2 -> 0
- net /ANALOG_FRONTEND_INA851/Z_INA_OUT+: track 42.5 -> 0.00 mm, vias 1 -> 0
- net /ANALOG_FRONTEND_INA851/Z_INA_OUT-: track 42.3 -> 0.00 mm, vias 1 -> 0
- net /SENSOR_OFFSET_DRIVERS/OFF_Y_DRV: track 34.4 -> 0.00 mm, vias 2 -> 0
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- removed copper zone on F.Cu, net +5VA
- removed copper zone on F.Cu, net -5VA
- removed copper zone on F.Cu, net /SENSOR_OFFSET_DRIVERS/OFF_X_SENSE_P
- removed copper zone on F.Cu, net /SENSOR_OFFSET_DRIVERS/OFF_Z_SENSE_P
- removed copper zone on F.Cu, net /SENSOR_SET_RESET_DRIVER/18V_IN
- removed copper zone on F.Cu, net /SENSOR_SET_RESET_DRIVER/18V_PULSE
Other:
- board size 40 x 60 mm -> 42 x 62 mm
- board text added: "Magnetic sensor v2 2026-06-??"
- board text removed: "1"
- board text removed: "10"
- board text removed: "11"
- board text removed: "20"
- board text removed: "AAF: Fc=360Hz"
- board text removed: "Magnetic sensor v1 2026-03-04"

Commit message: clearing git
Parts:
- removed C23: 220n, Capacitor_SMD:C_0603_1608Metric
- removed C29: 4u7, Capacitor_SMD:C_1206_3216Metric
- removed C35: 100n, Capacitor_SMD:C_0603_1608Metric
- removed J2: 528850374, magnode_footprints:CONN_MOLEX_02x15_52885-0374
- removed R12, R32, R34: 470, Resistor_SMD:R_0603_1608Metric
- removed R13, R29: 22k, Resistor_SMD:R_0603_1608Metric
- removed R27: 20k, Resistor_SMD:R_0603_1608Metric
- removed R37, R39: 48,7, Resistor_SMD:R_0603_1608Metric
- added C39: 1n, Capacitor_SMD:C_0603_1608Metric, F.Cu at (174.8, 17.2)
- added C40: 220n, Capacitor_SMD:C_0603_1608Metric, F.Cu at (174.8, 19.7)
- added C43: 1n, Capacitor_SMD:C_0603_1608Metric, F.Cu at (174.8, 22.2)
- added C44: 220n, Capacitor_SMD:C_0603_1608Metric, F.Cu at (174.8, 24.7)
- added C46: 100n, Capacitor_SMD:C_0603_1608Metric, F.Cu at (174.8, 27.2)
- added C47: 4u7, Capacitor_SMD:C_1206_3216Metric, F.Cu at (188.1, 32.7)
- added C48: 4u7, Capacitor_SMD:C_1206_3216Metric, F.Cu at (188.1, 36.0)
- added C49: 1n, Capacitor_SMD:C_0603_1608Metric, F.Cu at (174.8, 29.7)
- added C50: 220n, Capacitor_SMD:C_0603_1608Metric, F.Cu at (178.8, 17.2)
- added C51: 4u7, Capacitor_SMD:C_1206_3216Metric, F.Cu at (188.1, 39.4)
- added C52: 100n, Capacitor_SMD:C_0603_1608Metric, F.Cu at (178.8, 19.7)
- added C53: 4u7, Capacitor_SMD:C_1206_3216Metric, F.Cu at (188.1, 42.7)
- added J1: 528850374, magnode_footprints:CONN_MOLEX_02x15_52885-0374, F.Cu at (177.4, 72.8)
- added Q11: D882, Package_TO_SOT_SMD:SOT-89-3, F.Cu at (139.4, 43.5)
- added Q12: B772, Package_TO_SOT_SMD:SOT-89-3, F.Cu at (139.4, 49.7)
- added R10: 470, Resistor_SMD:R_0603_1608Metric, F.Cu at (153.9, 19.7)
- added R43: 1k, Resistor_SMD:R_0603_1608Metric, F.Cu at (178.8, 22.2)
- added R49: 1k, Resistor_SMD:R_0603_1608Metric, F.Cu at (178.8, 24.7)
- added R51: 1k, Resistor_SMD:R_0603_1608Metric, F.Cu at (178.8, 27.2)
- added R52: 1k, Resistor_SMD:R_0603_1608Metric, F.Cu at (178.8, 29.7)
- added R53: 1k, Resistor_SMD:R_0603_1608Metric, F.Cu at (182.8, 17.2)
- added R54: 20k, Resistor_SMD:R_0603_1608Metric, F.Cu at (182.8, 19.7)
- added R55: 1k, Resistor_SMD:R_0603_1608Metric, F.Cu at (182.8, 22.2)
- added R56: 1k, Resistor_SMD:R_0603_1608Metric, F.Cu at (182.8, 24.7)
- added R57: 1k, Resistor_SMD:R_0603_1608Metric, F.Cu at (182.8, 27.2)
- added R9: 200, Resistor_SMD:R_1206_3216Metric, F.Cu at (162.7, 17.6)
- added RN10: 5k, Resistor_SMD:R_Array_Convex_2x0603, F.Cu at (179.1, 35.7)
- added RN11: 5k, Resistor_SMD:R_Array_Convex_2x0603, F.Cu at (179.1, 38.9)
- added RN12: 20k, Resistor_SMD:R_Array_Convex_2x0603, F.Cu at (183.2, 32.6)
- added RN13: 10k, Resistor_SMD:R_Array_Convex_4x0603, F.Cu at (183.2, 42.8)
- added RN14: 5k, Resistor_SMD:R_Array_Convex_2x0603, F.Cu at (183.2, 35.7)
- added RN15: 5k, Resistor_SMD:R_Array_Convex_2x0603, F.Cu at (183.2, 38.9)
- added RN4: 20k, Resistor_SMD:R_Array_Convex_2x0603, F.Cu at (174.9, 32.6)
- added RN5: 10k, Resistor_SMD:R_Array_Convex_4x0603, F.Cu at (174.9, 42.8)
- added RN6: 5k, Resistor_SMD:R_Array_Convex_2x0603, F.Cu at (174.9, 35.7)
- added RN7: 5k, Resistor_SMD:R_Array_Convex_2x0603, F.Cu at (174.9, 38.9)
- added RN8: 20k, Resistor_SMD:R_Array_Convex_2x0603, F.Cu at (179.1, 32.6)
- added RN9: 10k, Resistor_SMD:R_Array_Convex_4x0603, F.Cu at (179.1, 42.8)
- added U10: DAC8571IDGK, Package_SO:MSOP-8_3x3mm_P0.65mm, F.Cu at (188.6, 24.9)
- added U11: THS4551IRGTR, magnode_footprints:VQFN-16-1EP_3x3mm_P0.5mm_EP1.68x1.68mm, F.Cu at (170.2, 29.2)
- added U12: THS4551IRGTR, magnode_footprints:VQFN-16-1EP_3x3mm_P0.5mm_EP1.68x1.68mm, F.Cu at (170.2, 34.5)
- added U13: DAC7678SPWR, Package_SO:TSSOP-16_4.4x5mm_P0.65mm, F.Cu at (189.6, 19.2)
- added U14: THS4551IRGTR, magnode_footprints:VQFN-16-1EP_3x3mm_P0.5mm_EP1.68x1.68mm, F.Cu at (170.2, 39.8)
- added U4: DAC7678SPWR, Package_SO:TSSOP-16_4.4x5mm_P0.65mm, F.Cu at (157.3, 39.0)
- added U9: THS4551IRGTR, magnode_footprints:VQFN-16-1EP_3x3mm_P0.5mm_EP1.68x1.68mm, F.Cu at (170.2, 23.9)
- C10, C20, C30, C36: value 100n -> 4u7; footprint Capacitor_SMD:C_0603_1608Metric -> Capacitor_SMD:C_1206_3216Metric
- C13, C21, C33, C9: value 4u7 -> 100n; footprint Capacitor_SMD:C_1206_3216Metric -> Capacitor_SMD:C_0603_1608Metric
- C18: value 220n -> 4u7; footprint Capacitor_SMD:C_0603_1608Metric -> Capacitor_SMD:C_1206_3216Metric
- C22, C34: value 100n -> 10n
- C28: value 220n -> 10n
- Q7: value D882 -> MMBT5551; footprint Package_TO_SOT_SMD:SOT-89-3 -> PCM_Package_TO_SOT_SMD_AKL:SOT-23
- Q8: value B772 -> MMBT5401; footprint Package_TO_SOT_SMD:SOT-89-3 -> PCM_Package_TO_SOT_SMD_AKL:SOT-23
- R1: value 20k -> 220; footprint Resistor_SMD:R_0603_1608Metric -> Resistor_SMD:R_2512_6332Metric
- R11: value 22k -> 20k
- R14: value 22k -> 470
- R17, R23: value 1k -> 200; footprint Resistor_SMD:R_0603_1608Metric -> Resistor_SMD:R_1206_3216Metric
- R18, R24: value 48,7 -> 470
- R19, R5: value 1k -> 470
- R2: value 220 -> 1k; footprint Resistor_SMD:R_2512_6332Metric -> Resistor_SMD:R_0603_1608Metric
- R20, R22: value 1k -> 22k
- R21: value 48,7 -> 20; footprint Resistor_SMD:R_0603_1608Metric -> Resistor_SMD:R_1206_3216Metric
- R25: value 1k -> 20k
- R26: value 20 -> 49.9; footprint Resistor_SMD:R_1206_3216Metric -> Resistor_SMD:R_0603_1608Metric
- R28: value 10 -> 100
- R30, R31: value 200 -> 49.9; footprint Resistor_SMD:R_1206_3216Metric -> Resistor_SMD:R_0603_1608Metric
- R33: value 200 -> 100; footprint Resistor_SMD:R_1206_3216Metric -> Resistor_SMD:R_0603_1608Metric
- R35, R36, R40: value 48,7 -> 49.9
- R38: value 48,7 -> 100
- R6, R8: value 470 -> 22k
- R7: value 470 -> 10
- RN1, RN2, RN3: footprint Resistor_SMD:R_Array_Convex_4x0612 -> Resistor_SMD:R_Array_Convex_4x0603
- U3: value DAC7678SPWR -> OPA4197xPW; footprint Package_SO:TSSOP-16_4.4x5mm_P0.65mm -> Package_SO:TSSOP-14_4.4x5mm_P0.65mm
- U8: value OPA4197xPW -> THS4551IRGTR; footprint Package_SO:TSSOP-14_4.4x5mm_P0.65mm -> magnode_footprints:VQFN-16-1EP_3x3mm_P0.5mm_EP1.68x1.68mm
- moved C31 46.7 mm to (175.2, 61.0)
- moved C34 40.8 mm to (179.2, 48.5)
- moved R28 40.3 mm to (179.2, 56.0)
- moved R5 40.3 mm to (149.9, 24.7)
- moved C33 39.9 mm to (175.2, 63.5)
- moved U8 39.5 mm to (170.2, 18.6)
- moved R30 38.5 mm to (179.2, 58.5)
- moved R25 38.3 mm to (169.5, 77.5)
- moved R31 38.2 mm to (179.2, 61.0)
- moved R33 37.9 mm to (179.2, 63.5)
- moved R26 37.8 mm to (179.2, 53.5)
- moved C32 36.5 mm to (170.3, 62.3)
- moved C28 34.1 mm to (175.2, 58.5)
- moved C36 33.5 mm to (170.3, 65.6)
- moved C30 31.8 mm to (170.3, 58.9)
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Connections:
- C10 pad 1: Net-(U3-V_{REFIN}/V_{REFOUT}) -> Net-(U4-AV_{DD})
- C11 pad 1: /SENSOR_OFFSET_DRIVERS/OFF_X_INN -> /MAGNETIC_OFFSET_DRIVERS/OFF_X_INN
- C12 pad 1: /SENSOR_OFFSET_DRIVERS/OFF_Y_INN -> /MAGNETIC_OFFSET_DRIVERS/OFF_X_INP
- C13 pad 1: /SENSOR_OFFSET_DRIVERS/OFF_Y_INP -> Net-(U4-V_{REFIN}/V_{REFOUT})
- C14 pad 1: /SENSOR_OFFSET_DRIVERS/OFF_Z_INN -> Net-(U4-V_{REFIN}/V_{REFOUT})
- C15 pad 1: /SENSOR_OFFSET_DRIVERS/OFF_Z_INP -> /MAGNETIC_OFFSET_DRIVERS/OFF_Y_INN
- C16 pad 1: +5VA -> /MAGNETIC_OFFSET_DRIVERS/OFF_Y_INP
- C17 pad 1: +5VA -> +1V65B
- C18 pad 1: /ANALOG_FRONTEND_INA851/X_INA_OUT+ -> /MAGNETIC_OFFSET_DRIVERS/OFF_Z_INN
- C18 pad 2: /ANALOG_FRONTEND_INA851/X_INA_OUT- -> GND
- C19 pad 1: +5VA -> /MAGNETIC_OFFSET_DRIVERS/OFF_Z_INP
- C21 pad 1: -5VA -> +5VA
- C22 pad 1: -5VA -> /INA_GAIN/BR_FTL_X+
- C22 pad 2: GND -> /INA_GAIN/BR_FTL_X-
- C28 pad 1: /ANALOG_FRONTEND_INA851/Y_INA_OUT+ -> /INA_GAIN/BR_FTL_X+
- C28 pad 2: /ANALOG_FRONTEND_INA851/Y_INA_OUT- -> /INA_GAIN/BR_FTL_X-
- C30 pad 1: -5VA -> +5VA
- C31 pad 1: +1V65B -> +5VA
- C32 pad 1: Net-(U3-V_{REFIN}/V_{REFOUT}) -> -5VA
- C33 pad 1: Net-(U3-AV_{DD}) -> -5VA
- C34 pad 1: Net-(U3-AV_{DD}) -> /INA_GAIN/BR_FTL_X+
- C34 pad 2: GND -> /INA_GAIN/BR_FTL_X-
- C36 pad 1: /ANALOG_FRONTEND_INA851/BR_FTL_X+ -> -5VA
- C36 pad 2: /ANALOG_FRONTEND_INA851/BR_FTL_X- -> GND
- C37 pad 1: /ANALOG_FRONTEND_INA851/BR_FTL_X+ -> -5VA
- C37 pad 2: /ANALOG_FRONTEND_INA851/BR_FTL_X- -> GND
- C9 pad 1: /SENSOR_OFFSET_DRIVERS/OFF_X_INP -> Net-(U4-AV_{DD})
- Q10 pad 1: /SENSOR_OFFSET_DRIVERS/OFF_Z_BP -> /MAGNETIC_OFFSET_DRIVERS/OFF_Y_BP
- Q10 pad 3: /SENSOR_OFFSET_DRIVERS/OFF_Z_SENSE_P -> /MAGNETIC_OFFSET_DRIVERS/OFF_Y_SENSE_P
- Q5 pad 1: /SENSOR_OFFSET_DRIVERS/OFF_X_BN -> /MAGNETIC_OFFSET_DRIVERS/OFF_X_BN
- Q5 pad 3: /SENSOR_OFFSET_DRIVERS/OFF_X_SENSE_P -> /MAGNETIC_OFFSET_DRIVERS/OFF_X_SENSE_P
- Q6 pad 1: /SENSOR_OFFSET_DRIVERS/OFF_X_BP -> /MAGNETIC_OFFSET_DRIVERS/OFF_X_BP
- Q6 pad 3: /SENSOR_OFFSET_DRIVERS/OFF_X_SENSE_P -> /MAGNETIC_OFFSET_DRIVERS/OFF_X_SENSE_P
- Q7 pad 1: /SENSOR_OFFSET_DRIVERS/OFF_Y_BN -> unconnected-(Q7-B-Pad1)
- Q7 pad 2: +5VA -> Net-(Q7-E)
- Q7 pad 3: /SENSOR_OFFSET_DRIVERS/OFF_Y_SENSE_P -> unconnected-(Q7-C-Pad3)
- Q8 pad 1: /SENSOR_OFFSET_DRIVERS/OFF_Y_BP -> unconnected-(Q8-B-Pad1)
- Q8 pad 2: -5VA -> Net-(Q7-E)
- Q8 pad 3: /SENSOR_OFFSET_DRIVERS/OFF_Y_SENSE_P -> unconnected-(Q8-C-Pad3)
- Q9 pad 1: /SENSOR_OFFSET_DRIVERS/OFF_Z_BN -> /MAGNETIC_OFFSET_DRIVERS/OFF_Y_BN
- Q9 pad 3: /SENSOR_OFFSET_DRIVERS/OFF_Z_SENSE_P -> /MAGNETIC_OFFSET_DRIVERS/OFF_Y_SENSE_P
- R1 pad 1: /CONNECTOR/DEVICE_DETECT -> /SENSOR_SET_RESET_DRIVER/18V_IN
- R1 pad 2: GND -> +18V
- R11 pad 1: /SENSOR_OFFSET_DRIVERS/OFF_Y_SENSE_P -> Net-(U4-~{CLR})
- R11 pad 2: /SENSOR_OFFSET_DRIVERS/OFF_Y_BN -> +5VA
- R14 pad 1: /SENSOR_OFFSET_DRIVERS/OFF_Z_SENSE_P -> /MAGNETIC_OFFSET_DRIVERS/OFF_Y_DRV
- R14 pad 2: /SENSOR_OFFSET_DRIVERS/OFF_Z_BN -> /MAGNETIC_OFFSET_DRIVERS/OFF_Y_BN
- R15 pad 1: /SENSOR_OFFSET_DRIVERS/OFF_X_SENSE_P -> /MAGNETIC_OFFSET_DRIVERS/OFF_Y_SENSE_P
- R15 pad 2: /SENSOR_OFFSET_DRIVERS/OFF_X_BN -> /MAGNETIC_OFFSET_DRIVERS/OFF_Y_BN
- R16 pad 1: /SENSOR_OFFSET_DRIVERS/OFF_Z_SENSE_P -> /MAGNETIC_OFFSET_DRIVERS/OFF_Y_SENSE_P
- R16 pad 2: /SENSOR_OFFSET_DRIVERS/OFF_Z_BP -> /MAGNETIC_OFFSET_DRIVERS/OFF_Y_BP
- R17 pad 1: /ANALOG_FRONTEND_INA851/X_INA_PRE_AAF+ -> /MAGNETIC_OFFSET_DRIVERS/OFF_Y_SENSE_P
- R17 pad 2: /ANALOG_FRONTEND_INA851/X_INA_OUT+ -> /MAGNETIC_OFFSET_DRIVERS/OFFSET_Y+
- R18 pad 1: /ANALOG_FRONTEND_INA851/X_RG+ -> /MAGNETIC_OFFSET_DRIVERS/OFF_Y_DRV
- R18 pad 2: /ANALOG_FRONTEND_INA851/X_RG- -> /MAGNETIC_OFFSET_DRIVERS/OFF_Y_BP
- R19 pad 1: /ANALOG_FRONTEND_INA851/X_INA_PRE_AAF- -> /MAGNETIC_OFFSET_DRIVERS/OFF_Z_DRV
- R19 pad 2: /ANALOG_FRONTEND_INA851/X_INA_OUT- -> /MAGNETIC_OFFSET_DRIVERS/OFF_Z_BN
- R2 pad 2: +18V -> /SENSOR_SET_RESET_DRIVER/18V_BUF
- R20 pad 1: /ANALOG_FRONTEND_INA851/Z_INA_PRE_AAF+ -> /MAGNETIC_OFFSET_DRIVERS/OFF_Z_SENSE_P
- R20 pad 2: /ANALOG_FRONTEND_INA851/Z_INA_OUT+ -> /MAGNETIC_OFFSET_DRIVERS/OFF_Z_BN
- R21 pad 1: /ANALOG_FRONTEND_INA851/Z_RG+ -> /MAGNETIC_OFFSET_DRIVERS/1V65_FB
- R21 pad 2: /ANALOG_FRONTEND_INA851/Z_RG- -> +1V65B
- R22 pad 1: /ANALOG_FRONTEND_INA851/Z_INA_PRE_AAF- -> /MAGNETIC_OFFSET_DRIVERS/OFF_Z_SENSE_P
- R22 pad 2: /ANALOG_FRONTEND_INA851/Z_INA_OUT- -> /MAGNETIC_OFFSET_DRIVERS/OFF_Z_BP
- R23 pad 1: /ANALOG_FRONTEND_INA851/Y_INA_PRE_AAF+ -> /MAGNETIC_OFFSET_DRIVERS/OFF_Z_SENSE_P
- R23 pad 2: /ANALOG_FRONTEND_INA851/Y_INA_OUT+ -> /MAGNETIC_OFFSET_DRIVERS/OFFSET_Z+
- R24 pad 1: /ANALOG_FRONTEND_INA851/Y_RG+ -> /MAGNETIC_OFFSET_DRIVERS/OFF_Z_DRV
- R24 pad 2: /ANALOG_FRONTEND_INA851/Y_RG- -> /MAGNETIC_OFFSET_DRIVERS/OFF_Z_BP
- R25 pad 1: /ANALOG_FRONTEND_INA851/Y_INA_PRE_AAF- -> /CONNECTOR/DEVICE_DETECT
- R25 pad 2: /ANALOG_FRONTEND_INA851/Y_INA_OUT- -> GND
- R26 pad 1: /SENSOR_OFFSET_DRIVERS/1V65_FB -> /INA_GAIN/BR_X+
- R26 pad 2: +1V65B -> /INA_GAIN/BR_FTL_X+
- R28 pad 1: +5VA -> /INA_GAIN/X_RG-
- R28 pad 2: Net-(U3-AV_{DD}) -> /INA_GAIN/X_RG+
- R3 pad 1: /SENSOR_SET_RESET_DRIVER/18V_IN -> /SENSOR_SET_RESET_DRIVER/18V_BUF
- R3 pad 2: /SENSOR_SET_RESET_DRIVER/18V_BUF -> /SENSOR_SET_RESET_DRIVER/PULL_DOWN
- R30 pad 1: /SENSOR_OFFSET_DRIVERS/OFF_X_SENSE_P -> /INA_GAIN/BR_X-
- R30 pad 2: /SENSOR_3AXIS_HMC100X/OFFSET_X+ -> /INA_GAIN/BR_FTL_X-
- R31 pad 1: /SENSOR_OFFSET_DRIVERS/OFF_Y_SENSE_P -> /INA_GAIN/BR_Z+
- R31 pad 2: /SENSOR_3AXIS_HMC100X/OFFSET_Y+ -> /INA_GAIN/BR_FTL_X+
- R33 pad 1: /SENSOR_OFFSET_DRIVERS/OFF_Z_SENSE_P -> /INA_GAIN/Z_RG-
- R33 pad 2: /SENSOR_3AXIS_HMC100X/OFFSET_Z+ -> /INA_GAIN/Z_RG+
- R35 pad 1: /ANALOG_FRONTEND_INA851/BR_X- -> /INA_GAIN/BR_Z-
- R35 pad 2: /ANALOG_FRONTEND_INA851/BR_FTL_X- -> /INA_GAIN/BR_FTL_X-
- R36 pad 1: /ANALOG_FRONTEND_INA851/BR_X+ -> /INA_GAIN/BR_Y+
- R36 pad 2: /ANALOG_FRONTEND_INA851/BR_FTL_X+ -> /INA_GAIN/BR_FTL_X+
- R38 pad 1: /ANALOG_FRONTEND_INA851/BR_Y- -> /INA_GAIN/Y_RG-
- R38 pad 2: /ANALOG_FRONTEND_INA851/BR_FTL_X- -> /INA_GAIN/Y_RG+
- R4 pad 1: /SENSOR_SET_RESET_DRIVER/18V_BUF -> /CONNECTOR/SENSOR_SET_CTRL
- R4 pad 2: /SENSOR_SET_RESET_DRIVER/PULL_DOWN -> /SENSOR_SET_RESET_DRIVER/3V3_SET_CTRL
- R40 pad 1: /ANALOG_FRONTEND_INA851/BR_Z- -> /INA_GAIN/BR_Y-
- R40 pad 2: /ANALOG_FRONTEND_INA851/BR_FTL_X- -> /INA_GAIN/BR_FTL_X-
- R5 pad 1: /CONNECTOR/SENSOR_SET_CTRL -> /MAGNETIC_OFFSET_DRIVERS/OFF_X_DRV
- R5 pad 2: /SENSOR_SET_RESET_DRIVER/3V3_SET_CTRL -> /MAGNETIC_OFFSET_DRIVERS/OFF_X_BN
- R6 pad 1: /SENSOR_OFFSET_DRIVERS/OFF_X_DRV -> /MAGNETIC_OFFSET_DRIVERS/OFF_X_SENSE_P
- R6 pad 2: /SENSOR_OFFSET_DRIVERS/OFF_X_BN -> /MAGNETIC_OFFSET_DRIVERS/OFF_X_BN
- R7 pad 1: /SENSOR_OFFSET_DRIVERS/OFF_X_DRV -> +5VA
- R7 pad 2: /SENSOR_OFFSET_DRIVERS/OFF_X_BP -> Net-(U4-AV_{DD})
- R8 pad 1: /SENSOR_OFFSET_DRIVERS/OFF_Y_DRV -> /MAGNETIC_OFFSET_DRIVERS/OFF_X_SENSE_P
- R8 pad 2: /SENSOR_OFFSET_DRIVERS/OFF_Y_BN -> /MAGNETIC_OFFSET_DRIVERS/OFF_X_BP
- RN1 pad 1: /SENSOR_OFFSET_DRIVERS/VOUTA -> /MAGNETIC_OFFSET_DRIVERS/VOUTA
- RN1 pad 2: /SENSOR_OFFSET_DRIVERS/VOUTB -> /MAGNETIC_OFFSET_DRIVERS/VOUTB
- RN1 pad 3: /SENSOR_OFFSET_DRIVERS/OFF_X_INP -> /MAGNETIC_OFFSET_DRIVERS/OFF_X_INP
- RN1 pad 4: /SENSOR_OFFSET_DRIVERS/OFF_X_INN -> /MAGNETIC_OFFSET_DRIVERS/OFF_X_INN
- RN1 pad 5: /SENSOR_3AXIS_HMC100X/OFFSET_X+ -> /MAGNETIC_OFFSET_DRIVERS/OFFSET_X+
- RN1 pad 6: /SENSOR_OFFSET_DRIVERS/OFF_X_SENSE_P -> /MAGNETIC_OFFSET_DRIVERS/OFF_X_SENSE_P
- RN1 pad 7: /SENSOR_OFFSET_DRIVERS/OFF_X_INN -> /MAGNETIC_OFFSET_DRIVERS/OFF_X_INN
- RN1 pad 8: /SENSOR_OFFSET_DRIVERS/OFF_X_INP -> /MAGNETIC_OFFSET_DRIVERS/OFF_X_INP
- RN2 pad 1: /SENSOR_OFFSET_DRIVERS/VOUTC -> /MAGNETIC_OFFSET_DRIVERS/VOUTC
- RN2 pad 2: /SENSOR_OFFSET_DRIVERS/VOUTD -> /MAGNETIC_OFFSET_DRIVERS/VOUTD
- RN2 pad 3: /SENSOR_OFFSET_DRIVERS/OFF_Y_INP -> /MAGNETIC_OFFSET_DRIVERS/OFF_Y_INP
- RN2 pad 4: /SENSOR_OFFSET_DRIVERS/OFF_Y_INN -> /MAGNETIC_OFFSET_DRIVERS/OFF_Y_INN
- RN2 pad 5: /SENSOR_3AXIS_HMC100X/OFFSET_Y+ -> /MAGNETIC_OFFSET_DRIVERS/OFFSET_Y+
- RN2 pad 6: /SENSOR_OFFSET_DRIVERS/OFF_Y_SENSE_P -> /MAGNETIC_OFFSET_DRIVERS/OFF_Y_SENSE_P
- RN2 pad 7: /SENSOR_OFFSET_DRIVERS/OFF_Y_INN -> /MAGNETIC_OFFSET_DRIVERS/OFF_Y_INN
- RN2 pad 8: /SENSOR_OFFSET_DRIVERS/OFF_Y_INP -> /MAGNETIC_OFFSET_DRIVERS/OFF_Y_INP
- RN3 pad 1: /SENSOR_OFFSET_DRIVERS/VOUTE -> /MAGNETIC_OFFSET_DRIVERS/VOUTE
- RN3 pad 2: /SENSOR_OFFSET_DRIVERS/VOUTF -> /MAGNETIC_OFFSET_DRIVERS/VOUTF
- RN3 pad 3: /SENSOR_OFFSET_DRIVERS/OFF_Z_INP -> /MAGNETIC_OFFSET_DRIVERS/OFF_Z_INP
- RN3 pad 4: /SENSOR_OFFSET_DRIVERS/OFF_Z_INN -> /MAGNETIC_OFFSET_DRIVERS/OFF_Z_INN
- RN3 pad 5: /SENSOR_3AXIS_HMC100X/OFFSET_Z+ -> /MAGNETIC_OFFSET_DRIVERS/OFFSET_Z+
- RN3 pad 6: /SENSOR_OFFSET_DRIVERS/OFF_Z_SENSE_P -> /MAGNETIC_OFFSET_DRIVERS/OFF_Z_SENSE_P
- RN3 pad 7: /SENSOR_OFFSET_DRIVERS/OFF_Z_INN -> /MAGNETIC_OFFSET_DRIVERS/OFF_Z_INN
- RN3 pad 8: /SENSOR_OFFSET_DRIVERS/OFF_Z_INP -> /MAGNETIC_OFFSET_DRIVERS/OFF_Z_INP
- U1 pad 2: /SENSOR_3AXIS_HMC100X/OFFSET_Z+ -> /MAGNETIC_OFFSET_DRIVERS/OFFSET_Z+
- U1 pad 5: /ANALOG_FRONTEND_INA851/BR_Z- -> /INA_GAIN/BR_Z-
- U1 pad 8: /ANALOG_FRONTEND_INA851/BR_Z+ -> /INA_GAIN/BR_Z+
- U2 pad 12: /ANALOG_FRONTEND_INA851/BR_Y- -> /INA_GAIN/BR_Y-
- U2 pad 15: /SENSOR_3AXIS_HMC100X/OFFSET_Y+ -> /MAGNETIC_OFFSET_DRIVERS/OFFSET_Y+
- U2 pad 17: /SENSOR_3AXIS_HMC100X/OFFSET_X+ -> /MAGNETIC_OFFSET_DRIVERS/OFFSET_X+
- U2 pad 2: /ANALOG_FRONTEND_INA851/BR_X+ -> /INA_GAIN/BR_X+
- U2 pad 5: /ANALOG_FRONTEND_INA851/BR_X- -> /INA_GAIN/BR_X-
- U2 pad 9: /ANALOG_FRONTEND_INA851/BR_Y+ -> /INA_GAIN/BR_Y+
- U3 pad 1: unconnected-(U3-~{LDAC}-Pad1) -> /MAGNETIC_OFFSET_DRIVERS/OFF_X_DRV
- U3 pad 10: unconnected-(U3-V_{OUT}H-Pad10) -> /MAGNETIC_OFFSET_DRIVERS/OFF_Z_INP
- U3 pad 11: /SENSOR_OFFSET_DRIVERS/VOUTF -> -5VA
- U3 pad 12: /SENSOR_OFFSET_DRIVERS/VOUTD -> +1V65
- U3 pad 13: /SENSOR_OFFSET_DRIVERS/VOUTB -> /MAGNETIC_OFFSET_DRIVERS/1V65_FB
- U3 pad 14: GND -> /MAGNETIC_OFFSET_DRIVERS/1V65_FB
- U3 pad 2: GND -> /MAGNETIC_OFFSET_DRIVERS/OFF_X_INN
- U3 pad 3: Net-(U3-AV_{DD}) -> /MAGNETIC_OFFSET_DRIVERS/OFF_X_INP
- U3 pad 4: /SENSOR_OFFSET_DRIVERS/VOUTA -> +5VA
- U3 pad 5: /SENSOR_OFFSET_DRIVERS/VOUTC -> /MAGNETIC_OFFSET_DRIVERS/OFF_Y_INP
- U3 pad 6: /SENSOR_OFFSET_DRIVERS/VOUTE -> /MAGNETIC_OFFSET_DRIVERS/OFF_Y_INN
- U3 pad 7: unconnected-(U3-V_{OUT}G-Pad7) -> /MAGNETIC_OFFSET_DRIVERS/OFF_Y_DRV
- U3 pad 8: Net-(U3-V_{REFIN}/V_{REFOUT}) -> /MAGNETIC_OFFSET_DRIVERS/OFF_Z_DRV
- U3 pad 9: Net-(U3-~{CLR}) -> /MAGNETIC_OFFSET_DRIVERS/OFF_Z_INN
- U5 pad 1: /ANALOG_FRONTEND_INA851/BR_FTL_X+ -> /INA_GAIN/BR_FTL_X+
- U5 pad 10: /ANALOG_FRONTEND_INA851/X_INA_PRE_AAF- -> /INA_GAIN/X_INA_OUT-
- U5 pad 11: /ANALOG_FRONTEND_INA851/X_INA_PRE_AAF+ -> /INA_GAIN/X_INA_OUT+
- U5 pad 2: /ANALOG_FRONTEND_INA851/X_RG+ -> /INA_GAIN/X_RG+
- U5 pad 3: /ANALOG_FRONTEND_INA851/X_RG- -> /INA_GAIN/X_RG-
- U5 pad 4: /ANALOG_FRONTEND_INA851/BR_FTL_X- -> /INA_GAIN/BR_FTL_X-
- U6 pad 1: /ANALOG_FRONTEND_INA851/BR_FTL_X+ -> /INA_GAIN/BR_FTL_X+
- U6 pad 10: /ANALOG_FRONTEND_INA851/Z_INA_PRE_AAF- -> /INA_GAIN/Z_INA_OUT-
- U6 pad 11: /ANALOG_FRONTEND_INA851/Z_INA_PRE_AAF+ -> /INA_GAIN/Z_INA_OUT+
- U6 pad 2: /ANALOG_FRONTEND_INA851/Z_RG+ -> /INA_GAIN/Z_RG+
- U6 pad 3: /ANALOG_FRONTEND_INA851/Z_RG- -> /INA_GAIN/Z_RG-
- U6 pad 4: /ANALOG_FRONTEND_INA851/BR_FTL_X- -> /INA_GAIN/BR_FTL_X-
- U7 pad 1: /ANALOG_FRONTEND_INA851/BR_FTL_X+ -> /INA_GAIN/BR_FTL_X+
- U7 pad 10: /ANALOG_FRONTEND_INA851/Y_INA_PRE_AAF- -> /INA_GAIN/Y_INA_OUT-
- U7 pad 11: /ANALOG_FRONTEND_INA851/Y_INA_PRE_AAF+ -> /INA_GAIN/Y_INA_OUT+
- U7 pad 2: /ANALOG_FRONTEND_INA851/Y_RG+ -> /INA_GAIN/Y_RG+
- U7 pad 3: /ANALOG_FRONTEND_INA851/Y_RG- -> /INA_GAIN/Y_RG-
- U7 pad 4: /ANALOG_FRONTEND_INA851/BR_FTL_X- -> /INA_GAIN/BR_FTL_X-
- U8 pad 1: /SENSOR_OFFSET_DRIVERS/OFF_X_DRV -> unconnected-(U8-FB--Pad1)
- U8 pad 10: /SENSOR_OFFSET_DRIVERS/OFF_Z_INP -> /BRIDGE_OFFSET/V_{COMP}-
- U8 pad 11: -5VA -> /BRIDGE_OFFSET/V_{COMP}+
- U8 pad 12: +1V65 -> unconnected-(U8-~{PD}-Pad12)
- U8 pad 13: /SENSOR_OFFSET_DRIVERS/1V65_FB -> GND
- U8 pad 14: /SENSOR_OFFSET_DRIVERS/1V65_FB -> GND
- U8 pad 2: /SENSOR_OFFSET_DRIVERS/OFF_X_INN -> /BRIDGE_OFFSET/COMP_POS_FB
- U8 pad 3: /SENSOR_OFFSET_DRIVERS/OFF_X_INP -> Net-(R47-Pad2)
- U8 pad 4: +5VA -> unconnected-(U8-FB+-Pad4)
- U8 pad 5: /SENSOR_OFFSET_DRIVERS/OFF_Y_INP -> +3V3A
- U8 pad 6: /SENSOR_OFFSET_DRIVERS/OFF_Y_INN -> +3V3A
- U8 pad 7: /SENSOR_OFFSET_DRIVERS/OFF_Y_DRV -> +3V3A
- U8 pad 8: /SENSOR_OFFSET_DRIVERS/OFF_Z_DRV -> +3V3A
- U8 pad 9: /SENSOR_OFFSET_DRIVERS/OFF_Z_INN -> +1V65B
