File: hardware/pcb/Expension_card_design/Simulation_mag_v2/Simulation_mag_v2.kicad_sch (KiCad schematic)
At the start: 25 parts, among them U1 HMC1001_SPICE, U2 INA851_Spice, U3 ${SIM.PARAMS}, U4 ${SIM.PARAMS}

Commit message: kicad mag board done
Other:
- note added: ".param A=10m"
- note removed: ".param A=0m"
Changed lines of the file:
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@@
 	(generator_version "10.0")
 	(paper "A3")
-	(text ".param A=0m\n"
+	(text ".param A=10m\n"
 		(exclude_from_sim no)
 		(at 32.512 63.754 0)
@@
 		(unit 1)
 		(body_style 1)
-		(exclude_from_sim yes)
+		(exclude_from_sim no)
 		(in_bom yes)
 		(on_board yes)
@@
 			)
 		)
-		(property "Sim.Params" "OFFSET=30m"
+		(property "Sim.Params" "OFFSET=-80m"
 			(at 86.36 91.44 0)
 			(hide yes)
@@
 		(unit 1)
 		(body_style 1)
-		(exclude_from_sim no)
+		(exclude_from_sim yes)
 		(in_bom yes)
 		(on_board yes)
