File: hardware/pcb/Expension_card_design/magnetic_expension_v2/magnetic_expension_v2.kicad_pcb (KiCad board)
At the start: 4 copper layers, 65 x 42 mm, 76 parts, among them J1 528850374, Q1 D882, Q2 D882, Q3 B772, U1 HMC1001-RC, U10 OPA2197xD, U11 INA851RGTR, U12 THP210DGK, U2 HMC1002-TR, U3 OPA4197xD, U4 OPA2197xD, U7 OPA2197xD

Commit message: kicad mag board done
Parts:
- added C29: 100n, Capacitor_SMD:C_0603_1608Metric, F.Cu at (94.3, 86.7)
- added C30: 100n, Capacitor_SMD:C_0603_1608Metric, F.Cu at (96.0, 81.7)
- added C31: 47u, Capacitor_SMD:C_1206_3216Metric, F.Cu at (100.9, 88.2)
- added C32: 100n, Capacitor_SMD:C_0603_1608Metric, F.Cu at (119.2, 88.5)
- added C33: 4u7, Capacitor_SMD:C_1206_3216Metric, F.Cu at (116.5, 90.5)
- added C34: 100n, Capacitor_SMD:C_0603_1608Metric, F.Cu at (105.0, 85.8)
- added C35: 4u7, Capacitor_SMD:C_1206_3216Metric, F.Cu at (102.0, 81.6)
- added C36: 4u7, Capacitor_SMD:C_1206_3216Metric, F.Cu at (104.5, 81.6)
- added C37: 220n, Capacitor_SMD:C_0805_2012Metric, F.Cu at (124.0, 84.5)
- added C38: 100n, Capacitor_SMD:C_0603_1608Metric, F.Cu at (114.5, 85.5)
- added C39: 100n, Capacitor_SMD:C_0603_1608Metric, F.Cu at (110.0, 80.8)
- added C40: 4u7, Capacitor_SMD:C_1206_3216Metric, F.Cu at (114.0, 80.5)
- added C41: 10n, Capacitor_SMD:C_0603_1608Metric, F.Cu at (83.4, 107.6)
- added C42: 4u7, Capacitor_SMD:C_1206_3216Metric, F.Cu at (89.9, 111.0)
- added C43: 100n, Capacitor_SMD:C_0603_1608Metric, F.Cu at (86.5, 110.7)
- added C44: 100n, Capacitor_SMD:C_0603_1608Metric, F.Cu at (87.5, 113.0)
- added C45: 47u, Capacitor_SMD:C_1206_3216Metric, F.Cu at (84.0, 117.5)
- added C46: 100n, Capacitor_SMD:C_0603_1608Metric, F.Cu at (121.5, 119.2)
- added C47: 4u7, Capacitor_SMD:C_1206_3216Metric, F.Cu at (123.5, 118.4)
- added C48: 100n, Capacitor_SMD:C_0603_1608Metric, F.Cu at (95.5, 119.0)
- added C49: 4u7, Capacitor_SMD:C_1206_3216Metric, F.Cu at (95.5, 115.0)
- added C50: 4u7, Capacitor_SMD:C_1206_3216Metric, F.Cu at (93.0, 115.0)
- added C51: 220n, Capacitor_SMD:C_0805_2012Metric, F.Cu at (124.0, 111.5)
- added C52: 100n, Capacitor_SMD:C_0603_1608Metric, F.Cu at (102.5, 120.0)
- added C53: 100n, Capacitor_SMD:C_0603_1608Metric, F.Cu at (102.5, 113.0)
- added C54: 4u7, Capacitor_SMD:C_1206_3216Metric, F.Cu at (102.5, 110.5)
- added C55: 220n, Capacitor_SMD:C_0805_2012Metric, F.Cu at (88.0, 85.2)
- added C56: 100n, Capacitor_SMD:C_0603_1608Metric, F.Cu at (107.8, 119.1)
- added C57: 100n, Capacitor_SMD:C_0603_1608Metric, F.Cu at (116.0, 88.5)
- added C58: 100n, Capacitor_SMD:C_0603_1608Metric, F.Cu at (119.5, 119.2)
- added Q4: DMC3028LSD, Package_SO:SO-8_3.9x4.9mm_P1.27mm, F.Cu at (81.0, 96.0)
- added R19: 20k, Resistor_SMD:R_0603_1608Metric, F.Cu at (87.8, 115.5)
- added R20: 100M, Resistor_SMD:R_0805_2012Metric, F.Cu at (90.5, 114.5)
- added R21: 100k, Resistor_SMD:R_0603_1608Metric, F.Cu at (81.6, 87.5)
- added R22: 100k, Resistor_SMD:R_0603_1608Metric, F.Cu at (82.4, 85.0)
- added R23: 100k, Resistor_SMD:R_0603_1608Metric, F.Cu at (80.8, 85.0)
- added RN14: 1k, Resistor_SMD:R_Array_Convex_2x0603, F.Cu at (85.0, 85.7)
- added TH1: 100k NTC, Resistor_SMD:R_0603_1608Metric, B.Cu at (96.0, 100.0)
- added U5: THP210DGK, Package_SO:VSSOP-8_3x3mm_P0.65mm, F.Cu at (109.5, 115.0)
- added U6: OPA2197xD, Package_SO:SOIC-8_3.9x4.9mm_P1.27mm, F.Cu at (113.5, 106.0)
- added U8: THP210DGK, Package_SO:VSSOP-8_3x3mm_P0.65mm, F.Cu at (117.9, 84.5)
- added U9: OPA2197xD, Package_SO:SOIC-8_3.9x4.9mm_P1.27mm, F.Cu at (109.5, 84.5)
- C10, C22, C28: value 10u -> 4u7
- C11: value 10n -> 4u7; footprint Capacitor_SMD:C_0603_1608Metric -> Capacitor_SMD:C_1206_3216Metric
- C13: value 100n -> 10n
- C14, C26: value 47u -> 4u7; footprint Capacitor_THT:C_Rect_L18.0mm_W7.0mm_P15.00mm_FKS3_FKP3 -> Capacitor_SMD:C_1206_3216Metric
- C15: value 220n -> 100n; footprint Capacitor_SMD:C_0805_2012Metric -> Capacitor_SMD:C_0603_1608Metric
- C16: value 10u -> 100n; footprint Capacitor_SMD:C_1206_3216Metric -> Capacitor_SMD:C_0603_1608Metric
- C17: value 10n -> 47u; footprint Capacitor_SMD:C_0603_1608Metric -> Capacitor_SMD:C_1206_3216Metric
- C18, C24, C9: value 4u7 -> 100n; footprint Capacitor_SMD:C_1206_3216Metric -> Capacitor_SMD:C_0603_1608Metric
- C19: value 100n -> 4u7; footprint Capacitor_SMD:C_0603_1608Metric -> Capacitor_SMD:C_1206_3216Metric
- C20: value 47u -> 100n; footprint Capacitor_THT:C_Rect_L18.0mm_W7.0mm_P15.00mm_FKS3_FKP3 -> Capacitor_SMD:C_0603_1608Metric
- C21: value 220n -> 4u7; footprint Capacitor_SMD:C_0805_2012Metric -> Capacitor_SMD:C_1206_3216Metric
- C23: value 10n -> 220n; footprint Capacitor_SMD:C_0603_1608Metric -> Capacitor_SMD:C_0805_2012Metric
- C27: value 220n -> 10n; footprint Capacitor_SMD:C_0805_2012Metric -> Capacitor_SMD:C_0603_1608Metric
- R10, R14, R18: value 100M -> 300k; footprint Resistor_SMD:R_0805_2012Metric -> Resistor_SMD:R_0603_1608Metric
- R11, R15: value 120 -> 20k
- R12, R16: value 300k -> 100M; footprint Resistor_SMD:R_0603_1608Metric -> Resistor_SMD:R_0805_2012Metric
- R13, R17, R9: value 20k -> 120
- R6: value 20k -> 20
- R7: value 120 -> 20
- R8: value 300k -> 20k
- U10, U4, U7: value OPA2197xD -> INA851RGTR; footprint Package_SO:SOIC-8_3.9x4.9mm_P1.27mm -> magnode_footprints:VQFN-16-1EP_3x3mm_P0.5mm_EP1.68x1.68mm
- U11: value INA851RGTR -> THP210DGK; footprint magnode_footprints:VQFN-16-1EP_3x3mm_P0.5mm_EP1.68x1.68mm -> Package_SO:VSSOP-8_3x3mm_P0.65mm
- U12: value THP210DGK -> OPA2197xD; footprint Package_SO:VSSOP-8_3x3mm_P0.65mm -> Package_SO:SOIC-8_3.9x4.9mm_P1.27mm
- U3: value OPA4197xD -> OPA2197xD; footprint Package_SO:SOIC-14_3.9x8.7mm_P1.27mm -> Package_SO:SOIC-8_3.9x4.9mm_P1.27mm
- moved C26 91.5 mm to (115.0, 110.0)
- moved C23 88.3 mm to (116.5, 113.0)
- moved RN12 87.8 mm to (123.5, 114.1), turned to -90 degrees
- moved U11 85.6 mm to (120.5, 114.5), turned to 90 degrees
- moved C25 81.7 mm to (111.5, 110.3), turned to -90 degrees
- moved U10 80.1 mm to (83.4, 112.1), turned to -90 degrees
- moved U12 78.6 mm to (100.5, 116.5)
- moved RN4 77.8 mm to (113.0, 114.4), turned to 180 degrees
- moved R18 75.3 mm to (84.5, 115.5)
- moved C11 75.0 mm to (124.5, 104.0), turned to -90 degrees
- moved RN13 74.4 mm to (98.6, 112.5), turned to 180 degrees
- moved RN10 73.5 mm to (83.6, 104.1), turned to -90 degrees
- moved C5 70.9 mm to (76.0, 109.2), turned to 90 degrees
- moved RN5 70.5 mm to (109.0, 110.5), turned to 180 degrees
- moved R17 68.8 mm to (83.3, 109.1)
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Connections:
- net Net-(U3B-+) renamed /VOLTAGE_REF/1V65_FLTR
- C11 pad 1: /ANALOG_BALANCING_X/BR_X+ -> /VOLTAGE_REF/4V5_DIV
- C11 pad 2: /ANALOG_BALANCING_X/BR_X- -> GND
- C13 pad 1: +9VA -> /SENSOR_3AXIS_HMC100X/BR_X+
- C13 pad 2: GND -> /SENSOR_3AXIS_HMC100X/BR_X-
- C14 pad 1: /ANALOG_BALANCING_X/INA_OUT_FLTR+ -> +9VA
- C14 pad 2: +4V5B -> GND
- C15 pad 1: /ANALOG_BALANCING_X/ERR_OUT- -> +9VA
- C15 pad 2: /ANALOG_BALANCING_X/ERR_OUT+ -> GND
- C16 pad 1: Net-(U4A--) -> +4V5B
- C16 pad 2: Net-(RN2B-R2.2) -> GND
- C17 pad 1: /ANALOG_BALANCING_Y/BR_X+ -> /X_BALANCING/INA_OUT_FLTR+
- C17 pad 2: /ANALOG_BALANCING_Y/BR_X- -> +4V5B
- C20 pad 1: /ANALOG_BALANCING_Y/INA_OUT_FLTR+ -> +4V5B
- C20 pad 2: +4V5B -> GND
- C21 pad 1: /ANALOG_BALANCING_Y/ERR_OUT- -> /X_BALANCING/INT_FB
- C21 pad 2: /ANALOG_BALANCING_Y/ERR_OUT+ -> /X_BALANCING/COMP+
- C22 pad 1: Net-(U7A--) -> /X_BALANCING/INT_FB
- C22 pad 2: Net-(RN6B-R2.2) -> /X_BALANCING/COMP+
- C23 pad 1: /ANALOG_BALANCING_Z/BR_X+ -> /CONNECTOR/X_CONN-
- C23 pad 2: /ANALOG_BALANCING_Z/BR_X- -> /CONNECTOR/X_CONN+
- C24 pad 1: +9VA -> +4V5B
- C26 pad 1: /ANALOG_BALANCING_Z/INA_OUT_FLTR+ -> +9VA
- C26 pad 2: +4V5B -> GND
- C27 pad 1: /ANALOG_BALANCING_Z/ERR_OUT- -> /SENSOR_3AXIS_HMC100X/BR_Y+
- C27 pad 2: /ANALOG_BALANCING_Z/ERR_OUT+ -> /SENSOR_3AXIS_HMC100X/BR_Y-
- C28 pad 1: Net-(U10A--) -> +9VA
- C28 pad 2: Net-(RN10B-R2.2) -> GND
- C9 pad 1: Net-(RN1A-R1.1) -> +9VA
- J1 pad 13: unconnected-(J1-Pad13) -> /CONNECTOR/TH+
- J1 pad 14: unconnected-(J1-Pad14) -> /CONNECTOR/TH-
- J1 pad 22: +3V3A -> +9Vb
- J1 pad 23: +3V3D -> +3V3A
- J1 pad 24: GND -> +3V3D
- J1 pad 28: /CONNECTOR/I2C.SCL -> unconnected-(J1-Pad28)
- J1 pad 29: /CONNECTOR/I2C.SDA -> unconnected-(J1-Pad29)
- R10 pad 1: Net-(U4A--) -> /X_BALANCING/INA_OUT+
- R10 pad 2: Net-(RN2B-R2.2) -> /X_BALANCING/INA_OUT_FLTR+
- R11 pad 1: /ANALOG_BALANCING_Y/X_RG- -> /X_BALANCING/INA_OUT_FLTR+
- R11 pad 2: /ANALOG_BALANCING_Y/X_RG+ -> /X_BALANCING/INT_FB
- R12 pad 1: /ANALOG_BALANCING_Y/INA_OUT+ -> /X_BALANCING/INT_FB
- R12 pad 2: /ANALOG_BALANCING_Y/INA_OUT_FLTR+ -> /X_BALANCING/COMP+
- R13 pad 1: /ANALOG_BALANCING_Y/INA_OUT_FLTR+ -> /Y_BALANCING/X_RG-
- R13 pad 2: Net-(U7A--) -> /Y_BALANCING/X_RG+
- R14 pad 1: Net-(U7A--) -> /Y_BALANCING/INA_OUT+
- R14 pad 2: Net-(RN6B-R2.2) -> /Y_BALANCING/INA_OUT_FLTR+
- R15 pad 1: /ANALOG_BALANCING_Z/X_RG- -> /Y_BALANCING/INA_OUT_FLTR+
- R15 pad 2: /ANALOG_BALANCING_Z/X_RG+ -> /Y_BALANCING/INT_FB
- R16 pad 1: /ANALOG_BALANCING_Z/INA_OUT+ -> /Y_BALANCING/INT_FB
- R16 pad 2: /ANALOG_BALANCING_Z/INA_OUT_FLTR+ -> /Y_BALANCING/COMP+
- R17 pad 1: /ANALOG_BALANCING_Z/INA_OUT_FLTR+ -> /Z_BALANCING/X_RG-
- R17 pad 2: Net-(U10A--) -> /Z_BALANCING/X_RG+
- R18 pad 1: Net-(U10A--) -> /Z_BALANCING/INA_OUT+
- R18 pad 2: Net-(RN10B-R2.2) -> /Z_BALANCING/INA_OUT_FLTR+
- R6 pad 1: /CONNECTOR/DEVICE_DETECT -> /VOLTAGE_REF/4V5_FB
- R6 pad 2: GND -> +4V5B
- R7 pad 1: /ANALOG_BALANCING_X/X_RG- -> /VOLTAGE_REF/1V65_FB
- R7 pad 2: /ANALOG_BALANCING_X/X_RG+ -> +1V65B
- R8 pad 1: /ANALOG_BALANCING_X/INA_OUT+ -> /CONNECTOR/DEVICE_DETECT
- R8 pad 2: /ANALOG_BALANCING_X/INA_OUT_FLTR+ -> GND
- R9 pad 1: /ANALOG_BALANCING_X/INA_OUT_FLTR+ -> /X_BALANCING/X_RG-
- R9 pad 2: Net-(U4A--) -> /X_BALANCING/X_RG+
- RN1 pad 1: Net-(RN1A-R1.1) -> /VOLTAGE_REF/4V5_DIV
- RN1 pad 3: Net-(RN1A-R1.1) -> /VOLTAGE_REF/4V5_DIV
- RN10 pad 3: Net-(RN10B-R2.2) -> /Z_BALANCING/COMP+
- RN10 pad 4: Net-(RN10A-R1.2) -> /Z_BALANCING/COMP-
- RN11 pad 1: /ANALOG_BALANCING_Z/BR_X- -> /SENSOR_3AXIS_HMC100X/BR_Z+
- RN11 pad 2: /ANALOG_BALANCING_Z/BR_X+ -> /SENSOR_3AXIS_HMC100X/BR_Z-
- RN12 pad 1: /ANALOG_BALANCING_Z/ERR_OUT+ -> /CONNECTOR/Z_CONN+
- RN12 pad 2: /ANALOG_BALANCING_Z/ERR_OUT- -> /CONNECTOR/Z_CONN-
- RN12 pad 3: Net-(RN12B-R2.2) -> /Z_BALANCING/THP_OUT-
- RN12 pad 4: Net-(RN12A-R1.2) -> /Z_BALANCING/THP_OUT+
- RN13 pad 1: Net-(RN13A-R1.1) -> /Z_BALANCING/INV_FB
- RN13 pad 2: Net-(RN10A-R1.2) -> /Z_BALANCING/COMP-
- RN13 pad 3: Net-(RN13A-R1.1) -> /Z_BALANCING/INV_FB
- RN13 pad 4: Net-(RN10B-R2.2) -> /Z_BALANCING/COMP+
- RN2 pad 3: Net-(RN2B-R2.2) -> /X_BALANCING/COMP+
- RN2 pad 4: Net-(RN2A-R1.2) -> /X_BALANCING/COMP-
- RN3 pad 1: /ANALOG_BALANCING_X/BR_X- -> /SENSOR_3AXIS_HMC100X/BR_X+
- RN3 pad 2: /ANALOG_BALANCING_X/BR_X+ -> /SENSOR_3AXIS_HMC100X/BR_X-
- RN4 pad 1: /ANALOG_BALANCING_X/ERR_OUT+ -> /CONNECTOR/X_CONN+
- RN4 pad 2: /ANALOG_BALANCING_X/ERR_OUT- -> /CONNECTOR/X_CONN-
- RN4 pad 3: Net-(RN4B-R2.2) -> /X_BALANCING/THP_OUT-
- RN4 pad 4: Net-(RN4A-R1.2) -> /X_BALANCING/THP_OUT+
- RN5 pad 1: Net-(RN5A-R1.1) -> /X_BALANCING/INV_FB
- RN5 pad 2: Net-(RN2A-R1.2) -> /X_BALANCING/COMP-
- RN5 pad 3: Net-(RN5A-R1.1) -> /X_BALANCING/INV_FB
- RN5 pad 4: Net-(RN2B-R2.2) -> /X_BALANCING/COMP+
- RN6 pad 3: Net-(RN6B-R2.2) -> /Y_BALANCING/COMP+
- RN6 pad 4: Net-(RN6A-R1.2) -> /Y_BALANCING/COMP-
- RN7 pad 1: /ANALOG_BALANCING_Y/BR_X- -> /SENSOR_3AXIS_HMC100X/BR_Y+
- RN7 pad 2: /ANALOG_BALANCING_Y/BR_X+ -> /SENSOR_3AXIS_HMC100X/BR_Y-
- RN8 pad 1: /ANALOG_BALANCING_Y/ERR_OUT+ -> /CONNECTOR/Y_CONN+
- RN8 pad 2: /ANALOG_BALANCING_Y/ERR_OUT- -> /CONNECTOR/Y_CONN-
- RN8 pad 3: Net-(RN8B-R2.2) -> /Y_BALANCING/THP_OUT-
- RN8 pad 4: Net-(RN8A-R1.2) -> /Y_BALANCING/THP_OUT+
- RN9 pad 1: Net-(RN9A-R1.1) -> /Y_BALANCING/INV_FB
- RN9 pad 2: Net-(RN6A-R1.2) -> /Y_BALANCING/COMP-
- RN9 pad 3: Net-(RN9A-R1.1) -> /Y_BALANCING/INV_FB
- RN9 pad 4: Net-(RN6B-R2.2) -> /Y_BALANCING/COMP+
- U10 pad 1: Net-(RN10B-R2.2) -> /SENSOR_3AXIS_HMC100X/BR_Z+
- U10 pad 2: Net-(U10A--) -> /Z_BALANCING/X_RG+
- U10 pad 3: +4V5B -> /Z_BALANCING/X_RG-
- U10 pad 4: GND -> /SENSOR_3AXIS_HMC100X/BR_Z-
- U10 pad 5: +4V5B -> GND
- U10 pad 6: Net-(RN13A-R1.1) -> unconnected-(U10-FDA_IN+-Pad6)
- U10 pad 7: Net-(RN10A-R1.2) -> GND
- U10 pad 8: +9VA -> unconnected-(U10-NC-Pad8)
- U11 pad 1: /ANALOG_BALANCING_Z/BR_X+ -> /Z_BALANCING/INA_OUT-
- U11 pad 2: /ANALOG_BALANCING_Z/X_RG+ -> +1V65B
- U11 pad 3: /ANALOG_BALANCING_Z/X_RG- -> +9VA
- U11 pad 4: /ANALOG_BALANCING_Z/BR_X- -> /Z_BALANCING/THP_OUT+
- U11 pad 5: GND -> /Z_BALANCING/THP_OUT-
- U11 pad 6: unconnected-(U11-FDA_IN+-Pad6) -> GND
- U11 pad 7: GND -> +9VA
- U11 pad 8: unconnected-(U11-NC-Pad8) -> /Z_BALANCING/INA_OUT+
- U12 pad 1: /ANALOG_BALANCING_Z/INA_OUT- -> /Z_BALANCING/COMP+
- U12 pad 2: +1V65B -> /Z_BALANCING/INT_FB
- U12 pad 3: +9VA -> +4V5B
- U12 pad 4: Net-(RN12A-R1.2) -> GND
- U12 pad 5: Net-(RN12B-R2.2) -> +4V5B
- U12 pad 6: GND -> /Z_BALANCING/INV_FB
- U12 pad 7: unconnected-(U12-~{PD}-Pad7) -> /Z_BALANCING/COMP-
- U12 pad 8: /ANALOG_BALANCING_Z/INA_OUT+ -> +9VA
- U3 pad 1: +4V5B -> /VOLTAGE_REF/4V5_FB
- U3 pad 2: +4V5B -> /VOLTAGE_REF/4V5_FB
- U3 pad 3: Net-(RN1A-R1.1) -> /VOLTAGE_REF/4V5_DIV
- U3 pad 4: unconnected-(U3E-V+-Pad4) -> GND
- U3 pad 6: +1V65B -> /VOLTAGE_REF/1V65_FB
- U3 pad 7: +1V65B -> /VOLTAGE_REF/1V65_FB
- U3 pad 8: unconnected-(U3-Pad8) -> +9VA
- U4 pad 1: Net-(RN2B-R2.2) -> /SENSOR_3AXIS_HMC100X/BR_X+
- U4 pad 2: Net-(U4A--) -> /X_BALANCING/X_RG+
- U4 pad 3: +4V5B -> /X_BALANCING/X_RG-
- U4 pad 4: GND -> /SENSOR_3AXIS_HMC100X/BR_X-
- U4 pad 5: +4V5B -> GND
- U4 pad 6: Net-(RN5A-R1.1) -> unconnected-(U4-FDA_IN+-Pad6)
- U4 pad 7: Net-(RN2A-R1.2) -> GND
- U4 pad 8: +9VA -> unconnected-(U4-NC-Pad8)
- U7 pad 1: Net-(RN6B-R2.2) -> /SENSOR_3AXIS_HMC100X/BR_Y+
- U7 pad 2: Net-(U7A--) -> /Y_BALANCING/X_RG+
- U7 pad 3: +4V5B -> /Y_BALANCING/X_RG-
- U7 pad 4: GND -> /SENSOR_3AXIS_HMC100X/BR_Y-
- U7 pad 5: +4V5B -> GND
- U7 pad 6: Net-(RN9A-R1.1) -> unconnected-(U7-FDA_IN+-Pad6)
- U7 pad 7: Net-(RN6A-R1.2) -> GND
- U7 pad 8: +9VA -> unconnected-(U7-NC-Pad8)
Routing:
- net +9VA: track 0.00 -> 200.3 mm, vias 0 -> 10
- net +4V5B: track 0.00 -> 150.6 mm, vias 0 -> 13
- net +9Vb: track 0.00 -> 92.6 mm, vias 0 -> 5
- net /CONNECTOR/SENSOR_RESET_CTRL: track 0.00 -> 88.1 mm, vias 0 -> 1
- net /CONNECTOR/SENSOR_SET_CTRL: track 0.00 -> 75.6 mm, vias 0 -> 1
- net +18V: track 0.00 -> 75.2 mm, vias 0 -> 2
- net +1V65B: track 0.00 -> 73.0 mm, vias 0 -> 3
- net +3V3A: track 0.00 -> 68.2 mm, vias 0 -> 3
- net /CONNECTOR/TH+: track 0.00 -> 51.3 mm, vias 0 -> 1
- net GND: track 0.00 -> 51.2 mm, vias 0 -> 125
- net /CONNECTOR/TH-: track 0.00 -> 49.9 mm, vias 0 -> 1
- net /Z_BALANCING/INA_OUT+: track 0.00 -> 44.8 mm, vias 0 -> 2
- net /Z_BALANCING/INA_OUT-: track 0.00 -> 41.2 mm, vias 0 -> 2
- net /X_BALANCING/COMP+: track 0.00 -> 38.2 mm, vias 0 -> 4
- net /Y_BALANCING/COMP+: track 0.00 -> 36.4 mm, vias 0 -> 2
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- added copper zone on F.Cu, net /SENSOR_SET_RESET_DRIVER/18V_PULSE
Other:
- board text added: "1"
