File: hardware/pcb/Expension_card_design/magnetic_expension_v2/magnetic_expension_v2.kicad_sch (KiCad schematic)
At the start: 0 parts

Commit message: kicad mag board done
Other:
- sheet ANALOG_BALANCING_X renamed X_BALANCING
- sheet ANALOG_BALANCING_Y renamed Y_BALANCING
- sheet ANALOG_BALANCING_Z renamed Z_BALANCING
- added sheet THERMISTOR (schematics/thermistor.kicad_sch)
- sheet CONNECTOR ports: added I2C{SDA SCL}, TH+, TH-; removed none
- sheet X_BALANCING ports: added BRIDGE+, BRIDGE-, ERR_OUT+, ERR_OUT-; removed none
- sheet Y_BALANCING ports: added BRIDGE+, BRIDGE-, ERR_OUT+, ERR_OUT-; removed none
- sheet Z_BALANCING ports: added BRIDGE+, BRIDGE-, ERR_OUT+, ERR_OUT-; removed none
