File: hardware/pcb/Expension_card_design/magnetic_expension_v2/schematics/ANALOG_BALANCING.kicad_sch (KiCad schematic)
At the start: 18 parts, among them U4 OPA2197xD, U5 INA851RGTR, U6 THP210DGK

Commit message: kicad mag board done
Parts:
- added C16, C18, C20, C24, C25, C56: 100n, Capacitor_SMD:C_0603_1608Metric, symbol Device:C
- added C19, C26: 4u7, Capacitor_SMD:C_1206_3216Metric, symbol Device:C
- C17: renamed from C14; footprint Capacitor_THT:C_Rect_L18.0mm_W7.0mm_P15.00mm_FKS3_FKP3 -> Capacitor_SMD:C_1206_3216Metric
- renumbered C11 to C13, C12 to C14, C13 to C15, C29 to C21, C16 to C22, C15 to C23, R8 to R10, R9 to R11, R10 to R12, R7 to R9, U5 to U4, U6 to U5, U4 to U6
Connections:
- net +1V65B: now also C56.1
- net +4V5B: now also C16.1, C20.1, C24.1
- net +9VA: now also U5.7 (~{PD}), C18.1, C19.1, C25.1, C26.1
- net GND: now also C16.2, C18.2, C19.2, C20.2, C24.2, C25.2, C26.2, C56.2
- net COMP+: now reaches C21.2, C22.2, R12.2, RN2.3 (R2.2), RN5.4 (R1.2), U6.1
- net INT_FB: now reaches C21.1, C22.1, R11.2, R12.1, U6.2 (-)
- net COMP-: now reaches RN2.4 (R1.2), RN5.2 (R2.1), U6.7
- net THP_OUT-: now reaches RN4.3 (R2.2), U5.5
- net THP_OUT+: now reaches RN4.4 (R1.2), U5.4
- net INV_FB: now reaches RN5.1 (R1.1), RN5.3 (R2.2), U6.6 (-)
- net BR_X+ renamed BRIDGE+
- net BRIDGE+: now also RN3.1 (R1.1); no longer RN3.2 (R2.1)
- net BR_X- renamed BRIDGE-
- net BRIDGE-: now also RN3.2 (R2.1); no longer RN3.1 (R1.1)
Other:
- moved on the sheet: C17, C21, C22, C23, R10, R11, R12, RN4A, RN4B, RN5B, U5, U6A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
