File: hardware/pcb/Expension_card_design/mainboard_v2/schematics/sensor_hmc100x_3axis.kicad_sch (KiCad schematic)
At the start: 6 parts, among them U1 HMC1001-RC, U2 HMC1002-TR

Commit message: kicad mag board done
Parts:
- removed C1: 10u, Capacitor_SMD:C_1206_3216Metric, symbol Device:C
- removed C2, C3, C4: 100n, Capacitor_SMD:C_0603_1608Metric, symbol Device:C
Connections:
- net GND: no longer U1.2 (OFFSET+), U2.15 (OFFSET+(B)), U2.17 (OFFSET(+A))
- net +9Vb renamed +9VA
- new net OFFSET_X+: U2.17 (OFFSET(+A))
- new net OFFSET_Y+: U2.15 (OFFSET+(B))
- new net OFFSET_Z+: U1.2 (OFFSET+)
Other:
- note added: "bypass cap"
